File: board/mainboard/peripherals.sch (KiCad schematic (older format))
At the start: 2 parts

Commit message: Added schematic for RTC
Parts:
- added C?: C, ~, symbol C
- added RTC?: S-35390A, ~, symbol S-35390A
- added X?: CRYSTAL_SMD, ~, symbol CRYSTAL_SMD
Connections:
- net labels added: RTCINT
- wire segments 10 -> 23
- no-connect marks 0 -> 1
Changed lines of the file:
@@
 Sheet 2 2
 Title ""
-Date "22 oct 2014"
+Date "23 oct 2014"
 Rev ""
 Comp ""
@@
 Text Notes 2150 1000 0    60   ~ 0
 Temperature Sensor\nI2C ADDR = 1001000x
+$Comp
+L S-35390A RTC?
+U 1 1 54485BFB
+P 2950 3350
+F 0 "RTC?" H 2950 3250 60  0000 C CNN
+F 1 "S-35390A" H 2950 3450 60  0000 C CNN
+F 2 "~" H 2950 3450 60  0000 C CNN
+F 3 "~" H 2950 3450 60  0000 C CNN
+	1    2950 3350
+	1    0    0    -1
+$EndComp
+Text GLabel 1700 3150 0    60   Input ~ 0
+RTCINT
+$Comp
+L CRYSTAL_SMD X?
+U 1 1 54485CEB
+P 1600 3550
+F 0 "X?" H 1600 3640 30  0000 C CNN
+F 1 "CRYSTAL_SMD" H 1630 3440 30  0000 L CNN
+F 2 "~" H 1600 3550 60  0000 C CNN
+F 3 "~" H 1600 3550 60  0000 C CNN
+	1    1600 3550
+	0    -1   -1   0
+$EndComp
 Wire Wire Line
 	1850 1450 1400 1450
@@
 Wire Wire Line
 	3450 1600 3250 1600
+Wire Wire Line
+	2150 3150 1700 3150
+Wire Wire Line
+	2150 3300 1600 3300
+Wire Wire Line
+	1600 3300 1600 3350
+Wire Wire Line
+	1900 3450 2150 3450
+$Comp
+L C C?
+U 1 1 54485D29
+P 1900 3950
+F 0 "C?" H 1900 4050 40  0000 L CNN
+F 1 "C" H 1906 3865 40  0000 L CNN
+F 2 "~" H 1938 3800 30  0000 C CNN
+F 3 "~" H 1900 3950 60  0000 C CNN
+	1    1900 3950
+	-1   0    0    1
+$EndComp
+Wire Wire Line
+	1900 3450 1900 3750
+Wire Wire Line
+	1900 3750 1600 3750
+$Comp
+L GND #PWR?
+U 1 1 54485DA7
+P 1900 4200
+F 0 "#PWR?" H 1900 4200 30  0001 C CNN
+F 1 "GND" H 1900 4130 30  0001 C CNN
+F 2 "" H 1900 4200 60  0000 C CNN
+F 3 "" H 1900 4200 60  0000 C CNN
+	1    1900 4200
+	1    0    0    -1
+$EndComp
+Wire Wire Line
+	1900 4150 1900 4200
+$Comp
+L GND #PWR?
+U 1 1 54485DC8
+P 2100 3850
+F 0 "#PWR?" H 2100 3850 30  0001 C CNN
+F 1 "GND" H 2100 3780 30  0001 C CNN
+F 2 "" H 2100 3850 60  0000 C CNN
+F 3 "" H 2100 3850 60  0000 C CNN
+	1    2100 3850
+	1    0    0    -1
+$EndComp
+Wire Wire Line
+	2100 3850 2100 3600
+Wire Wire Line
+	2100 3600 2150 3600
+$Comp
+L 3V3 #PWR?
+U 1 1 54485DFD
+P 3850 2950
+F 0 "#PWR?" H 3850 3050 40  0001 C CNN
+F 1 "3V3" H 3850 3075 40  0000 C CNN
+F 2 "" H 3850 2950 60  0000 C CNN
+F 3 "" H 3850 2950 60  0000 C CNN
+	1    3850 2950
+	1    0    0    -1
+$EndComp
+Wire Wire Line
+	3850 2950 3850 3150
+Wire Wire Line
+	3850 3150 3750 3150
+NoConn ~ 3750 3600
+Text GLabel 4000 3450 2    60   Input ~ 0
+I2C_CL
+Text GLabel 4000 3300 2    60   Input ~ 0
+I2C_DA
+Wire Wire Line
+	4000 3450 3750 3450
+Wire Wire Line
+	3750 3300 4000 3300
 $EndSCHEMATC

Commit message: Added The motor driver circuits
Parts:
- added MC? (x2): DRV8830, ~, symbol DRV8830
- added R? (x2): 0.2, ~, symbol R
- C?: value C -> Cg
- X?: value CRYSTAL_SMD -> 32.768kHz
Connections:
- net labels added: MOTOR1+, MOTOR1-, MOTOR1F, RTCINT1, RTCINT2
- net labels removed: RTCINT
- wire segments 23 -> 49
- no-connect marks 1 -> 4
Other:
- note added: "Motor 1 Driver Circuit\nI2C ADDR = 0xC0-0xC1"
- note added: "Motor 2 Driver Circuit\nI2C ADDR = 0xC2-0xC3"
- note added: "Real Time Clock\nAddress 60-6F"
Changed lines of the file:
@@
 $EndComp
 Text GLabel 1700 3150 0    60   Input ~ 0
-RTCINT
+RTCINT1
 $Comp
 L CRYSTAL_SMD X?
@@
 P 1600 3550
 F 0 "X?" H 1600 3640 30  0000 C CNN
-F 1 "CRYSTAL_SMD" H 1630 3440 30  0000 L CNN
+F 1 "32.768kHz" H 1630 3440 30  0000 L CNN
 F 2 "~" H 1600 3550 60  0000 C CNN
 F 3 "~" H 1600 3550 60  0000 C CNN
@@
 	0    -1   -1   0
 $EndComp
-Wire Wire Line
-	1850 1450 1400 1450
-Wire Wire Line
-	1850 1600 1650 1600
-Wire Wire Line
-	1650 1600 1650 2000
-Wire Wire Line
-	3250 1450 3550 1450
-Wire Wire Line
-	4000 1200 4000 1750
-Wire Wire Line
-	4000 1750 3250 1750
-Wire Wire Line
-	4000 2150 4000 2350
-Wire Wire Line
-	1850 1750 1650 1750
-Connection ~ 1650 1750
-Wire Wire Line
-	3450 1600 3450 2000
-Wire Wire Line
-	3450 1600 3250 1600
-Wire Wire Line
-	2150 3150 1700 3150
-Wire Wire Line
-	2150 3300 1600 3300
-Wire Wire Line
-	1600 3300 1600 3350
-Wire Wire Line
-	1900 3450 2150 3450
 $Comp
 L C C?
@@
 P 1900 3950
 F 0 "C?" H 1900 4050 40  0000 L CNN
-F 1 "C" H 1906 3865 40  0000 L CNN
+F 1 "Cg" H 1906 3865 40  0000 L CNN
 F 2 "~" H 1938 3800 30  0000 C CNN
 F 3 "~" H 1900 3950 60  0000 C CNN
@@
 	-1   0    0    1
 $EndComp
-Wire Wire Line
-	1900 3450 1900 3750
-Wire Wire Line
-	1900 3750 1600 3750
 $Comp
 L GND #PWR?
@@
 	1    0    0    -1
 $EndComp
-Wire Wire Line
-	1900 4150 1900 4200
 $Comp
 L GND #PWR?
@@
 	1    0    0    -1
 $EndComp
-Wire Wire Line
-	2100 3850 2100 3600
-Wire Wire Line
-	2100 3600 2150 3600
 $Comp
 L 3V3 #PWR?
@@
 	1    0    0    -1
 $EndComp
-Wire Wire Line
-	3850 2950 3850 3150
-Wire Wire Line
-	3850 3150 3750 3150
 NoConn ~ 3750 3600
 Text GLabel 4000 3450 2    60   Input ~ 0
@@
 Text GLabel 4000 3300 2    60   Input ~ 0
 I2C_DA
+$Comp
+L DRV8830 MC?
+U 1 1 544869FB
+P 9000 1850
+F 0 "MC?" H 9000 1700 60  0000 C CNN
+F 1 "DRV8830" H 9000 1950 60  0000 C CNN
+F 2 "~" H 8950 2050 60  0000 C CNN
+F 3 "~" H 8950 2050 60  0000 C CNN
+	1    9000 1850
+	1    0    0    -1
+$EndComp
+Text Notes 2600 2750 0    60   ~ 0
+Real Time Clock\nAddress 60-6F
+Text GLabel 10150 1750 2    60   Input ~ 0
+MOTOR1-
+Text GLabel 10150 1600 2    60   Input ~ 0
+MOTOR1+
+$Comp
+L 3V3 #PWR?
+U 1 1 54486A99
+P 7950 1100
+F 0 "#PWR?" H 7950 1200 40  0001 C CNN
+F 1 "3V3" H 7950 1225 40  0000 C CNN
+F 2 "" H 7950 1100 60  0000 C CNN
+F 3 "" H 7950 1100 60  0000 C CNN
+	1    7950 1100
+	1    0    0    -1
+$EndComp
+Text GLabel 7700 1750 0    60   Input ~ 0
+I2C_CL
+Text GLabel 7700 1600 0    60   Input ~ 0
+I2C_DA
+$Comp
+L GND #PWR?
+U 1 1 54486B17
+P 7900 2550
+F 0 "#PWR?" H 7900 2550 30  0001 C CNN
+F 1 "GND" H 7900 2480 30  0001 C CNN
+F 2 "" H 7900 2550 60  0000 C CNN
+F 3 "" H 7900 2550 60  0000 C CNN
+	1    7900 2550
+	1    0    0    -1
+$EndComp
+NoConn ~ 8150 2300
+$Comp
+L GND #PWR?
+U 1 1 54486B7F
+P 9000 2800
+F 0 "#PWR?" H 9000 2800 30  0001 C CNN
+F 1 "GND" H 9000 2730 30  0001 C CNN
+F 2 "" H 9000 2800 60  0000 C CNN
+F 3 "" H 9000 2800 60  0000 C CNN
+	1    9000 2800
+	1    0    0    -1
+$EndComp
+$Comp
+L R R?
+U 1 1 54486C37
+P 10050 2550
+F 0 "R?" V 10130 2550 40  0000 C CNN
+F 1 "0.2" V 10057 2551 40  0000 C CNN
+F 2 "~" V 9980 2550 30  0000 C CNN
+F 3 "~" H 10050 2550 30  0000 C CNN
+	1    10050 2550
+	1    0    0    -1
+$EndComp
+$Comp
+L GND #PWR?
+U 1 1 54486C8F
+P 10050 2900
+F 0 "#PWR?" H 10050 2900 30  0001 C CNN
+F 1 "GND" H 10050 2830 30  0001 C CNN
+F 2 "" H 10050 2900 60  0000 C CNN
+F 3 "" H 10050 2900 60  0000 C CNN
+	1    10050 2900
+	1    0    0    -1
+$EndComp
+$Comp
+L DRV8830 MC?
+U 1 1 544871A6
+P 9000 4250
+F 0 "MC?" H 9000 4100 60  0000 C CNN
+F 1 "DRV8830" H 9000 4350 60  0000 C CNN
+F 2 "~" H 8950 4450 60  0000 C CNN
+F 3 "~" H 8950 4450 60  0000 C CNN
+	1    9000 4250
+	1    0    0    -1
+$EndComp
+Text GLabel 10150 4150 2    60   Input ~ 0
+MOTOR1-
+Text GLabel 10150 4000 2    60   Input ~ 0
+MOTOR1+
+$Comp
+L 3V3 #PWR?
+U 1 1 544871AE
+P 7950 3500
+F 0 "#PWR?" H 7950 3600 40  0001 C CNN
+F 1 "3V3" H 7950 3625 40  0000 C CNN
+F 2 "" H 7950 3500 60  0000 C CNN
+F 3 "" H 7950 3500 60  0000 C CNN
+	1    7950 3500
+	1    0    0    -1
+$EndComp
+Text GLabel 7700 4150 0    60   Input ~ 0
+I2C_CL
+Text GLabel 7700 4000 0    60   Input ~ 0
+I2C_DA
+$Comp
+L GND #PWR?
+U 1 1 544871BA
+P 7900 4950
+F 0 "#PWR?" H 7900 4950 30  0001 C CNN
+F 1 "GND" H 7900 4880 30  0001 C CNN
+F 2 "" H 7900 4950 60  0000 C CNN
+F 3 "" H 7900 4950 60  0000 C CNN
+	1    7900 4950
+	1    0    0    -1
+$EndComp
+NoConn ~ 8150 4700
+$Comp
+L GND #PWR?
+U 1 1 544871C5
+P 9000 5200
+F 0 "#PWR?" H 9000 5200 30  0001 C CNN
+F 1 "GND" H 9000 5130 30  0001 C CNN
+F 2 "" H 9000 5200 60  0000 C CNN
+F 3 "" H 9000 5200 60  0000 C CNN
+	1    9000 5200
+	1    0    0    -1
+$EndComp
+$Comp
+L R R?
+U 1 1 544871CE
+P 10050 4950
+F 0 "R?" V 10130 4950 40  0000 C CNN
+F 1 "0.2" V 10057 4951 40  0000 C CNN
+F 2 "~" V 9980 4950 30  0000 C CNN
+F 3 "~" H 10050 4950 30  0000 C CNN
+	1    10050 4950
+	1    0    0    -1
+$EndComp
+$Comp
+L GND #PWR?
+U 1 1 544871D5
+P 10050 5300
+F 0 "#PWR?" H 10050 5300 30  0001 C CNN
+F 1 "GND" H 10050 5230 30  0001 C CNN
+F 2 "" H 10050 5300 60  0000 C CNN
+F 3 "" H 10050 5300 60  0000 C CNN
+	1    10050 5300
+	1    0    0    -1
+$EndComp
+NoConn ~ 8150 4350
+Text Notes 8550 3300 0    60   ~ 0
+Motor 2 Driver Circuit\nI2C ADDR = 0xC2-0xC3
+Text Notes 8450 900  0    60   ~ 0
+Motor 1 Driver Circuit\nI2C ADDR = 0xC0-0xC1
+Text GLabel 7700 2300 0    60   Input ~ 0
+MOTOR1F
+Text GLabel 7700 4700 0    60   Input ~ 0
+MOTOR1F
+Wire Wire Line
+	1850 1450 1400 1450
+Wire Wire Line
+	1850 1600 1650 1600
+Wire Wire Line
+	1650 1600 1650 2000
+Wire Wire Line
+	3250 1450 3550 1450
+Wire Wire Line
+	4000 1200 4000 1750
+Wire Wire Line
+	4000 1750 3250 1750
+Wire Wire Line
+	4000 2150 4000 2350
+Wire Wire Line
+	1850 1750 1650 1750
+Connection ~ 1650 1750
+Wire Wire Line
+	3450 1600 3450 2000
+Wire Wire Line
+	3450 1600 3250 1600
+Wire Wire Line
+	2150 3150 1700 3150
+Wire Wire Line
+	2150 3300 1600 3300
+Wire Wire Line
+	1600 3300 1600 3350
+Wire Wire Line
+	1900 3450 2150 3450
+Wire Wire Line
+	1900 3450 1900 3750
+Wire Wire Line
+	1900 3750 1600 3750
+Wire Wire Line
+	1900 4150 1900 4200
+Wire Wire Line
+	2100 3850 2100 3600
+Wire Wire Line
+	2100 3600 2150 3600
+Wire Wire Line
+	3850 2950 3850 3150
+Wire Wire Line
+	3850 3150 3750 3150
 Wire Wire Line
 	4000 3450 3750 3450
 Wire Wire Line
 	3750 3300 4000 3300
+Wire Wire Line
+	8150 1400 7950 1400
+Wire Wire Line
+	7950 1400 7950 1100
+Wire Wire Line
+	8150 1600 7700 1600
+Wire Wire Line
+	7700 1750 8150 1750
+Wire Wire Line
+	8150 1950 7900 1950
+Wire Wire Line
+	7900 1950 7900 2550
+Wire Wire Line
+	8150 2100 7900 2100
+Connection ~ 7900 2100
+Wire Wire Line
+	9000 2700 9000 2800
+Wire Wire Line
+	10150 1600 9850 1600
+Wire Wire Line
+	9850 1750 10150 1750
+Wire Wire Line
+	9850 2300 10050 2300
+Wire Wire Line
+	10050 2800 10050 2900
+Wire Wire Line
+	8150 3800 7950 3800
+Wire Wire Line
+	7950 3800 7950 3500
+Wire Wire Line
+	8150 4000 7700 4000
+Wire Wire Line
+	7700 4150 8150 4150
+Wire Wire Line
+	8150 4500 7900 4500
+Wire Wire Line
+	9000 5100 9000 5200
+Wire Wire Line
+	10150 4000 9850 4000
+Wire Wire Line
+	9850 4150 10150 4150
+Wire Wire Line
+	9850 4700 10050 4700
+Wire Wire Line
+	10050 5200 10050 5300
+Wire Wire Line
+	7900 4500 7900 4950
+Wire Wire Line
+	7700 2300 8150 2300
+Wire Wire Line
+	7700 4700 8150 4700
+Text GLabel 4000 3600 2    60   Input ~ 0
+RTCINT2
+Wire Wire Line
+	3750 3600 4000 3600
 $EndSCHEMATC

Commit message: Fixed motor controller 2 connecting to motor 1 nets
Connections:
- net labels added: MOTOR2+, MOTOR2-, MOTOR2F
Changed lines of the file:
@@
 $EndComp
 Text GLabel 10150 4150 2    60   Input ~ 0
-MOTOR1-
+MOTOR2-
 Text GLabel 10150 4000 2    60   Input ~ 0
-MOTOR1+
+MOTOR2+
 $Comp
 L 3V3 #PWR?
@@
 MOTOR1F
 Text GLabel 7700 4700 0    60   Input ~ 0
-MOTOR1F
+MOTOR2F
 Wire Wire Line
 	1850 1450 1400 1450
