File: board/mainboard/mainboard.sch (KiCad schematic (older format))
At the start: 1 part

Commit message: Removed RST inverter
Parts:
- removed INV?: SN74LVC1G04, symbol SN74LVC1G04
Connections:
- net labels removed: 3V3, GND, RST, ~RST
- wire segments 4 -> 0
Changed lines of the file:
@@
 F1 "SPI_peripherals.sch" 50
 $EndSheet
-Text GLabel 9650 1200 0    60   Input ~ 0
-~RST
-Text GLabel 10900 1200 2    60   Input ~ 0
-RST
-$Comp
-L GND #PWR?
-U 1 1 54556D99
-P 10200 1700
-F 0 "#PWR?" H 10200 1700 30  0001 C CNN
-F 1 "GND" H 10200 1630 30  0001 C CNN
-F 2 "" H 10200 1700 60  0000 C CNN
-F 3 "" H 10200 1700 60  0000 C CNN
-	1    10200 1700
-	1    0    0    -1
-$EndComp
-$Comp
-L 3V3 #PWR?
-U 1 1 54556DAA
-P 10200 700
-F 0 "#PWR?" H 10200 800 40  0001 C CNN
-F 1 "3V3" H 10200 825 40  0000 C CNN
-F 2 "" H 10200 700 60  0000 C CNN
-F 3 "" H 10200 700 60  0000 C CNN
-	1    10200 700
-	1    0    0    -1
-$EndComp
-$Comp
-L SN74LVC1G04 INV?
-U 1 1 54556F3C
-P 10200 1200
-F 0 "INV?" H 10500 1300 40  0000 C CNN
-F 1 "SN74LVC1G04" H 10500 1400 40  0000 C CNN
-F 2 "" H 10200 1200 60  0000 C CNN
-F 3 "" H 10200 1200 60  0000 C CNN
-	1    10200 1200
-	1    0    0    -1
-$EndComp
-Wire Wire Line
-	10200 700  10200 750
-Wire Wire Line
-	9700 1200 9650 1200
-Wire Wire Line
-	10200 1650 10200 1700
-Wire Wire Line
-	10900 1200 10850 1200
 $EndSCHEMATC
