File: board/mainboard/mainboard.sch (KiCad schematic (older format))
At the start: 0 parts

Commit message: Added capacitive touch/slider components Removed potentiometer as component
Changed lines of the file:
@@
 $Descr A4 11693 8268
 encoding utf-8
-Sheet 1 8
+Sheet 1 9
 Title ""
 Date "3 mar 2015"
@@
 F1 "Audio.sch" 50
 $EndSheet
+$Sheet
+S 3450 4550 2350 1450
+U 55A4709C
+F0 "Analog" 60
+F1 "Analog.sch" 60
+$EndSheet
 $EndSCHEMATC
