File: board/mainboard/AudioCodec.sch (KiCad schematic (older format))
At the start: 22 parts

Commit message: Fixed crystals and added mic to audio codec
Parts:
- added MIC?: CMA-4544PF-W, symbol CMA-4544PF-W
Connections:
- net labels removed: MIC_GND, MIC_IN
- wire segments 81 -> 83
Changed lines of the file:
@@
 $EndComp
 Wire Wire Line
-	8000 4200 8700 4200
+	8000 4200 8750 4200
 Wire Wire Line
 	8150 4200 8150 4400
@@
 	7700 5400 7700 5450
 Wire Wire Line
-	6800 5450 8650 5450
+	8750 5450 6800 5450
 Wire Wire Line
 	8150 5450 8150 4900
@@
 SPI_CS4
 Connection ~ 2000 3050
-Text GLabel 8700 4200 2    60   Input ~ 0
-MIC_IN
-Text GLabel 8650 5450 2    60   Input ~ 0
-MIC_GND
 Connection ~ 8150 4200
 Connection ~ 8150 5450
 NoConn ~ 4750 4500
 NoConn ~ 4750 4350
+$Comp
+L CMA-4544PF-W MIC?
+U 1 1 546AC917
+P 8700 4800
+F 0 "MIC?" H 8700 4550 60  0000 C CNN
+F 1 "CMA-4544PF-W" H 8650 5050 60  0001 C CNN
+F 2 "" H 8650 5050 60  0000 C CNN
+F 3 "" H 8650 5050 60  0000 C CNN
+	1    8700 4800
+	0    -1   -1   0
+$EndComp
+Wire Wire Line
+	8750 4200 8750 4500
+Wire Wire Line
+	8750 5100 8750 5450
 $EndSCHEMATC

Commit message: Changed buffers to 3v3 compatible version
Parts:
- U? (x4): value 74LS125 -> 74ALVC125
Changed lines of the file:
@@
 $Descr A4 11693 8268
 encoding utf-8
-Sheet 5 5
+Sheet 5 6
 Title ""
-Date "19 nov 2014"
+Date "23 nov 2014"
 Rev ""
 Comp ""
@@
 P 2650 1100
 F 0 "U?" H 2650 1200 50  0000 L BNN
-F 1 "74LS125" H 2700 950 40  0000 L TNN
+F 1 "74ALVC125" H 2700 950 40  0000 L TNN
 F 2 "~" H 2650 1100 60  0000 C CNN
 F 3 "~" H 2650 1100 60  0000 C CNN
@@
 P 2650 1650
 F 0 "U?" H 2650 1750 50  0000 L BNN
-F 1 "74LS125" H 2700 1500 40  0000 L TNN
+F 1 "74ALVC125" H 2700 1500 40  0000 L TNN
 F 2 "~" H 2650 1650 60  0000 C CNN
 F 3 "~" H 2650 1650 60  0000 C CNN
@@
 P 2650 2200
 F 0 "U?" H 2650 2300 50  0000 L BNN
-F 1 "74LS125" H 2700 2050 40  0000 L TNN
+F 1 "74ALVC125" H 2700 2050 40  0000 L TNN
 F 2 "~" H 2650 2200 60  0000 C CNN
 F 3 "~" H 2650 2200 60  0000 C CNN
@@
 P 2650 2750
 F 0 "U?" H 2650 2850 50  0000 L BNN
-F 1 "74LS125" H 2700 2600 40  0000 L TNN
+F 1 "74ALVC125" H 2700 2600 40  0000 L TNN
 F 2 "~" H 2650 2750 60  0000 C CNN
 F 3 "~" H 2650 2750 60  0000 C CNN

Commit message: Added decoupling caps to the codec
Parts:
- added C? (x2): 0.1uF, ~, symbol C
- added C? (x2): 10uF, ~, symbol CP1
Connections:
- wire segments 83 -> 95

Commit message: Added headphone jack for codec
Parts:
- added HP?: HP_JACK, symbol HP_JACK
Connections:
- net labels removed: AUD_LEFT_OUT, AUD_RIGHT_OUT
- wire segments 95 -> 99
Changed lines of the file:
@@
 Text GLabel 1850 2200 0    60   Input ~ 0
 AUD_DAC_CL
-Text GLabel 3250 3900 0    60   Input ~ 0
-AUD_LEFT_OUT
-Text GLabel 3250 4150 0    60   Input ~ 0
-AUD_RIGHT_OUT
 $Comp
 L CP C?
@@
 	4450 4150 4350 4150
 Wire Wire Line
-	3950 3900 3250 3900
-Wire Wire Line
-	3950 4150 3250 4150
+	2850 3900 3950 3900
+Wire Wire Line
+	3100 4150 3950 4150
 Wire Wire Line
 	3350 4250 3350 4150
@@
 	3350 4750 3350 4850
 Wire Wire Line
-	3350 4850 3500 4850
+	3000 4850 3500 4850
 Connection ~ 3500 4850
 Wire Wire Line
@@
 Wire Wire Line
 	4550 1600 4550 2700
+$Comp
+L HP_JACK HP?
+U 1 1 5472A284
+P 2500 3900
+F 0 "HP?" H 2500 4100 60  0000 C CNN
+F 1 "HP_JACK" H 2500 3700 60  0000 C CNN
+F 2 "" H 2500 4100 60  0000 C CNN
+F 3 "" H 2500 4100 60  0000 C CNN
+	1    2500 3900
+	-1   0    0    1
+$EndComp
+Wire Wire Line
+	3100 4150 3100 4050
+Wire Wire Line
+	3100 4050 2850 4050
+Wire Wire Line
+	2850 3800 3000 3800
+Wire Wire Line
+	3000 3800 3000 4850
+Connection ~ 3350 4850
 $EndSCHEMATC

Commit message: Added net names, fixed misnamed GLCD_A0
Parts:
- gave numbers to parts that had none: 25
Changed lines of the file:
@@
 $EndDescr
 $Comp
-L WM8731 AC?
+L WM8731 AC1
 U 1 1 5468180C
 P 5650 3600
-F 0 "AC?" H 5650 3550 60  0000 C CNN
+F 0 "AC1" H 5650 3550 60  0000 C CNN
 F 1 "WM8731" H 5650 3650 60  0000 C CNN
 F 2 "~" H 5650 3650 60  0000 C CNN
@@
 $EndComp
 $Comp
-L GND #PWR?
+L GND #PWR052
 U 1 1 54681825
 P 6800 5550
-F 0 "#PWR?" H 6800 5550 30  0001 C CNN
+F 0 "#PWR052" H 6800 5550 30  0001 C CNN
 F 1 "GND" H 6800 5480 30  0001 C CNN
 F 2 "" H 6800 5550 60  0000 C CNN
@@
 $EndComp
 $Comp
-L GND #PWR?
+L GND #PWR053
 U 1 1 54681A6E
 P 4550 5050
-F 0 "#PWR?" H 4550 5050 30  0001 C CNN
+F 0 "#PWR053" H 4550 5050 30  0001 C CNN
 F 1 "GND" H 4550 4980 30  0001 C CNN
 F 2 "" H 4550 5050 60  0000 C CNN
@@
 $EndComp
 $Comp
-L 3V3 #PWR?
+L 3V3 #PWR054
 U 1 1 54681A95
 P 4550 1600
-F 0 "#PWR?" H 4550 1700 40  0001 C CNN
+F 0 "#PWR054" H 4550 1700 40  0001 C CNN
 F 1 "3V3" H 4550 1725 40  0000 C CNN
 F 2 "" H 4550 1600 60  0000 C CNN
@@
 $EndComp
 $Comp
-L 3V3 #PWR?
+L 3V3 #PWR055
 U 1 1 54681AB8
 P 7000 1600
-F 0 "#PWR?" H 7000 1700 40  0001 C CNN
+F 0 "#PWR055" H 7000 1700 40  0001 C CNN
 F 1 "3V3" H 7000 1725 40  0000 C CNN
 F 2 "" H 7000 1600 60  0000 C CNN
@@
 $EndComp
 $Comp
-L 3V3 #PWR?
+L 3V3 #PWR056
 U 1 1 54681AD9
 P 3750 4550
-F 0 "#PWR?" H 3750 4650 40  0001 C CNN
+F 0 "#PWR056" H 3750 4650 40  0001 C CNN
 F 1 "3V3" H 3750 4675 40  0000 C CNN
 F 2 "" H 3750 4550 60  0000 C CNN
@@
 $EndComp
 $Comp
-L INDUCTOR L?
+L INDUCTOR L1
 U 1 1 54681B0F
 P 4150 4650
-F 0 "L?" V 4100 4650 40  0000 C CNN
+F 0 "L1" V 4100 4650 40  0000 C CNN
 F 1 "10uH" V 4250 4650 40  0000 C CNN
 F 2 "~" H 4150 4650 60  0000 C CNN
@@
 $EndComp
 $Comp
-L CP C?
+L CP C22
 U 1 1 54681BAE
 P 7050 4700
-F 0 "C?" H 7100 4800 40  0000 L CNN
+F 0 "C22" H 7100 4800 40  0000 L CNN
 F 1 "10uF" H 7100 4600 40  0000 L CNN
 F 2 "~" H 7150 4550 30  0000 C CNN
@@
 $EndComp
 $Comp
-L CRYSTAL X?
+L CRYSTAL X2
 U 1 1 54681C53
 P 7750 2850
-F 0 "X?" H 7750 3000 60  0000 C CNN
+F 0 "X2" H 7750 3000 60  0000 C CNN
 F 1 "12.288MHz" H 7750 2700 60  0000 C CNN
 F 2 "~" H 7750 2850 60  0000 C CNN
@@
 $EndComp
 $Comp
-L GND #PWR?
+L GND #PWR057
 U 1 1 54681CB6
 P 8750 2900
-F 0 "#PWR?" H 8750 2900 30  0001 C CNN
+F 0 "#PWR057" H 8750 2900 30  0001 C CNN
 F 1 "GND" H 8750 2830 30  0001 C CNN
 F 2 "" H 8750 2900 60  0000 C CNN
@@
 $EndComp
 $Comp
-L C C?
+L C C25
 U 1 1 54681CD4
 P 8400 2600
-F 0 "C?" H 8400 2700 40  0000 L CNN
+F 0 "C25" H 8400 2700 40  0000 L CNN
 F 1 "22pF" H 8406 2515 40  0000 L CNN
 F 2 "~" H 8438 2450 30  0000 C CNN
@@
 $EndComp
 $Comp
-L C C?
+L C C26
 U 1 1 54681CFC
 P 8400 3100
-F 0 "C?" H 8400 3200 40  0000 L CNN
+F 0 "C26" H 8400 3200 40  0000 L CNN
 F 1 "22pF" H 8406 3015 40  0000 L CNN
 F 2 "~" H 8438 2950 30  0000 C CNN
@@
 I2C_DA
 $Comp
-L R R?
+L R R21
 U 1 1 546A770D
 P 4350 3000
-F 0 "R?" V 4430 3000 40  0000 C CNN
+F 0 "R21" V 4430 3000 40  0000 C CNN
 F 1 "27" V 4357 3001 40  0000 C CNN
 F 2 "~" V 4280 3000 30  0000 C CNN
@@
 SPI_SCK
 $Comp
-L R R?
+L R R22
 U 1 1 546A776A
 P 4350 3150
-F 0 "R?" V 4430 3150 40  0000 C CNN
+F 0 "R22" V 4430 3150 40  0000 C CNN
 F 1 "1K" V 4357 3151 40  0000 C CNN
 F 2 "~" V 4280 3150 30  0000 C CNN
@@
 $EndComp
 $Comp
-L R R?
+L R R23
 U 1 1 546A7770
 P 4350 3450
-F 0 "R?" V 4430 3450 40  0000 C CNN
+F 0 "R23" V 4430 3450 40  0000 C CNN
 F 1 "27" V 4357 3451 40  0000 C CNN
 F 2 "~" V 4280 3450 30  0000 C CNN
@@
 AUD_DAC_CL
 $Comp
-L CP C?
+L CP C16
 U 1 1 546A78E2
 P 4150 3900
-F 0 "C?" H 4200 4000 40  0000 L CNN
+F 0 "C16" H 4200 4000 40  0000 L CNN
 F 1 "330uF" H 4200 3800 40  0000 L CNN
 F 2 "~" H 4250 3750 30  0000 C CNN
@@
 $EndComp
 $Comp
-L CP C?
+L CP C17
 U 1 1 546A78FF
 P 4150 4150
-F 0 "C?" H 4200 4250 40  0000 L CNN
+F 0 "C17" H 4200 4250 40  0000 L CNN
 F 1 "330uF" H 4200 4050 40  0000 L CNN
 F 2 "~" H 4250 4000 30  0000 C CNN
@@
 $EndComp
 $Comp
-L R R?
+L R R20
 U 1 1 546A79D0
 P 3500 4500
-F 0 "R?" V 3580 4500 40  0000 C CNN
+F 0 "R20" V 3580 4500 40  0000 C CNN
 F 1 "47K" V 3507 4501 40  0000 C CNN
 F 2 "~" V 3430 4500 30  0000 C CNN
@@
 $EndComp
 $Comp
-L R R?
+L R R19
 U 1 1 546A79D6
 P 3350 4500
-F 0 "R?" V 3430 4500 40  0000 C CNN
+F 0 "R19" V 3430 4500 40  0000 C CNN
 F 1 "47K" V 3357 4501 40  0000 C CNN
 F 2 "~" V 3280 4500 30  0000 C CNN
@@
 $EndComp
 $Comp
-L GND #PWR?
+L GND #PWR058
 U 1 1 546A7A54
 P 3500 4950
-F 0 "#PWR?" H 3500 4950 30  0001 C CNN
+F 0 "#PWR058" H 3500 4950 30  0001 C CNN
 F 1 "GND" H 3500 4880 30  0001 C CNN
 F 2 "" H 3500 4950 60  0000 C CNN
@@
 NoConn ~ 6550 4050
 $Comp
-L R R?
+L R R24
 U 1 1 546A7AD0
 P 7150 4200
-F 0 "R?" V 7230 4200 40  0000 C CNN
+F 0 "R24" V 7230 4200 40  0000 C CNN
 F 1 "330" V 7157 4201 40  0000 C CNN
 F 2 "~" V 7080 4200 30  0000 C CNN
@@
 $EndComp
 $Comp
-L C C?
+L C C24
 U 1 1 546A7AD6
 P 7800 4200
-F 0 "C?" H 7800 4300 40  0000 L CNN
+F 0 "C24" H 7800 4300 40  0000 L CNN
 F 1 "1nF" H 7806 4115 40  0000 L CNN
 F 2 "~" H 7838 4050 30  0000 C CNN
@@
 $EndComp
 $Comp
-L R R?
+L R R26
 U 1 1 546A7B29
 P 8150 4650
-F 0 "R?" V 8230 4650 40  0000 C CNN
+F 0 "R26" V 8230 4650 40  0000 C CNN
 F 1 "47K" V 8157 4651 40  0000 C CNN
 F 2 "~" V 8080 4650 30  0000 C CNN
@@
 $EndComp
 $Comp
-L R R?
+L R R25
 U 1 1 546A7B34
 P 7700 4650
-F 0 "R?" V 7780 4650 40  0000 C CNN
+F 0 "R25" V 7780 4650 40  0000 C CNN
 F 1 "680" V 7707 4651 40  0000 C CNN
 F 2 "~" V 7630 4650 30  0000 C CNN
@@
 $EndComp
 $Comp
-L C C?
+L C C23
 U 1 1 546A7C11
 P 7700 5200
-F 0 "C?" H 7700 5300 40  0000 L CNN
+F 0 "C23" H 7700 5300 40  0000 L CNN
 F 1 "1nF" H 7706 5115 40  0000 L CNN
 F 2 "~" H 7738 5050 30  0000 C CNN
@@
 $EndComp
 $Comp
-L 74LS125 U?
+L 74LS125 U2
 U 1 1 546AB3AA
 P 2650 1100
-F 0 "U?" H 2650 1200 50  0000 L BNN
+F 0 "U2" H 2650 1200 50  0000 L BNN
 F 1 "74ALVC125" H 2700 950 40  0000 L TNN
 F 2 "~" H 2650 1100 60  0000 C CNN
@@
 $EndComp
 $Comp
-L 74LS125 U?
-U 1 1 546AB3B7
+L 74LS125 U2
+U 2 1 546AB3B7
 P 2650 1650
-F 0 "U?" H 2650 1750 50  0000 L BNN
+F 0 "U2" H 2650 1750 50  0000 L BNN
 F 1 "74ALVC125" H 2700 1500 40  0000 L TNN
 F 2 "~" H 2650 1650 60  0000 C CNN
 F 3 "~" H 2650 1650 60  0000 C CNN
-	1    2650 1650
-	1    0    0    -1
-$EndComp
-$Comp
-L 74LS125 U?
-U 1 1 546AB3BD
+	2    2650 1650
+	1    0    0    -1
+$EndComp
+$Comp
+L 74LS125 U2
+U 3 1 546AB3BD
 P 2650 2200
-F 0 "U?" H 2650 2300 50  0000 L BNN
+F 0 "U2" H 2650 2300 50  0000 L BNN
 F 1 "74ALVC125" H 2700 2050 40  0000 L TNN
 F 2 "~" H 2650 2200 60  0000 C CNN
 F 3 "~" H 2650 2200 60  0000 C CNN
-	1    2650 2200
-	1    0    0    -1
-$EndComp
-$Comp
-L 74LS125 U?
-U 1 1 546AB3C3
+	3    2650 2200
+	1    0    0    -1
+$EndComp
+$Comp
+L 74LS125 U2
+U 4 1 546AB3C3
 P 2650 2750
-F 0 "U?" H 2650 2850 50  0000 L BNN
+F 0 "U2" H 2650 2850 50  0000 L BNN
 F 1 "74ALVC125" H 2700 2600 40  0000 L TNN
 F 2 "~" H 2650 2750 60  0000 C CNN
 F 3 "~" H 2650 2750 60  0000 C CNN
-	1    2650 2750
+	4    2650 2750
 	-1   0    0    -1
 $EndComp
@@
 NoConn ~ 4750 4350
 $Comp
-L CMA-4544PF-W MIC?
+L CMA-4544PF-W MIC1
 U 1 1 546AC917
 P 8700 4800
-F 0 "MIC?" H 8700 4550 60  0000 C CNN
+F 0 "MIC1" H 8700 4550 60  0000 C CNN
 F 1 "CMA-4544PF-W" H 8650 5050 60  0001 C CNN
 F 2 "" H 8650 5050 60  0000 C CNN
@@
 $EndComp
 $Comp
-L C C?
+L C C20
 U 1 1 547292FF
 P 6300 2050
-F 0 "C?" H 6300 2150 40  0000 L CNN
+F 0 "C20" H 6300 2150 40  0000 L CNN
 F 1 "0.1uF" H 6306 1965 40  0000 L CNN
 F 2 "~" H 6338 1900 30  0000 C CNN
@@
 $EndComp
 $Comp
-L CP1 C?
+L CP1 C21
 U 1 1 5472930E
 P 6600 2050
-F 0 "C?" H 6650 2150 50  0000 L CNN
+F 0 "C21" H 6650 2150 50  0000 L CNN
 F 1 "10uF" H 6650 1950 50  0000 L CNN
 F 2 "~" H 6600 2050 60  0000 C CNN
@@
 $EndComp
 $Comp
-L C C?
+L C C18
 U 1 1 5472976A
 P 5350 2050
-F 0 "C?" H 5350 2150 40  0000 L CNN
+F 0 "C18" H 5350 2150 40  0000 L CNN
 F 1 "0.1uF" H 5356 1965 40  0000 L CNN
 F 2 "~" H 5388 1900 30  0000 C CNN
@@
 $EndComp
 $Comp
-L CP1 C?
+L CP1 C19
 U 1 1 54729770
 P 5650 2050
-F 0 "C?" H 5700 2150 50  0000 L CNN
+F 0 "C19" H 5700 2150 50  0000 L CNN
 F 1 "10uF" H 5700 1950 50  0000 L CNN
 F 2 "~" H 5650 2050 60  0000 C CNN
@@
 	4550 1600 4550 2700
 $Comp
-L HP_JACK HP?
+L HP_JACK HP1
 U 1 1 5472A284
 P 2500 3900
-F 0 "HP?" H 2500 4100 60  0000 C CNN
+F 0 "HP1" H 2500 4100 60  0000 C CNN
 F 1 "HP_JACK" H 2500 3700 60  0000 C CNN
 F 2 "" H 2500 4100 60  0000 C CNN
