File: board/mainboard/SPI_peripherals.sch (KiCad schematic (older format))
At the start: 7 parts

Commit message: Added schematic for DAC
Parts:
- added DAC?: MCP4902-E/SL, SO14, symbol MCP4902-E/SL
- added P?: CONN_2, symbol CONN_2
Connections:
- net labels added: SPI_CS2, ~RST
- wire segments 26 -> 50
Changed lines of the file:
@@
 Sheet 3 3
 Title ""
-Date "23 oct 2014"
+Date "1 nov 2014"
 Rev ""
 Comp ""
@@
 	1    0    0    -1
 $EndComp
-Wire Wire Line
-	1250 950  1250 850
-Wire Wire Line
-	1500 850  1500 950
-Wire Wire Line
-	1750 850  1750 950
-Connection ~ 1500 850
-Wire Wire Line
-	2000 850  2000 950
-Connection ~ 1750 850
-Wire Wire Line
-	2250 850  2250 950
-Connection ~ 2000 850
 $Comp
 L GND #PWR?
@@
 	1    0    0    -1
 $EndComp
-Wire Wire Line
-	1100 850  2450 850
-Wire Wire Line
-	2450 700  2450 2500
-Connection ~ 2250 850
-Wire Wire Line
-	2450 2500 2550 2500
-Connection ~ 2450 850
-Wire Wire Line
-	2450 2800 2550 2800
-Wire Wire Line
-	2450 2800 2450 4150
-Wire Wire Line
-	1250 1450 1250 3100
-Wire Wire Line
-	1250 3100 2550 3100
-Wire Wire Line
-	1500 1450 1500 2950
-Wire Wire Line
-	1000 2950 2550 2950
-Wire Wire Line
-	1750 1450 1750 2350
-Wire Wire Line
-	1000 2350 2550 2350
-Wire Wire Line
-	2000 1450 2000 2200
-Wire Wire Line
-	1000 2200 2550 2200
-Wire Wire Line
-	2550 2050 2250 2050
-Wire Wire Line
-	2250 2050 2250 1450
 Text GLabel 1000 2200 0    60   Input ~ 0
 SPI_CS1
-Connection ~ 2000 2200
 Text GLabel 1000 2650 0    60   Input ~ 0
 SPI_SCK
-Wire Wire Line
-	2550 2650 1000 2650
 Text GLabel 1000 2350 0    60   Input ~ 0
 SPI_MOSI
-Connection ~ 1750 2350
 Text GLabel 1000 2950 0    60   Input ~ 0
 SPI_MISO
-Connection ~ 1500 2950
-Wire Wire Line
-	2550 3250 1100 3250
-Wire Wire Line
-	1100 3250 1100 850
-Connection ~ 1250 850
 Text GLabel 1900 3400 0    60   Input ~ 0
 SD_SWITCH
@@
 	1    0    0    -1
 $EndComp
+Text GLabel 6950 1700 0    60   Input ~ 0
+SPI_CS2
+Text GLabel 6950 1550 0    60   Input ~ 0
+SPI_SCK
+Text GLabel 6950 1400 0    60   Input ~ 0
+SPI_MOSI
+$Comp
+L MCP4902-E/SL DAC?
+U 1 1 54555CC0
+P 8250 1650
+F 0 "DAC?" H 8400 2050 40  0000 L BNN
+F 1 "MCP4902-E/SL" H 8400 2000 40  0000 L BNN
+F 2 "SO14" H 8250 1650 30  0000 C CIN
+F 3 "" H 8250 1650 60  0000 C CNN
+	1    8250 1650
+	1    0    0    -1
+$EndComp
+$Comp
+L CONN_2 P?
+U 1 1 54555DA8
+P 9300 1650
+F 0 "P?" V 9250 1650 40  0000 C CNN
+F 1 "CONN_2" V 9350 1650 40  0000 C CNN
+F 2 "" H 9300 1650 60  0000 C CNN
+F 3 "" H 9300 1650 60  0000 C CNN
+	1    9300 1650
+	1    0    0    -1
+$EndComp
+$Comp
+L 3V3 #PWR?
+U 1 1 54555E65
+P 8150 900
+F 0 "#PWR?" H 8150 1000 40  0001 C CNN
+F 1 "3V3" H 8150 1025 40  0000 C CNN
+F 2 "" H 8150 900 60  0000 C CNN
+F 3 "" H 8150 900 60  0000 C CNN
+	1    8150 900
+	1    0    0    -1
+$EndComp
+$Comp
+L GND #PWR?
+U 1 1 54555F87
+P 8150 2400
+F 0 "#PWR?" H 8150 2400 30  0001 C CNN
+F 1 "GND" H 8150 2330 30  0001 C CNN
+F 2 "" H 8150 2400 60  0000 C CNN
+F 3 "" H 8150 2400 60  0000 C CNN
+	1    8150 2400
+	1    0    0    -1
+$EndComp
+Wire Wire Line
+	1250 950  1250 850
+Wire Wire Line
+	1500 850  1500 950
+Wire Wire Line
+	1750 850  1750 950
+Connection ~ 1500 850
+Wire Wire Line
+	2000 850  2000 950
+Connection ~ 1750 850
+Wire Wire Line
+	2250 850  2250 950
+Connection ~ 2000 850
+Wire Wire Line
+	1100 850  2450 850
+Wire Wire Line
+	2450 700  2450 2500
+Connection ~ 2250 850
+Wire Wire Line
+	2450 2500 2550 2500
+Connection ~ 2450 850
+Wire Wire Line
+	2450 2800 2550 2800
+Wire Wire Line
+	2450 2800 2450 4150
+Wire Wire Line
+	1250 1450 1250 3100
+Wire Wire Line
+	1250 3100 2550 3100
+Wire Wire Line
+	1500 1450 1500 2950
+Wire Wire Line
+	1000 2950 2550 2950
+Wire Wire Line
+	1750 1450 1750 2350
+Wire Wire Line
+	1000 2350 2550 2350
+Wire Wire Line
+	2000 1450 2000 2200
+Wire Wire Line
+	1000 2200 2550 2200
+Wire Wire Line
+	2550 2050 2250 2050
+Wire Wire Line
+	2250 2050 2250 1450
+Connection ~ 2000 2200
+Wire Wire Line
+	2550 2650 1000 2650
+Connection ~ 1750 2350
+Connection ~ 1500 2950
+Wire Wire Line
+	2550 3250 1100 3250
+Wire Wire Line
+	1100 3250 1100 850
+Connection ~ 1250 850
 Wire Wire Line
 	2250 4000 2450 4000
@@
 	1900 3400 2550 3400
 Connection ~ 2250 3400
+Wire Wire Line
+	7700 1550 6950 1550
+Wire Wire Line
+	8800 1800 8850 1800
+Wire Wire Line
+	8850 1800 8850 1750
+Wire Wire Line
+	8800 1500 8850 1500
+Wire Wire Line
+	8850 1500 8850 1550
+Wire Wire Line
+	8300 2100 8300 2150
+Wire Wire Line
+	8150 1000 9500 1000
+Wire Wire Line
+	8300 1000 8300 1200
+Wire Wire Line
+	8150 1200 8150 900
+Connection ~ 8150 1000
+Connection ~ 8300 1000
+Wire Wire Line
+	8850 1550 8950 1550
+Wire Wire Line
+	8850 1750 8950 1750
+Wire Wire Line
+	9500 1000 9500 2150
+Wire Wire Line
+	8150 2100 8150 2400
+Wire Wire Line
+	7700 1750 7600 1750
+Wire Wire Line
+	7600 1750 7600 2200
+Wire Wire Line
+	7600 2200 8150 2200
+Connection ~ 8150 2200
+Wire Wire Line
+	6950 1700 7100 1700
+Wire Wire Line
+	7100 1700 7100 1650
+Wire Wire Line
+	7100 1650 7700 1650
+Wire Wire Line
+	6950 1400 7100 1400
+Wire Wire Line
+	7100 1400 7100 1450
+Wire Wire Line
+	7100 1450 7700 1450
+Wire Wire Line
+	9500 2150 8300 2150
+Text GLabel 6950 1850 0    60   Input ~ 0
+~RST
+Wire Wire Line
+	6950 1850 7700 1850
 $EndSCHEMATC

Commit message: Changed pull-down on SD card to 10k
Parts:
- R?: value 50k -> 10k
Changed lines of the file:
@@
 Sheet 3 3
 Title ""
-Date "1 nov 2014"
+Date "11 nov 2014"
 Rev ""
 Comp ""
@@
 P 2250 3750
 F 0 "R?" V 2330 3750 40  0000 C CNN
-F 1 "50k" V 2257 3751 40  0000 C CNN
+F 1 "10k" V 2257 3751 40  0000 C CNN
 F 2 "~" V 2180 3750 30  0000 C CNN
 F 3 "~" H 2250 3750 30  0000 C CNN

Commit message: Added GLCD to schematic
Parts:
- added C? (x8): 1uF, ~, symbol C
- added GLCD?: NHD-C12832A1Z-NSW-BBW-3V3, ~, symbol NHD-C12832A1Z-NSW-BBW-3V3
Connections:
- net labels added: GLCD_A0, RST, SPI_CS3
- net labels removed: ~RST
- wire segments 50 -> 74

Commit message: Swapped DAC to one in mainboard library
Parts:
- removed DAC?: MCP4902-E/SL, SO14, symbol MCP4902-E/SL
- added DAC?: MCP4902, SO14, symbol MCP4902
Other:
- note added: "DAC"
- note added: "Graphic LCD"
- note added: "SD Card"
Changed lines of the file:
@@
 Sheet 3 3
 Title ""
-Date "11 nov 2014"
+Date "15 nov 2014"
 Rev ""
 Comp ""
@@
 SPI_MOSI
 $Comp
-L MCP4902-E/SL DAC?
-U 1 1 54555CC0
-P 8700 1850
-F 0 "DAC?" H 8850 2250 40  0000 L BNN
-F 1 "MCP4902-E/SL" H 8850 2200 40  0000 L BNN
-F 2 "SO14" H 8700 1850 30  0000 C CIN
-F 3 "" H 8700 1850 60  0000 C CNN
-	1    8700 1850
-	1    0    0    -1
-$EndComp
-$Comp
 L CONN_2 P?
 U 1 1 54555DA8
@@
 Wire Wire Line
 	7050 3600 7050 3800
+Text Notes 3200 1700 0    60   ~ 0
+SD Card
+Text Notes 8150 1350 0    60   ~ 0
+DAC
+Text Notes 8050 3350 0    60   ~ 0
+Graphic LCD
+$Comp
+L MCP4902 DAC?
+U 1 1 5467E291
+P 8700 1850
+F 0 "DAC?" H 8850 2250 40  0000 L BNN
+F 1 "MCP4902" H 8850 2200 40  0000 L BNN
+F 2 "SO14" H 8700 1850 30  0000 C CIN
+F 3 "" H 8700 1850 60  0000 C CNN
+	1    8700 1850
+	1    0    0    -1
+$EndComp
 $EndSCHEMATC

Commit message: Added SPI CS decoder
Parts:
- added D? (x3): DIODESCH, ~, symbol DIODESCH
- added R?: 47k, ~, symbol R
- added U?: 74LS138, ~, symbol 74LS138
Connections:
- net labels added: SPI_CS4, SPI_CS5, SPI_CS6, SPI_CS7, SPI_SEL0, SPI_SEL1, SPI_SEL2
- wire segments 74 -> 102
- no-connect marks 0 -> 1
Changed lines of the file:
@@
 $Descr A4 11693 8268
 encoding utf-8
-Sheet 3 3
+Sheet 3 5
 Title ""
-Date "15 nov 2014"
+Date "18 nov 2014"
 Rev ""
 Comp ""
@@
 	1    0    0    -1
 $EndComp
+$Comp
+L 74LS138 U?
+U 1 1 546AA00B
+P 2800 5800
+F 0 "U?" H 2900 6300 60  0000 C CNN
+F 1 "74LS138" H 2950 5251 60  0000 C CNN
+F 2 "~" H 2800 5800 60  0000 C CNN
+F 3 "~" H 2800 5800 60  0000 C CNN
+	1    2800 5800
+	1    0    0    -1
+$EndComp
+Text GLabel 1200 5400 0    60   Input ~ 0
+SPI_SEL0
+Text GLabel 1200 5550 0    60   Input ~ 0
+SPI_SEL1
+Text GLabel 1200 5700 0    60   Input ~ 0
+SPI_SEL2
+Wire Wire Line
+	1200 5550 2200 5550
+Wire Wire Line
+	1200 5400 2050 5400
+Wire Wire Line
+	2050 5400 2050 5450
+Wire Wire Line
+	2050 5450 2200 5450
+Wire Wire Line
+	1200 5700 2050 5700
+Wire Wire Line
+	2050 5700 2050 5650
+Wire Wire Line
+	2050 5650 2200 5650
+Text GLabel 3700 5550 2    60   Input ~ 0
+SPI_CS1
+Text GLabel 4150 5650 2    60   Input ~ 0
+SPI_CS2
+Text GLabel 3700 5750 2    60   Input ~ 0
+SPI_CS3
+Text GLabel 4150 5850 2    60   Input ~ 0
+SPI_CS4
+Text GLabel 3700 5950 2    60   Input ~ 0
+SPI_CS5
+Text GLabel 4150 6050 2    60   Input ~ 0
+SPI_CS6
+Text GLabel 3700 6150 2    60   Input ~ 0
+SPI_CS7
+Wire Wire Line
+	3400 5550 3700 5550
+Wire Wire Line
+	3400 5650 4150 5650
+Wire Wire Line
+	3400 5750 3700 5750
+Wire Wire Line
+	3400 5850 4150 5850
+Wire Wire Line
+	3400 5950 3700 5950
+Wire Wire Line
+	3400 6050 4150 6050
+Wire Wire Line
+	3400 6150 3700 6150
+$Comp
+L DIODESCH D?
+U 1 1 546AA578
+P 1600 5950
+F 0 "D?" H 1600 6050 40  0000 C CNN
+F 1 "DIODESCH" H 1600 5850 40  0000 C CNN
+F 2 "~" H 1600 5950 60  0000 C CNN
+F 3 "~" H 1600 5950 60  0000 C CNN
+	1    1600 5950
+	0    1    1    0
+$EndComp
+$Comp
+L DIODESCH D?
+U 1 1 546AA5F2
+P 1300 5950
+F 0 "D?" H 1300 6050 40  0000 C CNN
+F 1 "DIODESCH" H 1300 5850 40  0000 C CNN
+F 2 "~" H 1300 5950 60  0000 C CNN
+F 3 "~" H 1300 5950 60  0000 C CNN
+	1    1300 5950
+	0    1    1    0
+$EndComp
+Wire Wire Line
+	1300 5750 1300 5400
+Connection ~ 1300 5400
+Wire Wire Line
+	1600 5750 1600 5550
+Connection ~ 1600 5550
+$Comp
+L DIODESCH D?
+U 1 1 546AA823
+P 1900 5950
+F 0 "D?" H 1900 6050 40  0000 C CNN
+F 1 "DIODESCH" H 1900 5850 40  0000 C CNN
+F 2 "~" H 1900 5950 60  0000 C CNN
+F 3 "~" H 1900 5950 60  0000 C CNN
+	1    1900 5950
+	0    1    1    0
+$EndComp
+Wire Wire Line
+	1900 5750 1900 5700
+Connection ~ 1900 5700
+Wire Wire Line
+	1300 6150 1300 6200
+Wire Wire Line
+	1900 6200 1900 6150
+Wire Wire Line
+	1600 6150 1600 6300
+Connection ~ 1600 6200
+$Comp
+L GND #PWR?
+U 1 1 546AA98C
+P 1600 6900
+F 0 "#PWR?" H 1600 6900 30  0001 C CNN
+F 1 "GND" H 1600 6830 30  0001 C CNN
+F 2 "" H 1600 6900 60  0000 C CNN
+F 3 "" H 1600 6900 60  0000 C CNN
+	1    1600 6900
+	1    0    0    -1
+$EndComp
+$Comp
+L R R?
+U 1 1 546AA99B
+P 1600 6550
+F 0 "R?" V 1680 6550 40  0000 C CNN
+F 1 "47k" V 1607 6551 40  0000 C CNN
+F 2 "~" V 1530 6550 30  0000 C CNN
+F 3 "~" H 1600 6550 30  0000 C CNN
+	1    1600 6550
+	1    0    0    -1
+$EndComp
+Wire Wire Line
+	1600 6800 1600 6900
+Wire Wire Line
+	2050 6200 2050 5950
+Wire Wire Line
+	2050 5950 2200 5950
+Connection ~ 1900 6200
+Wire Wire Line
+	2200 6050 2150 6050
+Wire Wire Line
+	2150 6050 2150 6850
+Wire Wire Line
+	2150 6150 2200 6150
+Wire Wire Line
+	2150 6850 1600 6850
+Connection ~ 1600 6850
+Connection ~ 2150 6150
+Wire Wire Line
+	1300 6200 2050 6200
+NoConn ~ 3400 5450
 $EndSCHEMATC

Commit message: Swapped the diode OR gate on the 3-8 to pulldowns
Parts:
- removed D? (x3): DIODESCH, ~, symbol DIODESCH
- removed R?: 47k, ~, symbol R
- added R? (x4): 47k, ~, symbol R
Connections:
- wire segments 102 -> 101
Changed lines of the file:
@@
 Wire Wire Line
 	3400 6150 3700 6150
-$Comp
-L DIODESCH D?
-U 1 1 546AA578
-P 1600 5950
-F 0 "D?" H 1600 6050 40  0000 C CNN
-F 1 "DIODESCH" H 1600 5850 40  0000 C CNN
-F 2 "~" H 1600 5950 60  0000 C CNN
-F 3 "~" H 1600 5950 60  0000 C CNN
-	1    1600 5950
-	0    1    1    0
-$EndComp
-$Comp
-L DIODESCH D?
-U 1 1 546AA5F2
-P 1300 5950
-F 0 "D?" H 1300 6050 40  0000 C CNN
-F 1 "DIODESCH" H 1300 5850 40  0000 C CNN
-F 2 "~" H 1300 5950 60  0000 C CNN
-F 3 "~" H 1300 5950 60  0000 C CNN
-	1    1300 5950
-	0    1    1    0
-$EndComp
 Wire Wire Line
-	1300 5750 1300 5400
+	1300 5400 1300 6200
 Connection ~ 1300 5400
-Wire Wire Line
-	1600 5750 1600 5550
-Connection ~ 1600 5550
-$Comp
-L DIODESCH D?
-U 1 1 546AA823
-P 1900 5950
-F 0 "D?" H 1900 6050 40  0000 C CNN
-F 1 "DIODESCH" H 1900 5850 40  0000 C CNN
-F 2 "~" H 1900 5950 60  0000 C CNN
-F 3 "~" H 1900 5950 60  0000 C CNN
-	1    1900 5950
-	0    1    1    0
-$EndComp
-Wire Wire Line
-	1900 5750 1900 5700
-Connection ~ 1900 5700
-Wire Wire Line
-	1300 6150 1300 6200
-Wire Wire Line
-	1900 6200 1900 6150
-Wire Wire Line
-	1600 6150 1600 6300
-Connection ~ 1600 6200
-$Comp
-L GND #PWR?
-U 1 1 546AA98C
-P 1600 6900
-F 0 "#PWR?" H 1600 6900 30  0001 C CNN
-F 1 "GND" H 1600 6830 30  0001 C CNN
-F 2 "" H 1600 6900 60  0000 C CNN
-F 3 "" H 1600 6900 60  0000 C CNN
-	1    1600 6900
-	1    0    0    -1
-$EndComp
-$Comp
-L R R?
-U 1 1 546AA99B
-P 1600 6550
-F 0 "R?" V 1680 6550 40  0000 C CNN
-F 1 "47k" V 1607 6551 40  0000 C CNN
-F 2 "~" V 1530 6550 30  0000 C CNN
-F 3 "~" H 1600 6550 30  0000 C CNN
-	1    1600 6550
-	1    0    0    -1
-$EndComp
-Wire Wire Line
-	1600 6800 1600 6900
 Wire Wire Line
 	2050 6200 2050 5950
 Wire Wire Line
 	2050 5950 2200 5950
-Connection ~ 1900 6200
 Wire Wire Line
 	2200 6050 2150 6050
@@
 Wire Wire Line
 	2150 6150 2200 6150
+Connection ~ 2150 6150
+NoConn ~ 3400 5450
+$Comp
+L GND #PWR?
+U 1 1 546AB116
+P 2150 6850
+F 0 "#PWR?" H 2150 6850 30  0001 C CNN
+F 1 "GND" H 2150 6780 30  0001 C CNN
+F 2 "" H 2150 6850 60  0000 C CNN
+F 3 "" H 2150 6850 60  0000 C CNN
+	1    2150 6850
+	1    0    0    -1
+$EndComp
+$Comp
+L R R?
+U 1 1 546AB125
+P 2050 6450
+F 0 "R?" V 2130 6450 40  0000 C CNN
+F 1 "47k" V 2057 6451 40  0000 C CNN
+F 2 "~" V 1980 6450 30  0000 C CNN
+F 3 "~" H 2050 6450 30  0000 C CNN
+	1    2050 6450
+	1    0    0    -1
+$EndComp
+$Comp
+L R R?
+U 1 1 546AB137
+P 1800 6450
+F 0 "R?" V 1880 6450 40  0000 C CNN
+F 1 "47k" V 1807 6451 40  0000 C CNN
+F 2 "~" V 1730 6450 30  0000 C CNN
+F 3 "~" H 1800 6450 30  0000 C CNN
+	1    1800 6450
+	1    0    0    -1
+$EndComp
+$Comp
+L R R?
+U 1 1 546AB13D
+P 1550 6450
+F 0 "R?" V 1630 6450 40  0000 C CNN
+F 1 "47k" V 1557 6451 40  0000 C CNN
+F 2 "~" V 1480 6450 30  0000 C CNN
+F 3 "~" H 1550 6450 30  0000 C CNN
+	1    1550 6450
+	1    0    0    -1
+$EndComp
+$Comp
+L R R?
+U 1 1 546AB143
+P 1300 6450
+F 0 "R?" V 1380 6450 40  0000 C CNN
+F 1 "47k" V 1307 6451 40  0000 C CNN
+F 2 "~" V 1230 6450 30  0000 C CNN
+F 3 "~" H 1300 6450 30  0000 C CNN
+	1    1300 6450
+	1    0    0    -1
+$EndComp
 Wire Wire Line
-	2150 6850 1600 6850
-Connection ~ 1600 6850
-Connection ~ 2150 6150
+	1550 6200 1550 5550
+Connection ~ 1550 5550
 Wire Wire Line
-	1300 6200 2050 6200
-NoConn ~ 3400 5450
+	1800 6200 1800 5700
+Connection ~ 1800 5700
+Wire Wire Line
+	1300 6750 2150 6750
+Wire Wire Line
+	2050 6750 2050 6700
+Connection ~ 2150 6750
+Wire Wire Line
+	1800 6750 1800 6700
+Connection ~ 2050 6750
+Wire Wire Line
+	1550 6750 1550 6700
+Connection ~ 1800 6750
+Wire Wire Line
+	1300 6750 1300 6700
+Connection ~ 1550 6750
 $EndSCHEMATC

Commit message: Named some default named connectors, fixed incorrect pull down
Parts:
- removed R?: 47k, ~, symbol R
- P?: value CONN_2 -> DAC
Connections:
- wire segments 101 -> 99
Changed lines of the file:
@@
 P 9750 1850
 F 0 "P?" V 9700 1850 40  0000 C CNN
-F 1 "CONN_2" V 9800 1850 40  0000 C CNN
+F 1 "DAC" V 9800 1850 40  0000 C CNN
 F 2 "" H 9750 1850 60  0000 C CNN
 F 3 "" H 9750 1850 60  0000 C CNN
@@
 Connection ~ 1300 5400
 Wire Wire Line
-	2050 6200 2050 5950
-Wire Wire Line
 	2050 5950 2200 5950
 Wire Wire Line
@@
 $Comp
 L R R?
-U 1 1 546AB125
-P 2050 6450
-F 0 "R?" V 2130 6450 40  0000 C CNN
-F 1 "47k" V 2057 6451 40  0000 C CNN
-F 2 "~" V 1980 6450 30  0000 C CNN
-F 3 "~" H 2050 6450 30  0000 C CNN
-	1    2050 6450
-	1    0    0    -1
-$EndComp
-$Comp
-L R R?
 U 1 1 546AB137
 P 1800 6450
@@
 Wire Wire Line
 	1300 6750 2150 6750
-Wire Wire Line
-	2050 6750 2050 6700
 Connection ~ 2150 6750
 Wire Wire Line
 	1800 6750 1800 6700
-Connection ~ 2050 6750
 Wire Wire Line
 	1550 6750 1550 6700
@@
 	1300 6750 1300 6700
 Connection ~ 1550 6750
+$Comp
+L 3V3 #PWR?
+U 1 1 546ABAD8
+P 2050 5950
+F 0 "#PWR?" H 2050 6050 40  0001 C CNN
+F 1 "3V3" H 2050 6075 40  0000 C CNN
+F 2 "" H 2050 5950 60  0000 C CNN
+F 3 "" H 2050 5950 60  0000 C CNN
+	1    2050 5950
+	1    0    0    -1
+$EndComp
 $EndSCHEMATC
