File: board/mainboard/SPI_peripherals.sch (KiCad schematic (older format))
At the start: 26 parts

Commit message: Added net names, fixed misnamed GLCD_A0
Parts:
- gave numbers to parts that had none: 26
Changed lines of the file:
@@
 $EndDescr
 $Comp
-L SDCARD_PUSH SD?
+L SDCARD_PUSH SD1
 U 1 1 544877FA
 P 3450 2650
-F 0 "SD?" H 3450 2550 60  0000 C CNN
+F 0 "SD1" H 3450 2550 60  0000 C CNN
 F 1 "SDCARD_PUSH" H 3450 2750 60  0000 C CNN
 F 2 "~" H 3450 2750 60  0000 C CNN
@@
 $EndComp
 $Comp
-L R R?
+L R R15
 U 1 1 54487C3C
 P 5700 3550
-F 0 "R?" V 5780 3550 40  0000 C CNN
+F 0 "R15" V 5780 3550 40  0000 C CNN
 F 1 "50k" V 5707 3551 40  0000 C CNN
 F 2 "~" V 5630 3550 30  0000 C CNN
@@
 $EndComp
 $Comp
-L R R?
+L R R14
 U 1 1 54487C57
 P 5550 3550
-F 0 "R?" V 5630 3550 40  0000 C CNN
+F 0 "R14" V 5630 3550 40  0000 C CNN
 F 1 "50k" V 5557 3551 40  0000 C CNN
 F 2 "~" V 5480 3550 30  0000 C CNN
@@
 $EndComp
 $Comp
-L 3V3 #PWR?
+L 3V3 #PWR027
 U 1 1 54487C67
 P 2450 1200
-F 0 "#PWR?" H 2450 1300 40  0001 C CNN
+F 0 "#PWR027" H 2450 1300 40  0001 C CNN
 F 1 "3V3" H 2450 1325 40  0000 C CNN
 F 2 "" H 2450 1200 60  0000 C CNN
@@
 $EndComp
 $Comp
-L GND #PWR?
+L GND #PWR028
 U 1 1 54487D03
 P 2450 4150
-F 0 "#PWR?" H 2450 4150 30  0001 C CNN
+F 0 "#PWR028" H 2450 4150 30  0001 C CNN
 F 1 "GND" H 2450 4080 30  0001 C CNN
 F 2 "" H 2450 4150 60  0000 C CNN
@@
 SD_SWITCH
 $Comp
-L R R?
+L R R12
 U 1 1 544883FE
 P 2250 3750
-F 0 "R?" V 2330 3750 40  0000 C CNN
+F 0 "R12" V 2330 3750 40  0000 C CNN
 F 1 "10k" V 2257 3751 40  0000 C CNN
 F 2 "~" V 2180 3750 30  0000 C CNN
@@
 SPI_MOSI
 $Comp
-L CONN_2 P?
+L CONN_2 P5
 U 1 1 54555DA8
 P 9750 1850
-F 0 "P?" V 9700 1850 40  0000 C CNN
+F 0 "P5" V 9700 1850 40  0000 C CNN
 F 1 "DAC" V 9800 1850 40  0000 C CNN
 F 2 "" H 9750 1850 60  0000 C CNN
@@
 $EndComp
 $Comp
-L 3V3 #PWR?
+L 3V3 #PWR029
 U 1 1 54555E65
 P 8600 1100
-F 0 "#PWR?" H 8600 1200 40  0001 C CNN
+F 0 "#PWR029" H 8600 1200 40  0001 C CNN
 F 1 "3V3" H 8600 1225 40  0000 C CNN
 F 2 "" H 8600 1100 60  0000 C CNN
@@
 RST
 $Comp
-L NHD-C12832A1Z-NSW-BBW-3V3 GLCD?
+L NHD-C12832A1Z-NSW-BBW-3V3 GLCD1
 U 1 1 54618A74
 P 8300 3950
-F 0 "GLCD?" H 8300 3850 60  0000 C CNN
+F 0 "GLCD1" H 8300 3850 60  0000 C CNN
 F 1 "NHD-C12832A1Z-NSW-BBW-3V3" H 8300 4050 60  0000 C CNN
 F 2 "~" H 8300 4050 60  0000 C CNN
@@
 SPI_MOSI
 $Comp
-L 3V3 #PWR?
+L 3V3 #PWR030
 U 1 1 54618BA1
 P 8300 5150
-F 0 "#PWR?" H 8300 5250 40  0001 C CNN
+F 0 "#PWR030" H 8300 5250 40  0001 C CNN
 F 1 "3V3" H 8300 5275 40  0000 C CNN
 F 2 "" H 8300 5150 60  0000 C CNN
@@
 $EndComp
 $Comp
-L GND #PWR?
+L GND #PWR031
 U 1 1 54618BF4
 P 8450 5500
-F 0 "#PWR?" H 8450 5500 30  0001 C CNN
+F 0 "#PWR031" H 8450 5500 30  0001 C CNN
 F 1 "GND" H 8450 5430 30  0001 C CNN
 F 2 "" H 8450 5500 60  0000 C CNN
@@
 $EndComp
 $Comp
-L C C?
+L C C6
 U 1 1 54618DB7
 P 8600 5150
-F 0 "C?" H 8600 5250 40  0000 L CNN
+F 0 "C6" H 8600 5250 40  0000 L CNN
 F 1 "1uF" H 8606 5065 40  0000 L CNN
 F 2 "~" H 8638 5000 30  0000 C CNN
@@
 $EndComp
 $Comp
-L C C?
+L C C11
 U 1 1 54618A8D
 P 9950 3650
-F 0 "C?" H 9950 3750 40  0000 L CNN
+F 0 "C11" H 9950 3750 40  0000 L CNN
 F 1 "1uF" H 9956 3565 40  0000 L CNN
 F 2 "~" H 9988 3500 30  0000 C CNN
@@
 $EndComp
 $Comp
-L C C?
+L C C12
 U 1 1 5461A864
 P 9950 3800
-F 0 "C?" H 9950 3900 40  0000 L CNN
+F 0 "C12" H 9950 3900 40  0000 L CNN
 F 1 "1uF" H 9956 3715 40  0000 L CNN
 F 2 "~" H 9988 3650 30  0000 C CNN
@@
 $EndComp
 $Comp
-L C C?
+L C C13
 U 1 1 5461A86A
 P 9950 3950
-F 0 "C?" H 9950 4050 40  0000 L CNN
+F 0 "C13" H 9950 4050 40  0000 L CNN
 F 1 "1uF" H 9956 3865 40  0000 L CNN
 F 2 "~" H 9988 3800 30  0000 C CNN
@@
 $EndComp
 $Comp
-L C C?
+L C C14
 U 1 1 5461A870
 P 9950 4100
-F 0 "C?" H 9950 4200 40  0000 L CNN
+F 0 "C14" H 9950 4200 40  0000 L CNN
 F 1 "1uF" H 9956 4015 40  0000 L CNN
 F 2 "~" H 9988 3950 30  0000 C CNN
@@
 $EndComp
 $Comp
-L C C?
+L C C15
 U 1 1 5461A876
 P 9950 4250
-F 0 "C?" H 9950 4350 40  0000 L CNN
+F 0 "C15" H 9950 4350 40  0000 L CNN
 F 1 "1uF" H 9956 4165 40  0000 L CNN
 F 2 "~" H 9988 4100 30  0000 C CNN
@@
 $EndComp
 $Comp
-L C C?
+L C C7
 U 1 1 5461AB82
 P 8900 5150
-F 0 "C?" H 8900 5250 40  0000 L CNN
+F 0 "C7" H 8900 5250 40  0000 L CNN
 F 1 "1uF" H 8906 5065 40  0000 L CNN
 F 2 "~" H 8938 5000 30  0000 C CNN
@@
 $EndComp
 $Comp
-L C C?
+L C C10
 U 1 1 5461AB88
 P 9200 5150
-F 0 "C?" H 9200 5250 40  0000 L CNN
+F 0 "C10" H 9200 5250 40  0000 L CNN
 F 1 "1uF" H 9206 5065 40  0000 L CNN
 F 2 "~" H 9238 5000 30  0000 C CNN
@@
 GLCD_A0
 $Comp
-L GND #PWR?
+L GND #PWR032
 U 1 1 5461AE8D
 P 7050 4150
-F 0 "#PWR?" H 7050 4150 30  0001 C CNN
+F 0 "#PWR032" H 7050 4150 30  0001 C CNN
 F 1 "GND" H 7050 4080 30  0001 C CNN
 F 2 "" H 7050 4150 60  0000 C CNN
@@
 Graphic LCD
 $Comp
-L MCP4902 DAC?
+L MCP4902 DAC1
 U 1 1 5467E291
 P 8700 1850
-F 0 "DAC?" H 8850 2250 40  0000 L BNN
+F 0 "DAC1" H 8850 2250 40  0000 L BNN
 F 1 "MCP4902" H 8850 2200 40  0000 L BNN
 F 2 "SO14" H 8700 1850 30  0000 C CIN
@@
 $EndComp
 $Comp
-L 74LS138 U?
+L 74LS138 U1
 U 1 1 546AA00B
 P 2800 5800
-F 0 "U?" H 2900 6300 60  0000 C CNN
+F 0 "U1" H 2900 6300 60  0000 C CNN
 F 1 "74LS138" H 2950 5251 60  0000 C CNN
 F 2 "~" H 2800 5800 60  0000 C CNN
@@
 NoConn ~ 3400 5450
 $Comp
-L GND #PWR?
+L GND #PWR033
 U 1 1 546AB116
 P 2150 6850
-F 0 "#PWR?" H 2150 6850 30  0001 C CNN
+F 0 "#PWR033" H 2150 6850 30  0001 C CNN
 F 1 "GND" H 2150 6780 30  0001 C CNN
 F 2 "" H 2150 6850 60  0000 C CNN
@@
 $EndComp
 $Comp
-L R R?
+L R R9
 U 1 1 546AB137
 P 1800 6450
-F 0 "R?" V 1880 6450 40  0000 C CNN
+F 0 "R9" V 1880 6450 40  0000 C CNN
 F 1 "47k" V 1807 6451 40  0000 C CNN
 F 2 "~" V 1730 6450 30  0000 C CNN
@@
 $EndComp
 $Comp
-L R R?
+L R R8
 U 1 1 546AB13D
 P 1550 6450
-F 0 "R?" V 1630 6450 40  0000 C CNN
+F 0 "R8" V 1630 6450 40  0000 C CNN
 F 1 "47k" V 1557 6451 40  0000 C CNN
 F 2 "~" V 1480 6450 30  0000 C CNN
@@
 $EndComp
 $Comp
-L R R?
+L R R7
 U 1 1 546AB143
 P 1300 6450
-F 0 "R?" V 1380 6450 40  0000 C CNN
+F 0 "R7" V 1380 6450 40  0000 C CNN
 F 1 "47k" V 1307 6451 40  0000 C CNN
 F 2 "~" V 1230 6450 30  0000 C CNN
@@
 $EndComp
 $Comp
-L 3V3 #PWR?
+L 3V3 #PWR034
 U 1 1 546ABAD8
 P 2050 5950
-F 0 "#PWR?" H 2050 6050 40  0001 C CNN
+F 0 "#PWR034" H 2050 6050 40  0001 C CNN
 F 1 "3V3" H 2050 6075 40  0000 C CNN
 F 2 "" H 2050 5950 60  0000 C CNN
@@
 $EndComp
 $Comp
-L CONN_8 P?
+L CONN_8 P4
 U 1 1 54726C0B
 P 6200 4450
-F 0 "P?" V 6150 4450 60  0000 C CNN
+F 0 "P4" V 6150 4450 60  0000 C CNN
 F 1 "CONN_8" V 6250 4450 60  0000 C CNN
 F 2 "" H 6200 4450 60  0000 C CNN
@@
 $EndComp
 $Comp
-L GND #PWR?
+L GND #PWR035
 U 1 1 54726C24
 P 5700 5050
-F 0 "#PWR?" H 5700 5050 30  0001 C CNN
+F 0 "#PWR035" H 5700 5050 30  0001 C CNN
 F 1 "GND" H 5700 4980 30  0001 C CNN
 F 2 "" H 5700 5050 60  0000 C CNN
@@
 $EndComp
 $Comp
-L 3V3 #PWR?
+L 3V3 #PWR036
 U 1 1 54726D33
 P 5800 3100
-F 0 "#PWR?" H 5800 3200 40  0001 C CNN
+F 0 "#PWR036" H 5800 3200 40  0001 C CNN
 F 1 "3V3" H 5800 3225 40  0000 C CNN
 F 2 "" H 5800 3100 60  0000 C CNN
@@
 Connection ~ 5800 3200
 $Comp
-L R R?
+L R R13
 U 1 1 54487C51
 P 2450 1700
-F 0 "R?" V 2530 1700 40  0000 C CNN
+F 0 "R13" V 2530 1700 40  0000 C CNN
 F 1 "50k" V 2457 1701 40  0000 C CNN
 F 2 "~" V 2380 1700 30  0000 C CNN
@@
 $EndComp
 $Comp
-L R R?
+L R R11
 U 1 1 54487C5D
 P 2150 1700
-F 0 "R?" V 2230 1700 40  0000 C CNN
+F 0 "R11" V 2230 1700 40  0000 C CNN
 F 1 "50k" V 2157 1701 40  0000 C CNN
 F 2 "~" V 2080 1700 30  0000 C CNN
@@
 Connection ~ 2150 1300
 $Comp
-L CONN_2 J?
+L CONN_2 J1
 U 1 1 54728756
 P 6700 3350
-F 0 "J?" V 6650 3350 40  0000 C CNN
+F 0 "J1" V 6650 3350 40  0000 C CNN
 F 1 "BACKL" V 6750 3350 40  0000 C CNN
 F 2 "" H 6700 3350 60  0000 C CNN
@@
 	7050 3800 7050 3450
 $Comp
-L 3V3 #PWR?
+L 3V3 #PWR037
 U 1 1 54728806
 P 7050 2900
-F 0 "#PWR?" H 7050 3000 40  0001 C CNN
+F 0 "#PWR037" H 7050 3000 40  0001 C CNN
 F 1 "3V3" H 7050 3025 40  0000 C CNN
 F 2 "" H 7050 2900 60  0000 C CNN
@@
 	7050 3250 7050 2900
 $Comp
-L C C?
+L C C8
 U 1 1 54728B01
 P 9200 2550
-F 0 "C?" H 9200 2650 40  0000 L CNN
+F 0 "C8" H 9200 2650 40  0000 L CNN
 F 1 "0.1uF" H 9206 2465 40  0000 L CNN
 F 2 "~" H 9238 2400 30  0000 C CNN
@@
 Connection ~ 9500 2350
 $Comp
-L CP1 C?
+L CP1 C9
 U 1 1 54728C3B
 P 9200 2800
-F 0 "C?" H 9250 2900 50  0000 L CNN
+F 0 "C9" H 9250 2900 50  0000 L CNN
 F 1 "10uF" H 9250 2700 50  0000 L CNN
 F 2 "~" H 9200 2800 60  0000 C CNN
@@
 	1650 2950 2550 2950
 $Comp
-L R R?
+L R R10
 U 1 1 5472863C
 P 1850 1700
-F 0 "R?" V 1930 1700 40  0000 C CNN
+F 0 "R10" V 1930 1700 40  0000 C CNN
 F 1 "50k" V 1857 1701 40  0000 C CNN
 F 2 "~" V 1780 1700 30  0000 C CNN
@@
 Connection ~ 8600 2550
 $Comp
-L GND #PWR?
+L GND #PWR038
 U 1 1 54729C52
 P 8600 2900
-F 0 "#PWR?" H 8600 2900 30  0001 C CNN
+F 0 "#PWR038" H 8600 2900 30  0001 C CNN
 F 1 "GND" H 8600 2830 30  0001 C CNN
 F 2 "" H 8600 2900 60  0000 C CNN

Commit message: Fixed double use of SPI_CS4
Parts:
- removed P4: CONN_8, symbol CONN_8
- added P?: CONN_7, symbol CONN_7
Connections:
- wire segments 127 -> 124
Changed lines of the file:
@@
-$EndComp
-$Comp
-L CONN_8 P4
-U 1 1 54726C0B
-P 6200 4450
-F 0 "P4" V 6150 4450 60  0000 C CNN
-F 1 "CONN_8" V 6250 4450 60  0000 C CNN
-F 2 "" H 6200 4450 60  0000 C CNN
-F 3 "" H 6200 4450 60  0000 C CNN
-	1    6200 4450
-	1    0    0    -1
 $EndComp
 $Comp
 L GND #PWR035
 U 1 1 54726C24
-P 5700 5050
-F 0 "#PWR035" H 5700 5050 30  0001 C CNN
-F 1 "GND" H 5700 4980 30  0001 C CNN
-F 2 "" H 5700 5050 60  0000 C CNN
-F 3 "" H 5700 5050 60  0000 C CNN
-	1    5700 5050
+P 5700 4950
+F 0 "#PWR035" H 5700 4950 30  0001 C CNN
+F 1 "GND" H 5700 4880 30  0001 C CNN
+F 2 "" H 5700 4950 60  0000 C CNN
+F 3 "" H 5700 4950 60  0000 C CNN
+	1    5700 4950
 	1    0    0    -1
 $EndComp
@@
 	1    0    0    -1
 $EndComp
-Text GLabel 5300 3950 0    60   Input ~ 0
+Text GLabel 5300 4000 0    60   Input ~ 0
 SPI_SCK
-Text GLabel 5300 4100 0    60   Input ~ 0
+Text GLabel 5300 4150 0    60   Input ~ 0
 SPI_MOSI
-Text GLabel 5300 4250 0    60   Input ~ 0
+Text GLabel 5300 4300 0    60   Input ~ 0
 SPI_MISO
-Text GLabel 5300 4400 0    60   Input ~ 0
+Text GLabel 4200 6950 0    60   Input ~ 0
 SPI_CS5
-Text GLabel 4200 6950 0    60   Input ~ 0
-SPI_CS4
 Text GLabel 4550 6950 2    60   Input ~ 0
 SPI_CS_CC
-Text GLabel 5300 4550 0    60   Input ~ 0
+Text GLabel 5300 4450 0    60   Input ~ 0
 SPI_CS6
-Text GLabel 5300 4700 0    60   Input ~ 0
+Text GLabel 5300 4600 0    60   Input ~ 0
 SPI_CS7
 Wire Wire Line
@@
 	5700 3800 5700 4200
 Wire Wire Line
-	5500 4100 5850 4100
-Wire Wire Line
-	5500 3950 5500 4100
-Wire Wire Line
-	5300 3950 5500 3950
-Wire Wire Line
-	5450 4200 5850 4200
-Wire Wire Line
-	5450 4100 5450 4200
-Wire Wire Line
-	5300 4100 5450 4100
-Wire Wire Line
-	5400 4300 5850 4300
-Wire Wire Line
-	5400 4250 5400 4300
-Wire Wire Line
-	5300 4250 5400 4250
-Wire Wire Line
-	5300 4400 5850 4400
-Wire Wire Line
-	5400 4500 5850 4500
-Wire Wire Line
-	5400 4550 5400 4500
-Wire Wire Line
-	5300 4550 5400 4550
-Wire Wire Line
-	5450 4600 5850 4600
-Wire Wire Line
-	5450 4700 5450 4600
-Wire Wire Line
-	5300 4700 5450 4700
+	5450 4100 5850 4100
+Wire Wire Line
+	5400 4200 5850 4200
+Wire Wire Line
+	5300 4300 5850 4300
 Wire Wire Line
 	4200 6950 4550 6950
 Wire Wire Line
-	5700 4800 5700 5050
-Wire Wire Line
-	5850 4800 5700 4800
+	5700 4700 5700 4950
+Wire Wire Line
+	5850 4700 5700 4700
 Connection ~ 1550 6750
 Wire Wire Line
@@
 Wire Wire Line
 	2450 2800 2550 2800
-Wire Wire Line
-	5800 4700 5850 4700
-Wire Wire Line
-	5800 3100 5800 4700
 Wire Wire Line
 	5550 3200 5800 3200
@@
 $EndComp
 Connection ~ 8600 2800
+$Comp
+L CONN_7 P?
+U 1 1 5472B1C0
+P 6200 4400
+F 0 "P?" V 6170 4400 60  0000 C CNN
+F 1 "CONN_7" V 6270 4400 60  0000 C CNN
+F 2 "" H 6200 4400 60  0000 C CNN
+F 3 "" H 6200 4400 60  0000 C CNN
+	1    6200 4400
+	1    0    0    -1
+$EndComp
+Wire Wire Line
+	5850 4600 5800 4600
+Wire Wire Line
+	5800 4600 5800 3100
+Wire Wire Line
+	5400 4200 5400 4150
+Wire Wire Line
+	5400 4150 5300 4150
+Wire Wire Line
+	5450 4100 5450 4000
+Wire Wire Line
+	5450 4000 5300 4000
+Wire Wire Line
+	5850 4400 5400 4400
+Wire Wire Line
+	5400 4400 5400 4450
+Wire Wire Line
+	5400 4450 5300 4450
+Wire Wire Line
+	5850 4500 5450 4500
+Wire Wire Line
+	5450 4500 5450 4600
+Wire Wire Line
+	5450 4600 5300 4600
 $EndSCHEMATC

Commit message: Added net name for swapped header row
Parts:
- gave numbers to parts that had none: 1
Changed lines of the file:
@@
 Connection ~ 8600 2800
 $Comp
-L CONN_7 P?
+L CONN_7 P4
 U 1 1 5472B1C0
 P 6200 4400
-F 0 "P?" V 6170 4400 60  0000 C CNN
+F 0 "P4" V 6170 4400 60  0000 C CNN
 F 1 "CONN_7" V 6270 4400 60  0000 C CNN
 F 2 "" H 6200 4400 60  0000 C CNN

Commit message: Annotations, DRC fixing, and first round of footprint matching
Parts:
- P4: value CONN_7 -> SPI
Changed lines of the file:
@@
 $Descr A4 11693 8268
 encoding utf-8
-Sheet 3 7
+Sheet 3 8
 Title ""
 Date "24 nov 2014"
@@
 P 6200 4400
 F 0 "P4" V 6170 4400 60  0000 C CNN
-F 1 "CONN_7" V 6270 4400 60  0000 C CNN
+F 1 "SPI" V 6270 4400 60  0000 C CNN
 F 2 "" H 6200 4400 60  0000 C CNN
 F 3 "" H 6200 4400 60  0000 C CNN

Commit message: Replaced buffers with CPLD
Parts:
- removed R7, R8, R9: 47k, ~, symbol R
- removed U1: 74LS138, ~, symbol 74LS138
Connections:
- net labels removed: SPI_CS4, SPI_CS5, SPI_CS_CC, SPI_SEL0, SPI_SEL1, SPI_SEL2
- wire segments 124 -> 98
- no-connect marks 1 -> 0
Changed lines of the file:
@@
 $Descr A4 11693 8268
 encoding utf-8
-Sheet 3 8
+Sheet 3 7
 Title ""
-Date "25 nov 2014"
+Date "13 feb 2015"
 Rev ""
 Comp ""
@@
 $EndComp
 $Comp
-L 74LS138 U1
-U 1 1 546AA00B
-P 2800 5800
-F 0 "U1" H 2900 6300 60  0000 C CNN
-F 1 "74LS138" H 2950 5251 60  0000 C CNN
-F 2 "~" H 2800 5800 60  0000 C CNN
-F 3 "~" H 2800 5800 60  0000 C CNN
-	1    2800 5800
-	1    0    0    -1
-$EndComp
-Text GLabel 1200 5400 0    60   Input ~ 0
-SPI_SEL0
-Text GLabel 1200 5550 0    60   Input ~ 0
-SPI_SEL1
-Text GLabel 1200 5700 0    60   Input ~ 0
-SPI_SEL2
-Text GLabel 3700 5550 2    60   Input ~ 0
-SPI_CS1
-Text GLabel 4150 5650 2    60   Input ~ 0
-SPI_CS2
-Text GLabel 3700 5750 2    60   Input ~ 0
-SPI_CS3
-Text GLabel 4150 5850 2    60   Input ~ 0
-SPI_CS4
-Text GLabel 3700 5950 2    60   Input ~ 0
-SPI_CS5
-Text GLabel 4150 6050 2    60   Input ~ 0
-SPI_CS6
-Text GLabel 3700 6150 2    60   Input ~ 0
-SPI_CS7
-NoConn ~ 3400 5450
-$Comp
-L GND #PWR033
-U 1 1 546AB116
-P 2150 6850
-F 0 "#PWR033" H 2150 6850 30  0001 C CNN
-F 1 "GND" H 2150 6780 30  0001 C CNN
-F 2 "" H 2150 6850 60  0000 C CNN
-F 3 "" H 2150 6850 60  0000 C CNN
-	1    2150 6850
-	1    0    0    -1
-$EndComp
-$Comp
-L R R9
-U 1 1 546AB137
-P 1800 6450
-F 0 "R9" V 1880 6450 40  0000 C CNN
-F 1 "47k" V 1807 6451 40  0000 C CNN
-F 2 "~" V 1730 6450 30  0000 C CNN
-F 3 "~" H 1800 6450 30  0000 C CNN
-	1    1800 6450
-	1    0    0    -1
-$EndComp
-$Comp
-L R R8
-U 1 1 546AB13D
-P 1550 6450
-F 0 "R8" V 1630 6450 40  0000 C CNN
-F 1 "47k" V 1557 6451 40  0000 C CNN
-F 2 "~" V 1480 6450 30  0000 C CNN
-F 3 "~" H 1550 6450 30  0000 C CNN
-	1    1550 6450
-	1    0    0    -1
-$EndComp
-$Comp
-L R R7
-U 1 1 546AB143
-P 1300 6450
-F 0 "R7" V 1380 6450 40  0000 C CNN
-F 1 "47k" V 1307 6451 40  0000 C CNN
-F 2 "~" V 1230 6450 30  0000 C CNN
-F 3 "~" H 1300 6450 30  0000 C CNN
-	1    1300 6450
-	1    0    0    -1
-$EndComp
-$Comp
-L 3V3 #PWR034
-U 1 1 546ABAD8
-P 2050 5950
-F 0 "#PWR034" H 2050 6050 40  0001 C CNN
-F 1 "3V3" H 2050 6075 40  0000 C CNN
-F 2 "" H 2050 5950 60  0000 C CNN
-F 3 "" H 2050 5950 60  0000 C CNN
-	1    2050 5950
-	1    0    0    -1
-$EndComp
-$Comp
 L GND #PWR035
 U 1 1 54726C24
@@
 Text GLabel 5300 4300 0    60   Input ~ 0
 SPI_MISO
-Text GLabel 4200 6950 0    60   Input ~ 0
-SPI_CS5
-Text GLabel 4550 6950 2    60   Input ~ 0
-SPI_CS_CC
 Text GLabel 5300 4450 0    60   Input ~ 0
 SPI_CS6
@@
 	5300 4300 5850 4300
 Wire Wire Line
-	4200 6950 4550 6950
-Wire Wire Line
 	5700 4700 5700 4950
 Wire Wire Line
 	5850 4700 5700 4700
-Connection ~ 1550 6750
-Wire Wire Line
-	1300 6750 1300 6700
-Connection ~ 1800 6750
-Wire Wire Line
-	1550 6750 1550 6700
-Wire Wire Line
-	1800 6750 1800 6700
-Connection ~ 2150 6750
-Wire Wire Line
-	1300 6750 2150 6750
-Connection ~ 1800 5700
-Wire Wire Line
-	1800 6200 1800 5700
-Connection ~ 1550 5550
-Wire Wire Line
-	1550 6200 1550 5550
-Connection ~ 2150 6150
-Wire Wire Line
-	2150 6150 2200 6150
-Wire Wire Line
-	2150 6050 2150 6850
-Wire Wire Line
-	2200 6050 2150 6050
-Wire Wire Line
-	2050 5950 2200 5950
-Connection ~ 1300 5400
-Wire Wire Line
-	1300 5400 1300 6200
-Wire Wire Line
-	3400 6150 3700 6150
-Wire Wire Line
-	3400 6050 4150 6050
-Wire Wire Line
-	3400 5950 3700 5950
-Wire Wire Line
-	3400 5850 4150 5850
-Wire Wire Line
-	3400 5750 3700 5750
-Wire Wire Line
-	3400 5650 4150 5650
-Wire Wire Line
-	3400 5550 3700 5550
-Wire Wire Line
-	2050 5650 2200 5650
-Wire Wire Line
-	2050 5700 2050 5650
-Wire Wire Line
-	1200 5700 2050 5700
-Wire Wire Line
-	2050 5450 2200 5450
-Wire Wire Line
-	2050 5400 2050 5450
-Wire Wire Line
-	1200 5400 2050 5400
-Wire Wire Line
-	1200 5550 2200 5550
 Wire Wire Line
 	7050 3950 7050 4150

Commit message: Various fixes to schematics and footprints:
* Added pullup resistors to bumpers
* Changed value of RLED resistor
* Added resistor to GLED
* Changed SPI pullup resistors to 47k
* Added JTAG header for CPLD
* Changed motor driver footprint to MSOP
Parts:
- R10, R11, R13, R14, R15: value 50k -> 47k
Changed lines of the file:
@@
 P 5700 3550
 F 0 "R15" V 5780 3550 40  0000 C CNN
-F 1 "50k" V 5707 3551 40  0000 C CNN
+F 1 "47k" V 5707 3551 40  0000 C CNN
 F 2 "~" V 5630 3550 30  0000 C CNN
 F 3 "~" H 5700 3550 30  0000 C CNN
@@
 P 5550 3550
 F 0 "R14" V 5630 3550 40  0000 C CNN
-F 1 "50k" V 5557 3551 40  0000 C CNN
+F 1 "47k" V 5557 3551 40  0000 C CNN
 F 2 "~" V 5480 3550 30  0000 C CNN
 F 3 "~" H 5550 3550 30  0000 C CNN
@@
 $EndComp
 $Comp
-L GND #PWR035
+L GND #PWR033
 U 1 1 54726C24
 P 5700 4950
-F 0 "#PWR035" H 5700 4950 30  0001 C CNN
+F 0 "#PWR033" H 5700 4950 30  0001 C CNN
 F 1 "GND" H 5700 4880 30  0001 C CNN
 F 2 "" H 5700 4950 60  0000 C CNN
@@
 $EndComp
 $Comp
-L 3V3 #PWR036
+L 3V3 #PWR034
 U 1 1 54726D33
 P 5800 3100
-F 0 "#PWR036" H 5800 3200 40  0001 C CNN
+F 0 "#PWR034" H 5800 3200 40  0001 C CNN
 F 1 "3V3" H 5800 3225 40  0000 C CNN
 F 2 "" H 5800 3100 60  0000 C CNN
@@
 P 2450 1700
 F 0 "R13" V 2530 1700 40  0000 C CNN
-F 1 "50k" V 2457 1701 40  0000 C CNN
+F 1 "47k" V 2457 1701 40  0000 C CNN
 F 2 "~" V 2380 1700 30  0000 C CNN
 F 3 "~" H 2450 1700 30  0000 C CNN
@@
 P 2150 1700
 F 0 "R11" V 2230 1700 40  0000 C CNN
-F 1 "50k" V 2157 1701 40  0000 C CNN
+F 1 "47k" V 2157 1701 40  0000 C CNN
 F 2 "~" V 2080 1700 30  0000 C CNN
 F 3 "~" H 2150 1700 30  0000 C CNN
@@
 	7050 3800 7050 3450
 $Comp
-L 3V3 #PWR037
+L 3V3 #PWR035
 U 1 1 54728806
 P 7050 2900
-F 0 "#PWR037" H 7050 3000 40  0001 C CNN
+F 0 "#PWR035" H 7050 3000 40  0001 C CNN
 F 1 "3V3" H 7050 3025 40  0000 C CNN
 F 2 "" H 7050 2900 60  0000 C CNN
@@
 P 1850 1700
 F 0 "R10" V 1930 1700 40  0000 C CNN
-F 1 "50k" V 1857 1701 40  0000 C CNN
+F 1 "47k" V 1857 1701 40  0000 C CNN
 F 2 "~" V 1780 1700 30  0000 C CNN
 F 3 "~" H 1850 1700 30  0000 C CNN
@@
 Connection ~ 8600 2550
 $Comp
-L GND #PWR038
+L GND #PWR036
 U 1 1 54729C52
 P 8600 2900
-F 0 "#PWR038" H 8600 2900 30  0001 C CNN
+F 0 "#PWR036" H 8600 2900 30  0001 C CNN
 F 1 "GND" H 8600 2830 30  0001 C CNN
 F 2 "" H 8600 2900 60  0000 C CNN
