File: board/mainboard/SPI_peripherals.sch (KiCad schematic (older format))
At the start: 22 parts, among them J1 BACKL, P4 SPI, P5 DAC

Commit message: Finished draft 1 of Rev 2 layout
Parts:
- removed R10: 47k, ~, symbol R
Connections:
- wire segments 98 -> 96
Changed lines of the file:
@@
 $Descr A4 11693 8268
 encoding utf-8
-Sheet 3 7
+Sheet 3 8
 Title ""
-Date "26 feb 2015"
+Date "1 mar 2015"
 Rev ""
 Comp ""
@@
 Wire Wire Line
 	2300 2500 2300 1300
-Wire Wire Line
-	1850 1300 2450 1300
 Connection ~ 2450 1300
 Wire Wire Line
@@
 Wire Wire Line
 	1650 2950 2550 2950
-$Comp
-L R R10
-U 1 1 5472863C
-P 1850 1700
-F 0 "R10" V 1930 1700 40  0000 C CNN
-F 1 "47k" V 1857 1701 40  0000 C CNN
-F 2 "~" V 1780 1700 30  0000 C CNN
-F 3 "~" H 1850 1700 30  0000 C CNN
-	1    1850 1700
-	1    0    0    -1
-$EndComp
-Wire Wire Line
-	1850 1450 1850 1300
-Connection ~ 2000 1300
-Wire Wire Line
-	1850 2200 1850 1950
 Connection ~ 1850 2200
 Wire Wire Line
@@
 Wire Wire Line
 	5450 4600 5300 4600
+Wire Wire Line
+	2000 1300 2450 1300
 $EndSCHEMATC
