File: board/mainboard/i2c_peripherals.sch (KiCad schematic (older format))
At the start: 14 parts

Commit message: Removed temperature sensor
Parts:
- removed C?: 0.1uF, ~, symbol C
- removed TMP?: TMP100, ~, symbol TMP100
- added R? (x2): R_i2c, ~, symbol R
Connections:
- wire segments 78 -> 74
Other:
- note removed: "Temperature Sensor\nI2C ADDR = 1001000x"

Commit message: Added i2c exposed header
Parts:
- added P?: I2C, symbol CONN_4
- added P?: MOTORS, symbol CONN_4
Connections:
- wire segments 74 -> 89
Changed lines of the file:
@@
 	1    0    0    -1
 $EndComp
-Wire Wire Line
-	2100 1650 1650 1650
-Wire Wire Line
-	2100 1800 1550 1800
-Wire Wire Line
-	1550 1800 1550 1850
-Wire Wire Line
-	1850 1950 2100 1950
-Wire Wire Line
-	1850 1950 1850 2250
-Wire Wire Line
-	1850 2250 1550 2250
-Wire Wire Line
-	1850 2650 1850 2700
-Wire Wire Line
-	2050 2350 2050 2100
-Wire Wire Line
-	2050 2100 2100 2100
-Wire Wire Line
-	3800 1450 3800 1650
-Wire Wire Line
-	3800 1650 3700 1650
-Wire Wire Line
-	3950 1950 3700 1950
-Wire Wire Line
-	3700 1800 3950 1800
-Wire Wire Line
-	8150 1400 7950 1400
-Wire Wire Line
-	7950 1400 7950 1100
-Wire Wire Line
-	8150 1600 7700 1600
-Wire Wire Line
-	7700 1750 8150 1750
-Wire Wire Line
-	8150 1950 7900 1950
-Wire Wire Line
-	7900 1950 7900 2550
-Wire Wire Line
-	8150 2100 7900 2100
-Connection ~ 7900 2100
-Wire Wire Line
-	9000 2700 9000 2800
-Wire Wire Line
-	10150 1600 9850 1600
-Wire Wire Line
-	9850 1750 10150 1750
-Wire Wire Line
-	9850 2300 10050 2300
-Wire Wire Line
-	10050 2800 10050 2900
-Wire Wire Line
-	8150 3800 7950 3800
-Wire Wire Line
-	7950 3800 7950 3500
-Wire Wire Line
-	8150 4000 7700 4000
-Wire Wire Line
-	7700 4150 8150 4150
-Wire Wire Line
-	8150 4500 7900 4500
-Wire Wire Line
-	9000 5100 9000 5200
-Wire Wire Line
-	10150 4000 9850 4000
-Wire Wire Line
-	9850 4150 10150 4150
-Wire Wire Line
-	9850 4700 10050 4700
-Wire Wire Line
-	10050 5200 10050 5300
-Wire Wire Line
-	7900 4500 7900 4950
-Wire Wire Line
-	7700 2300 8150 2300
-Wire Wire Line
-	7700 4700 8150 4700
-Wire Wire Line
-	3700 2100 3950 2100
-Wire Wire Line
-	2650 3200 2650 3650
-Wire Wire Line
-	2900 3200 2900 3650
-Wire Wire Line
-	3150 3200 3150 3650
-Wire Wire Line
-	3800 4350 4700 4350
-Wire Wire Line
-	4700 4350 4700 4500
-Wire Wire Line
-	3800 4500 4450 4500
-Wire Wire Line
-	2900 5800 2900 5550
-Wire Wire Line
-	2650 5550 2650 5650
-Wire Wire Line
-	2650 5650 3150 5650
-Connection ~ 2900 5650
-Wire Wire Line
-	3150 5650 3150 5550
-Wire Wire Line
-	2000 4800 1750 4800
-Wire Wire Line
-	1750 4800 1750 5000
-Wire Wire Line
-	1650 4600 2000 4600
-Wire Wire Line
-	1850 4500 1850 4400
-Wire Wire Line
-	1850 4400 2000 4400
-Wire Wire Line
-	1700 4050 2000 4050
-Wire Wire Line
-	1700 4200 2000 4200
-Wire Wire Line
-	4600 5150 4600 5000
-Wire Wire Line
-	4450 5000 4700 5000
-Wire Wire Line
-	4450 5000 4450 4900
-Wire Wire Line
-	4700 5000 4700 4900
-Connection ~ 4600 5000
-Wire Wire Line
-	3150 3250 3450 3250
-Wire Wire Line
-	3450 3250 3450 3300
-Connection ~ 3150 3250
-Wire Wire Line
-	2350 3700 2350 3800
-Wire Wire Line
-	3450 3700 3450 3800
-Wire Wire Line
-	2900 3250 2350 3250
-Wire Wire Line
-	2350 3250 2350 3300
-Connection ~ 2900 3250
 $Comp
 L GND #PWR?
@@
 	1    0    0    -1
 $EndComp
-Wire Wire Line
-	3950 5150 3950 4900
-Wire Wire Line
-	3950 4900 3800 4900
 Text GLabel 5200 6250 0    60   Input ~ 0
 I2C_CL
@@
 	1    0    0    -1
 $EndComp
-Wire Wire Line
-	5500 6250 5500 6150
-Wire Wire Line
-	5200 6250 5500 6250
 $Comp
 L 3V3 #PWR?
@@
 	1    0    0    -1
 $EndComp
-Wire Wire Line
-	5500 5650 5500 5450
 $Comp
 L R R?
@@
 	1    0    0    -1
 $EndComp
+$Comp
+L CONN_4 P?
+U 1 1 546AB17E
+P 6650 6400
+F 0 "P?" V 6600 6400 50  0000 C CNN
+F 1 "I2C" V 6700 6400 50  0000 C CNN
+F 2 "" H 6650 6400 60  0000 C CNN
+F 3 "" H 6650 6400 60  0000 C CNN
+	1    6650 6400
+	1    0    0    -1
+$EndComp
+Wire Wire Line
+	2100 1650 1650 1650
+Wire Wire Line
+	2100 1800 1550 1800
+Wire Wire Line
+	1550 1800 1550 1850
+Wire Wire Line
+	1850 1950 2100 1950
+Wire Wire Line
+	1850 1950 1850 2250
+Wire Wire Line
+	1850 2250 1550 2250
+Wire Wire Line
+	1850 2650 1850 2700
+Wire Wire Line
+	2050 2350 2050 2100
+Wire Wire Line
+	2050 2100 2100 2100
+Wire Wire Line
+	3800 1450 3800 1650
+Wire Wire Line
+	3800 1650 3700 1650
+Wire Wire Line
+	3950 1950 3700 1950
+Wire Wire Line
+	3700 1800 3950 1800
+Wire Wire Line
+	8150 1400 7950 1400
+Wire Wire Line
+	7950 1400 7950 1100
+Wire Wire Line
+	8150 1600 7700 1600
+Wire Wire Line
+	7700 1750 8150 1750
+Wire Wire Line
+	8150 1950 7900 1950
+Wire Wire Line
+	7900 1950 7900 2550
+Wire Wire Line
+	8150 2100 7900 2100
+Connection ~ 7900 2100
+Wire Wire Line
+	9000 2700 9000 2800
+Wire Wire Line
+	10150 1600 9850 1600
+Wire Wire Line
+	9850 1750 10150 1750
+Wire Wire Line
+	9850 2300 10050 2300
+Wire Wire Line
+	10050 2800 10050 2900
+Wire Wire Line
+	8150 3800 7950 3800
+Wire Wire Line
+	7950 3800 7950 3500
+Wire Wire Line
+	8150 4000 7700 4000
+Wire Wire Line
+	7700 4150 8150 4150
+Wire Wire Line
+	8150 4500 7900 4500
+Wire Wire Line
+	9000 5100 9000 5200
+Wire Wire Line
+	10150 4000 9850 4000
+Wire Wire Line
+	9850 4150 10150 4150
+Wire Wire Line
+	9850 4700 10050 4700
+Wire Wire Line
+	10050 5200 10050 5300
+Wire Wire Line
+	7900 4500 7900 4950
+Wire Wire Line
+	7700 2300 8150 2300
+Wire Wire Line
+	7700 4700 8150 4700
+Wire Wire Line
+	3700 2100 3950 2100
+Wire Wire Line
+	2650 3200 2650 3650
+Wire Wire Line
+	2900 3200 2900 3650
+Wire Wire Line
+	3150 3200 3150 3650
+Wire Wire Line
+	3800 4350 4700 4350
+Wire Wire Line
+	4700 4350 4700 4500
+Wire Wire Line
+	3800 4500 4450 4500
+Wire Wire Line
+	2900 5800 2900 5550
+Wire Wire Line
+	2650 5550 2650 5650
+Wire Wire Line
+	2650 5650 3150 5650
+Connection ~ 2900 5650
+Wire Wire Line
+	3150 5650 3150 5550
+Wire Wire Line
+	2000 4800 1750 4800
+Wire Wire Line
+	1750 4800 1750 5000
+Wire Wire Line
+	1650 4600 2000 4600
+Wire Wire Line
+	1850 4500 1850 4400
+Wire Wire Line
+	1850 4400 2000 4400
+Wire Wire Line
+	1700 4050 2000 4050
+Wire Wire Line
+	1700 4200 2000 4200
+Wire Wire Line
+	4600 5150 4600 5000
+Wire Wire Line
+	4450 5000 4700 5000
+Wire Wire Line
+	4450 5000 4450 4900
+Wire Wire Line
+	4700 5000 4700 4900
+Connection ~ 4600 5000
+Wire Wire Line
+	3150 3250 3450 3250
+Wire Wire Line
+	3450 3250 3450 3300
+Connection ~ 3150 3250
+Wire Wire Line
+	2350 3700 2350 3800
+Wire Wire Line
+	3450 3700 3450 3800
+Wire Wire Line
+	2900 3250 2350 3250
+Wire Wire Line
+	2350 3250 2350 3300
+Connection ~ 2900 3250
+Wire Wire Line
+	3950 5150 3950 4900
+Wire Wire Line
+	3950 4900 3800 4900
+Wire Wire Line
+	5500 6250 5500 6150
+Wire Wire Line
+	5500 5650 5500 5450
 Wire Wire Line
 	5700 5650 5700 5450
 Wire Wire Line
 	5200 6400 5700 6400
+Connection ~ 5500 6250
+Wire Wire Line
+	5200 6250 6300 6250
 Wire Wire Line
 	5700 6400 5700 6150
+Wire Wire Line
+	5700 6350 6300 6350
+Connection ~ 5700 6350
+$Comp
+L 3V3 #PWR?
+U 1 1 546AB46C
+P 6200 6150
+F 0 "#PWR?" H 6200 6250 40  0001 C CNN
+F 1 "3V3" H 6200 6275 40  0000 C CNN
+F 2 "" H 6200 6150 60  0000 C CNN
+F 3 "" H 6200 6150 60  0000 C CNN
+	1    6200 6150
+	1    0    0    -1
+$EndComp
+Wire Wire Line
+	6300 6450 6200 6450
+Wire Wire Line
+	6200 6450 6200 6150
+$Comp
+L GND #PWR?
+U 1 1 546AB4C5
+P 6200 6700
+F 0 "#PWR?" H 6200 6700 30  0001 C CNN
+F 1 "GND" H 6200 6630 30  0001 C CNN
+F 2 "" H 6200 6700 60  0000 C CNN
+F 3 "" H 6200 6700 60  0000 C CNN
+	1    6200 6700
+	1    0    0    -1
+$EndComp
+Wire Wire Line
+	6200 6700 6200 6550
+Wire Wire Line
+	6200 6550 6300 6550
+$Comp
+L CONN_4 P?
+U 1 1 546AB530
+P 9900 6300
+F 0 "P?" V 9850 6300 50  0000 C CNN
+F 1 "MOTORS" V 9950 6300 50  0000 C CNN
+F 2 "" H 9900 6300 60  0000 C CNN
+F 3 "" H 9900 6300 60  0000 C CNN
+	1    9900 6300
+	1    0    0    -1
+$EndComp
+Text GLabel 9150 6200 0    60   Input ~ 0
+MOTOR1-
+Text GLabel 9150 6050 0    60   Input ~ 0
+MOTOR1+
+Text GLabel 9150 6500 0    60   Input ~ 0
+MOTOR2-
+Text GLabel 9150 6350 0    60   Input ~ 0
+MOTOR2+
+Wire Wire Line
+	9150 6050 9350 6050
+Wire Wire Line
+	9350 6050 9350 6150
+Wire Wire Line
+	9350 6150 9550 6150
+Wire Wire Line
+	9150 6200 9250 6200
+Wire Wire Line
+	9250 6200 9250 6250
+Wire Wire Line
+	9250 6250 9550 6250
+Wire Wire Line
+	9150 6350 9550 6350
+Wire Wire Line
+	9150 6500 9250 6500
+Wire Wire Line
+	9250 6500 9250 6450
+Wire Wire Line
+	9250 6450 9550 6450
 $EndSCHEMATC

Commit message: Fixed crystals and added mic to audio codec
Parts:
- removed X?: 32.768kHz, ~, symbol CRYSTAL_SMD
- added X?: 32.768KHz, ~, symbol CRYSTAL
- C?: value Cg -> 5pF
- R? (x2): value R_i2c -> 4.7k
Changed lines of the file:
@@
 RTCINT1
-$Comp
-L CRYSTAL_SMD X?
-U 1 1 54485CEB
-P 1550 2050
-F 0 "X?" H 1550 2140 30  0000 C CNN
-F 1 "32.768kHz" H 1580 1940 30  0000 L CNN
-F 2 "~" H 1550 2050 60  0000 C CNN
-F 3 "~" H 1550 2050 60  0000 C CNN
-	1    1550 2050
-	0    -1   -1   0
-$EndComp
 $Comp
 L C C?
@@
 P 1850 2450
 F 0 "C?" H 1850 2550 40  0000 L CNN
-F 1 "Cg" H 1856 2365 40  0000 L CNN
+F 1 "5pF" H 1856 2365 40  0000 L CNN
 F 2 "~" H 1888 2300 30  0000 C CNN
 F 3 "~" H 1850 2450 60  0000 C CNN
@@
 P 5500 5900
 F 0 "R?" V 5580 5900 40  0000 C CNN
-F 1 "R_i2c" V 5507 5901 40  0000 C CNN
+F 1 "4.7k" V 5507 5901 40  0000 C CNN
 F 2 "~" V 5430 5900 30  0000 C CNN
 F 3 "~" H 5500 5900 30  0000 C CNN
@@
 P 5700 5900
 F 0 "R?" V 5780 5900 40  0000 C CNN
-F 1 "R_i2c" V 5707 5901 40  0000 C CNN
+F 1 "4.7k" V 5707 5901 40  0000 C CNN
 F 2 "~" V 5630 5900 30  0000 C CNN
 F 3 "~" H 5700 5900 30  0000 C CNN
@@
 	2100 1650 1650 1650
 Wire Wire Line
-	2100 1800 1550 1800
-Wire Wire Line
-	1550 1800 1550 1850
-Wire Wire Line
-	1850 1950 2100 1950
+	1600 1950 2100 1950
 Wire Wire Line
 	1850 1950 1850 2250
-Wire Wire Line
-	1850 2250 1550 2250
 Wire Wire Line
 	1850 2650 1850 2700
@@
 Wire Wire Line
 	9250 6450 9550 6450
+$Comp
+L CRYSTAL X?
+U 1 1 546AD855
+P 1200 2100
+F 0 "X?" H 1200 2250 60  0000 C CNN
+F 1 "32.768KHz" H 1200 1950 60  0000 C CNN
+F 2 "~" H 1200 2100 60  0000 C CNN
+F 3 "~" H 1200 2100 60  0000 C CNN
+	1    1200 2100
+	0    -1   -1   0
+$EndComp
+Wire Wire Line
+	2100 1800 1200 1800
+Wire Wire Line
+	1200 2400 1600 2400
+Wire Wire Line
+	1600 2400 1600 1950
+Connection ~ 1850 1950
 $EndSCHEMATC
