File: board/mainboard/i2c_peripherals.sch (KiCad schematic (older format))
At the start: 16 parts

Commit message: Added missing pullups on the RTC interrupt lines
Parts:
- added R? (x2): 4.7k, ~, symbol R
Connections:
- wire segments 89 -> 93
Changed lines of the file:
@@
 $Descr A4 11693 8268
 encoding utf-8
-Sheet 2 5
+Sheet 2 7
 Title ""
-Date "19 nov 2014"
+Date "24 nov 2014"
 Rev ""
 Comp ""
@@
 Text GLabel 7700 4700 0    60   Input ~ 0
 MOTOR2F
-Text GLabel 3950 2100 2    60   Input ~ 0
+Text GLabel 4600 2100 2    60   Input ~ 0
 RTCINT2
 $Comp
@@
 	7700 4700 8150 4700
 Wire Wire Line
-	3700 2100 3950 2100
+	3700 2100 4600 2100
 Wire Wire Line
 	2650 3200 2650 3650
@@
 	1600 2400 1600 1950
 Connection ~ 1850 1950
+$Comp
+L R R?
+U 1 1 54727DCC
+P 4450 1700
+F 0 "R?" V 4530 1700 40  0000 C CNN
+F 1 "4.7k" V 4457 1701 40  0000 C CNN
+F 2 "~" V 4380 1700 30  0000 C CNN
+F 3 "~" H 4450 1700 30  0000 C CNN
+	1    4450 1700
+	1    0    0    -1
+$EndComp
+$Comp
+L 3V3 #PWR?
+U 1 1 54727DD2
+P 4450 1250
+F 0 "#PWR?" H 4450 1350 40  0001 C CNN
+F 1 "3V3" H 4450 1375 40  0000 C CNN
+F 2 "" H 4450 1250 60  0000 C CNN
+F 3 "" H 4450 1250 60  0000 C CNN
+	1    4450 1250
+	1    0    0    -1
+$EndComp
+$Comp
+L R R?
+U 1 1 54727DD8
+P 1950 1300
+F 0 "R?" V 2030 1300 40  0000 C CNN
+F 1 "4.7k" V 1957 1301 40  0000 C CNN
+F 2 "~" V 1880 1300 30  0000 C CNN
+F 3 "~" H 1950 1300 30  0000 C CNN
+	1    1950 1300
+	1    0    0    -1
+$EndComp
+$Comp
+L 3V3 #PWR?
+U 1 1 54727DDE
+P 1950 850
+F 0 "#PWR?" H 1950 950 40  0001 C CNN
+F 1 "3V3" H 1950 975 40  0000 C CNN
+F 2 "" H 1950 850 60  0000 C CNN
+F 3 "" H 1950 850 60  0000 C CNN
+	1    1950 850
+	1    0    0    -1
+$EndComp
+Wire Wire Line
+	4450 1450 4450 1250
+Wire Wire Line
+	1950 1050 1950 850
+Wire Wire Line
+	1950 1550 1950 1650
+Connection ~ 1950 1650
+Wire Wire Line
+	4450 1950 4450 2100
+Connection ~ 4450 2100
 $EndSCHEMATC

Commit message: Split the motors into two separate headers
Parts:
- removed P?: MOTORS, symbol CONN_4
- added P?: Motor1, symbol CONN_2
- added P?: Motor2, symbol CONN_2
- R? (x2): value 4.7k -> 10K
Connections:
- wire segments 93 -> 87
Changed lines of the file:
@@
 Wire Wire Line
 	6200 6550 6300 6550
-$Comp
-L CONN_4 P?
-U 1 1 546AB530
-P 9900 6300
-F 0 "P?" V 9850 6300 50  0000 C CNN
-F 1 "MOTORS" V 9950 6300 50  0000 C CNN
-F 2 "" H 9900 6300 60  0000 C CNN
-F 3 "" H 9900 6300 60  0000 C CNN
-	1    9900 6300
-	1    0    0    -1
-$EndComp
-Text GLabel 9150 6200 0    60   Input ~ 0
+Text GLabel 9150 6250 0    60   Input ~ 0
 MOTOR1-
 Text GLabel 9150 6050 0    60   Input ~ 0
 MOTOR1+
-Text GLabel 9150 6500 0    60   Input ~ 0
+Text GLabel 9150 6750 0    60   Input ~ 0
 MOTOR2-
-Text GLabel 9150 6350 0    60   Input ~ 0
+Text GLabel 9150 6550 0    60   Input ~ 0
 MOTOR2+
-Wire Wire Line
-	9150 6050 9350 6050
-Wire Wire Line
-	9350 6050 9350 6150
-Wire Wire Line
-	9350 6150 9550 6150
-Wire Wire Line
-	9150 6200 9250 6200
-Wire Wire Line
-	9250 6200 9250 6250
-Wire Wire Line
-	9250 6250 9550 6250
-Wire Wire Line
-	9150 6350 9550 6350
-Wire Wire Line
-	9150 6500 9250 6500
-Wire Wire Line
-	9250 6500 9250 6450
-Wire Wire Line
-	9250 6450 9550 6450
 $Comp
 L CRYSTAL X?
@@
 P 4450 1700
 F 0 "R?" V 4530 1700 40  0000 C CNN
-F 1 "4.7k" V 4457 1701 40  0000 C CNN
+F 1 "10K" V 4457 1701 40  0000 C CNN
 F 2 "~" V 4380 1700 30  0000 C CNN
 F 3 "~" H 4450 1700 30  0000 C CNN
@@
 P 1950 1300
 F 0 "R?" V 2030 1300 40  0000 C CNN
-F 1 "4.7k" V 1957 1301 40  0000 C CNN
+F 1 "10K" V 1957 1301 40  0000 C CNN
 F 2 "~" V 1880 1300 30  0000 C CNN
 F 3 "~" H 1950 1300 30  0000 C CNN
@@
 	4450 1950 4450 2100
 Connection ~ 4450 2100
+$Comp
+L CONN_2 P?
+U 1 1 5472816B
+P 9650 6150
+F 0 "P?" V 9600 6150 40  0000 C CNN
+F 1 "Motor1" V 9700 6150 40  0000 C CNN
+F 2 "" H 9650 6150 60  0000 C CNN
+F 3 "" H 9650 6150 60  0000 C CNN
+	1    9650 6150
+	1    0    0    -1
+$EndComp
+Wire Wire Line
+	9150 6050 9300 6050
+Wire Wire Line
+	9150 6250 9300 6250
+$Comp
+L CONN_2 P?
+U 1 1 54728242
+P 9650 6650
+F 0 "P?" V 9600 6650 40  0000 C CNN
+F 1 "Motor2" V 9700 6650 40  0000 C CNN
+F 2 "" H 9650 6650 60  0000 C CNN
+F 3 "" H 9650 6650 60  0000 C CNN
+	1    9650 6650
+	1    0    0    -1
+$EndComp
+Wire Wire Line
+	9150 6550 9300 6550
+Wire Wire Line
+	9150 6750 9300 6750
 $EndSCHEMATC

Commit message: Added net names, fixed misnamed GLCD_A0
Parts:
- gave numbers to parts that had none: 19

Commit message: Various changes
* Began Rev2 Layout
* Added Pullup Resistors to LP I2C
* Added IrDA Module
Parts:
- removed R3, R4: 4.7k, ~, symbol R
Connections:
- wire segments 87 -> 84
Changed lines of the file:
@@
 Sheet 2 7
 Title ""
-Date "16 feb 2015"
+Date "26 feb 2015"
 Rev ""
 Comp ""
@@
 F 3 "~" H 1850 2450 60  0000 C CNN
 	1    1850 2450
-	-1   0    0    1
-$EndComp
-$Comp
-L GND #PWR2
+	1    0    0    -1
+$EndComp
+$Comp
+L GND #PWR01
 U 1 1 54485DA7
 P 1850 2700
-F 0 "#PWR2" H 1850 2700 30  0001 C CNN
+F 0 "#PWR01" H 1850 2700 30  0001 C CNN
 F 1 "GND" H 1850 2630 30  0001 C CNN
 F 2 "" H 1850 2700 60  0000 C CNN
@@
 $EndComp
 $Comp
-L GND #PWR5
+L GND #PWR02
 U 1 1 54485DC8
 P 2050 2350
-F 0 "#PWR5" H 2050 2350 30  0001 C CNN
+F 0 "#PWR02" H 2050 2350 30  0001 C CNN
 F 1 "GND" H 2050 2280 30  0001 C CNN
 F 2 "" H 2050 2350 60  0000 C CNN
@@
 $EndComp
 $Comp
-L 3V3 #PWR11
+L 3V3 #PWR03
 U 1 1 54485DFD
 P 3800 1450
-F 0 "#PWR11" H 3800 1550 40  0001 C CNN
+F 0 "#PWR03" H 3800 1550 40  0001 C CNN
 F 1 "3V3" H 3800 1575 40  0000 C CNN
 F 2 "" H 3800 1450 60  0000 C CNN
@@
 MOTOR1+
 $Comp
-L 3V3 #PWR21
+L 3V3 #PWR04
 U 1 1 54486A99
 P 7950 1100
-F 0 "#PWR21" H 7950 1200 40  0001 C CNN
+F 0 "#PWR04" H 7950 1200 40  0001 C CNN
 F 1 "3V3" H 7950 1225 40  0000 C CNN
 F 2 "" H 7950 1100 60  0000 C CNN
@@
 I2C_DA
 $Comp
-L GND #PWR19
+L GND #PWR05
 U 1 1 54486B17
 P 7900 2550
-F 0 "#PWR19" H 7900 2550 30  0001 C CNN
+F 0 "#PWR05" H 7900 2550 30  0001 C CNN
 F 1 "GND" H 7900 2480 30  0001 C CNN
 F 2 "" H 7900 2550 60  0000 C CNN
@@
 $EndComp
 $Comp
-L GND #PWR23
+L GND #PWR06
 U 1 1 54486B7F
 P 9000 2800
-F 0 "#PWR23" H 9000 2800 30  0001 C CNN
+F 0 "#PWR06" H 9000 2800 30  0001 C CNN
 F 1 "GND" H 9000 2730 30  0001 C CNN
 F 2 "" H 9000 2800 60  0000 C CNN
@@
 $EndComp
 $Comp
-L GND #PWR25
+L GND #PWR07
 U 1 1 54486C8F
 P 10050 2900
-F 0 "#PWR25" H 10050 2900 30  0001 C CNN
+F 0 "#PWR07" H 10050 2900 30  0001 C CNN
 F 1 "GND" H 10050 2830 30  0001 C CNN
 F 2 "" H 10050 2900 60  0000 C CNN
@@
 MOTOR2+
 $Comp
-L 3V3 #PWR22
+L 3V3 #PWR08
 U 1 1 544871AE
 P 7950 3500
-F 0 "#PWR22" H 7950 3600 40  0001 C CNN
+F 0 "#PWR08" H 7950 3600 40  0001 C CNN
 F 1 "3V3" H 7950 3625 40  0000 C CNN
 F 2 "" H 7950 3500 60  0000 C CNN
@@
 I2C_DA
 $Comp
-L GND #PWR20
+L GND #PWR09
 U 1 1 544871BA
 P 7900 4950
-F 0 "#PWR20" H 7900 4950 30  0001 C CNN
+F 0 "#PWR09" H 7900 4950 30  0001 C CNN
 F 1 "GND" H 7900 4880 30  0001 C CNN
 F 2 "" H 7900 4950 60  0000 C CNN
@@
 $EndComp
 $Comp
-L GND #PWR24
+L GND #PWR010
 U 1 1 544871C5
 P 9000 5200
-F 0 "#PWR24" H 9000 5200 30  0001 C CNN
+F 0 "#PWR010" H 9000 5200 30  0001 C CNN
 F 1 "GND" H 9000 5130 30  0001 C CNN
 F 2 "" H 9000 5200 60  0000 C CNN
@@
 $EndComp
 $Comp
-L GND #PWR26
+L GND #PWR011
 U 1 1 544871D5
 P 10050 5300
-F 0 "#PWR26" H 10050 5300 30  0001 C CNN
+F 0 "#PWR011" H 10050 5300 30  0001 C CNN
 F 1 "GND" H 10050 5230 30  0001 C CNN
 F 2 "" H 10050 5300 60  0000 C CNN
@@
 $EndComp
 $Comp
-L 3V3 #PWR7
+L 3V3 #PWR012
 U 1 1 54487B46
 P 2900 3200
-F 0 "#PWR7" H 2900 3300 40  0001 C CNN
+F 0 "#PWR012" H 2900 3300 40  0001 C CNN
 F 1 "3V3" H 2900 3325 40  0000 C CNN
 F 2 "" H 2900 3200 60  0000 C CNN
@@
 $EndComp
 $Comp
-L 3V3 #PWR9
+L 3V3 #PWR013
 U 1 1 54487B4C
 P 3150 3200
-F 0 "#PWR9" H 3150 3300 40  0001 C CNN
+F 0 "#PWR013" H 3150 3300 40  0001 C CNN
 F 1 "3V3" H 3150 3325 40  0000 C CNN
 F 2 "" H 3150 3200 60  0000 C CNN
@@
 $EndComp
 $Comp
-L GND #PWR8
+L GND #PWR014
 U 1 1 54487CE8
 P 2900 5800
-F 0 "#PWR8" H 2900 5800 30  0001 C CNN
+F 0 "#PWR014" H 2900 5800 30  0001 C CNN
 F 1 "GND" H 2900 5730 30  0001 C CNN
 F 2 "" H 2900 5800 60  0000 C CNN
@@
 NoConn ~ 2000 5150
 $Comp
-L GND #PWR1
+L GND #PWR015
 U 1 1 54487DE4
 P 1750 5000
-F 0 "#PWR1" H 1750 5000 30  0001 C CNN
+F 0 "#PWR015" H 1750 5000 30  0001 C CNN
 F 1 "GND" H 1750 4930 30  0001 C CNN
 F 2 "" H 1750 5000 60  0000 C CNN
@@
 MPUINT
 $Comp
-L GND #PWR3
+L GND #PWR016
 U 1 1 54487EB2
 P 1850 4500
-F 0 "#PWR3" H 1850 4500 30  0001 C CNN
+F 0 "#PWR016" H 1850 4500 30  0001 C CNN
 F 1 "GND" H 1850 4430 30  0001 C CNN
 F 2 "" H 1850 4500 60  0000 C CNN
@@
 I2C_DA
 $Comp
-L GND #PWR14
+L GND #PWR017
 U 1 1 54487F92
 P 4600 5150
-F 0 "#PWR14" H 4600 5150 30  0001 C CNN
+F 0 "#PWR017" H 4600 5150 30  0001 C CNN
 F 1 "GND" H 4600 5080 30  0001 C CNN
 F 2 "" H 4600 5150 60  0000 C CNN
@@
 $EndComp
 $Comp
-L GND #PWR10
+L GND #PWR018
 U 1 1 54488133
 P 3450 3800
-F 0 "#PWR10" H 3450 3800 30  0001 C CNN
+F 0 "#PWR018" H 3450 3800 30  0001 C CNN
 F 1 "GND" H 3450 3730 30  0001 C CNN
 F 2 "" H 3450 3800 60  0000 C CNN
@@
 $EndComp
 $Comp
-L GND #PWR6
+L GND #PWR019
 U 1 1 54488142
 P 2350 3800
-F 0 "#PWR6" H 2350 3800 30  0001 C CNN
+F 0 "#PWR019" H 2350 3800 30  0001 C CNN
 F 1 "GND" H 2350 3730 30  0001 C CNN
 F 2 "" H 2350 3800 60  0000 C CNN
@@
 $EndComp
 $Comp
-L GND #PWR12
+L GND #PWR020
 U 1 1 544882A5
 P 3950 5150
-F 0 "#PWR12" H 3950 5150 30  0001 C CNN
+F 0 "#PWR020" H 3950 5150 30  0001 C CNN
 F 1 "GND" H 3950 5080 30  0001 C CNN
 F 2 "" H 3950 5150 60  0000 C CNN
@@
 Text GLabel 5200 6400 0    60   Input ~ 0
 I2C_DA
-$Comp
-L R R3
-U 1 1 5467D6CE
-P 5500 5900
-F 0 "R3" V 5580 5900 40  0000 C CNN
-F 1 "4.7k" V 5507 5901 40  0000 C CNN
-F 2 "~" V 5430 5900 30  0000 C CNN
-F 3 "~" H 5500 5900 30  0000 C CNN
-	1    5500 5900
-	1    0    0    -1
-$EndComp
-$Comp
-L 3V3 #PWR15
-U 1 1 5467D7BD
-P 5500 5450
-F 0 "#PWR15" H 5500 5550 40  0001 C CNN
-F 1 "3V3" H 5500 5575 40  0000 C CNN
-F 2 "" H 5500 5450 60  0000 C CNN
-F 3 "" H 5500 5450 60  0000 C CNN
-	1    5500 5450
-	1    0    0    -1
-$EndComp
-$Comp
-L R R4
-U 1 1 5467D816
-P 5700 5900
-F 0 "R4" V 5780 5900 40  0000 C CNN
-F 1 "4.7k" V 5707 5901 40  0000 C CNN
-F 2 "~" V 5630 5900 30  0000 C CNN
-F 3 "~" H 5700 5900 30  0000 C CNN
-	1    5700 5900
-	1    0    0    -1
-$EndComp
-$Comp
-L 3V3 #PWR16
-U 1 1 5467D81C
-P 5700 5450
-F 0 "#PWR16" H 5700 5550 40  0001 C CNN
-F 1 "3V3" H 5700 5575 40  0000 C CNN
-F 2 "" H 5700 5450 60  0000 C CNN
-F 3 "" H 5700 5450 60  0000 C CNN
-	1    5700 5450
-	1    0    0    -1
-$EndComp
 $Comp
 L CONN_4 P1
@@
 	3950 4900 3800 4900
 Wire Wire Line
-	5500 6250 5500 6150
-Wire Wire Line
-	5500 5650 5500 5450
-Wire Wire Line
-	5700 5650 5700 5450
-Wire Wire Line
 	5200 6400 5700 6400
-Connection ~ 5500 6250
 Wire Wire Line
 	5200 6250 6300 6250
 Wire Wire Line
-	5700 6400 5700 6150
-Wire Wire Line
 	5700 6350 6300 6350
-Connection ~ 5700 6350
-$Comp
-L 3V3 #PWR17
+$Comp
+L 3V3 #PWR021
 U 1 1 546AB46C
 P 6200 6150
-F 0 "#PWR17" H 6200 6250 40  0001 C CNN
+F 0 "#PWR021" H 6200 6250 40  0001 C CNN
 F 1 "3V3" H 6200 6275 40  0000 C CNN
 F 2 "" H 6200 6150 60  0000 C CNN
@@
 	6200 6450 6200 6150
 $Comp
-L GND #PWR18
+L GND #PWR022
 U 1 1 546AB4C5
 P 6200 6700
-F 0 "#PWR18" H 6200 6700 30  0001 C CNN
+F 0 "#PWR022" H 6200 6700 30  0001 C CNN
 F 1 "GND" H 6200 6630 30  0001 C CNN
 F 2 "" H 6200 6700 60  0000 C CNN
@@
 $EndComp
 $Comp
-L 3V3 #PWR13
+L 3V3 #PWR023
 U 1 1 54727DD2
 P 4450 1250
-F 0 "#PWR13" H 4450 1350 40  0001 C CNN
+F 0 "#PWR023" H 4450 1350 40  0001 C CNN
 F 1 "3V3" H 4450 1375 40  0000 C CNN
 F 2 "" H 4450 1250 60  0000 C CNN
@@
 $EndComp
 $Comp
-L 3V3 #PWR4
+L 3V3 #PWR024
 U 1 1 54727DDE
 P 1950 850
-F 0 "#PWR4" H 1950 950 40  0001 C CNN
+F 0 "#PWR024" H 1950 950 40  0001 C CNN
 F 1 "3V3" H 1950 975 40  0000 C CNN
 F 2 "" H 1950 850 60  0000 C CNN
@@
 	2650 3650 2650 3250
 Connection ~ 2650 3250
+Wire Wire Line
+	5700 6400 5700 6350
 $EndSCHEMATC
