File: board/mainboard/i2c_peripherals.sch (KiCad schematic (older format))
At the start: 17 parts, among them P1 I2C, P2 Motor1, P3 Motor2, X1 32.768KHz

Commit message: Rebuilt power section to support switching, new buck converter for 3V3 net.
Parts:
- removed P2: Motor1, symbol CONN_2
- added P2: CONN_01X02, symbol CONN_01X02
- P1: symbol CONN_4 -> CONN_01X04
- P3: symbol CONN_2 -> CONN_01X02
Connections:
- wire segments 84 -> 93
Changed lines of the file:
@@
 LIBS:valves
 LIBS:mainboard-cache
-EELAYER 27 0
+EELAYER 25 0
 EELAYER END
 $Descr A4 11693 8268
@@
 I2C_DA
 $Comp
-L CONN_4 P1
+L CONN_01X04 P1
 U 1 1 546AB17E
 P 6650 6400
@@
 	5200 6400 5700 6400
 Wire Wire Line
-	5200 6250 6300 6250
-Wire Wire Line
-	5700 6350 6300 6350
+	5200 6250 6450 6250
+Wire Wire Line
+	5700 6350 6450 6350
 $Comp
 L 3V3 #PWR15
@@
 $EndComp
 Wire Wire Line
-	6300 6450 6200 6450
+	6200 6450 6450 6450
 Wire Wire Line
 	6200 6450 6200 6150
@@
 	6200 6700 6200 6550
 Wire Wire Line
-	6200 6550 6300 6550
+	6200 6550 6450 6550
 Text GLabel 9150 6250 0    60   Input ~ 0
 MOTOR1-
@@
 	4450 1950 4450 2100
 Connection ~ 4450 2100
-$Comp
-L CONN_2 P2
-U 1 1 5472816B
-P 9650 6150
-F 0 "P2" V 9600 6150 40  0000 C CNN
-F 1 "Motor1" V 9700 6150 40  0000 C CNN
-F 2 "" H 9650 6150 60  0000 C CNN
-F 3 "" H 9650 6150 60  0000 C CNN
-	1    9650 6150
-	1    0    0    -1
-$EndComp
 Wire Wire Line
 	9150 6050 9300 6050
@@
 	9150 6250 9300 6250
 $Comp
-L CONN_2 P3
+L CONN_01X02 P3
 U 1 1 54728242
 P 9650 6650
@@
 Wire Wire Line
 	8150 3800 7950 3800
+$Comp
+L CONN_01X02 P2
+U 1 1 55A1DE1A
+P 9600 6150
+F 0 "P2" H 9600 6300 50  0000 C CNN
+F 1 "CONN_01X02" V 9700 6150 50  0000 C CNN
+F 2 "" H 9600 6150 60  0000 C CNN
+F 3 "" H 9600 6150 60  0000 C CNN
+	1    9600 6150
+	1    0    0    -1
+$EndComp
+Wire Wire Line
+	9400 6100 9300 6100
+Wire Wire Line
+	9300 6100 9300 6050
+Wire Wire Line
+	9400 6200 9300 6200
+Wire Wire Line
+	9300 6200 9300 6250
+Wire Wire Line
+	9450 6550 9450 6600
+Wire Wire Line
+	9300 6550 9300 6600
+Wire Wire Line
+	9300 6600 9450 6600
+Wire Wire Line
+	9300 6750 9300 6700
+Wire Wire Line
+	9300 6700 9450 6700
 $EndSCHEMATC
