File: board/mainboard/BusSplitter.sch (KiCad schematic (older format))
At the start: 21 parts

Commit message: Added I2C transceiver
Parts:
- removed R? (x2): 47K, ~, symbol R
- removed U?: 74LS244, ~, symbol 74LS244
- added U?: PCA9515B, symbol PCA9515B
Connections:
- wire segments 69 -> 63

Commit message: Replaced cc3200 bus isolation with jumpers
Parts:
- removed R?: 47K, ~, symbol R
- removed U? (x8): 74ALVC125, ~, symbol 74LS125
- added P?: CC_ISO, symbol CONN_10X2
Connections:
- wire segments 63 -> 87

Commit message: Connected GLCD_A0 to Launchpad and buffered it
Parts:
- added U?: 74ALVC126, ~, symbol 74LS126
Connections:
- net labels added: GPIO_A0, GPIO_A0_LP
- wire segments 87 -> 90
Changed lines of the file:
@@
 $Descr A4 11693 8268
 encoding utf-8
-Sheet 6 6
+Sheet 6 7
 Title ""
 Date "23 nov 2014"
@@
 Wire Wire Line
 	7900 5450 8050 5450
-Wire Wire Line
-	2250 1350 2250 6050
 Connection ~ 2250 1750
 $Comp
@@
 Wire Wire Line
 	8950 3100 8750 3100
+Text GLabel 2000 6850 0    60   Input ~ 0
+GPIO_A0_LP
+Text GLabel 3600 6850 2    60   Input ~ 0
+GPIO_A0
+Wire Wire Line
+	3600 6850 3350 6850
+Wire Wire Line
+	2000 6850 2450 6850
+$Comp
+L 74LS126 U?
+U 1 1 547262C6
+P 2900 6850
+F 0 "U?" H 3000 7050 60  0000 C CNN
+F 1 "74ALVC126" H 3150 6700 60  0000 C CNN
+F 2 "~" H 2900 6850 60  0000 C CNN
+F 3 "~" H 2900 6850 60  0000 C CNN
+	1    2900 6850
+	1    0    0    -1
+$EndComp
+Wire Wire Line
+	2250 7150 2900 7150
+Wire Wire Line
+	2250 7150 2250 1350
 $EndSCHEMATC
