File: board/mainboard/BusSplitter.sch (KiCad schematic (older format))
At the start: 12 parts

Commit message: Added net names, fixed misnamed GLCD_A0
Parts:
- gave numbers to parts that had none: 6
Connections:
- net labels added: GLCD_A0, GLCD_A0_LP
- net labels removed: GPIO_A0, GPIO_A0_LP
Changed lines of the file:
@@
 CC_CONTROL
 $Comp
-L R R?
+L R R27
 U 1 1 54722583
 P 2250 1100
-F 0 "R?" V 2330 1100 40  0000 C CNN
+F 0 "R27" V 2330 1100 40  0000 C CNN
 F 1 "47K" V 2257 1101 40  0000 C CNN
 F 2 "~" V 2180 1100 30  0000 C CNN
@@
 UART_TX
 $Comp
-L 74LS126 U?
+L 74LS126 U3
 U 1 1 54722780
 P 2900 1450
-F 0 "U?" H 3000 1650 60  0000 C CNN
+F 0 "U3" H 3000 1650 60  0000 C CNN
 F 1 "74ALVC126" H 3150 1300 60  0000 C CNN
 F 2 "~" H 2900 1450 60  0000 C CNN
@@
 $EndComp
 $Comp
-L 74LS126 U?
-U 1 1 5472278D
+L 74LS126 U3
+U 2 1 5472278D
 P 2900 2050
-F 0 "U?" H 3000 2250 60  0000 C CNN
+F 0 "U3" H 3000 2250 60  0000 C CNN
 F 1 "74ALVC126" H 3150 1900 60  0000 C CNN
 F 2 "~" H 2900 2050 60  0000 C CNN
 F 3 "~" H 2900 2050 60  0000 C CNN
-	1    2900 2050
-	1    0    0    -1
-$EndComp
-$Comp
-L 74LS126 U?
+	2    2900 2050
+	1    0    0    -1
+$EndComp
+$Comp
+L 74LS126 U4
 U 1 1 547227AB
 P 2900 4000
-F 0 "U?" H 3000 4200 60  0000 C CNN
+F 0 "U4" H 3000 4200 60  0000 C CNN
 F 1 "74ALVC126" H 3150 3850 60  0000 C CNN
 F 2 "~" H 2900 4000 60  0000 C CNN
@@
 $EndComp
 $Comp
-L 74LS126 U?
-U 1 1 547227B1
+L 74LS126 U4
+U 2 1 547227B1
 P 2900 4600
-F 0 "U?" H 3000 4800 60  0000 C CNN
+F 0 "U4" H 3000 4800 60  0000 C CNN
 F 1 "74ALVC126" H 3150 4450 60  0000 C CNN
 F 2 "~" H 2900 4600 60  0000 C CNN
 F 3 "~" H 2900 4600 60  0000 C CNN
-	1    2900 4600
-	1    0    0    -1
-$EndComp
-$Comp
-L 74LS126 U?
-U 1 1 547227B7
+	2    2900 4600
+	1    0    0    -1
+$EndComp
+$Comp
+L 74LS126 U4
+U 3 1 547227B7
 P 2900 5150
-F 0 "U?" H 3000 5350 60  0000 C CNN
+F 0 "U4" H 3000 5350 60  0000 C CNN
 F 1 "74ALVC126" H 3150 5000 60  0000 C CNN
 F 2 "~" H 2900 5150 60  0000 C CNN
 F 3 "~" H 2900 5150 60  0000 C CNN
-	1    2900 5150
-	1    0    0    -1
-$EndComp
-$Comp
-L 74LS126 U?
-U 1 1 547227BD
+	3    2900 5150
+	1    0    0    -1
+$EndComp
+$Comp
+L 74LS126 U4
+U 4 1 547227BD
 P 2900 5750
-F 0 "U?" H 3000 5950 60  0000 C CNN
+F 0 "U4" H 3000 5950 60  0000 C CNN
 F 1 "74ALVC126" H 3150 5600 60  0000 C CNN
 F 2 "~" H 2900 5750 60  0000 C CNN
 F 3 "~" H 2900 5750 60  0000 C CNN
-	1    2900 5750
-	1    0    0    -1
-$EndComp
-$Comp
-L 74LS126 U?
-U 1 1 547227D5
+	4    2900 5750
+	1    0    0    -1
+$EndComp
+$Comp
+L 74LS126 U3
+U 3 1 547227D5
 P 2900 2600
-F 0 "U?" H 3000 2800 60  0000 C CNN
+F 0 "U3" H 3000 2800 60  0000 C CNN
 F 1 "74ALVC126" H 3150 2450 60  0000 C CNN
 F 2 "~" H 2900 2600 60  0000 C CNN
 F 3 "~" H 2900 2600 60  0000 C CNN
-	1    2900 2600
+	3    2900 2600
 	-1   0    0    -1
 $EndComp
 $Comp
-L 74LS126 U?
-U 1 1 547227DB
+L 74LS126 U3
+U 4 1 547227DB
 P 2900 3150
-F 0 "U?" H 3000 3350 60  0000 C CNN
+F 0 "U3" H 3000 3350 60  0000 C CNN
 F 1 "74ALVC126" H 3150 3000 60  0000 C CNN
 F 2 "~" H 2900 3150 60  0000 C CNN
 F 3 "~" H 2900 3150 60  0000 C CNN
-	1    2900 3150
+	4    2900 3150
 	-1   0    0    -1
 $EndComp
@@
 I2C_CL
 $Comp
-L PCA9515B U?
+L PCA9515B U6
 U 1 1 54723DAE
 P 8500 5300
-F 0 "U?" H 8500 5350 60  0000 C CNN
+F 0 "U6" H 8500 5350 60  0000 C CNN
 F 1 "PCA9515B" H 8500 5700 60  0000 C CNN
 F 2 "" H 8500 5700 60  0000 C CNN
@@
 $EndComp
 $Comp
-L 3V3 #PWR?
+L 3V3 #PWR059
 U 1 1 54723DBD
 P 7950 4900
-F 0 "#PWR?" H 7950 5000 40  0001 C CNN
+F 0 "#PWR059" H 7950 5000 40  0001 C CNN
 F 1 "3V3" H 7950 5025 40  0000 C CNN
 F 2 "" H 7950 4900 60  0000 C CNN
@@
 	7950 5350 8050 5350
 $Comp
-L GND #PWR?
+L GND #PWR060
 U 1 1 54723E16
 P 7950 5700
-F 0 "#PWR?" H 7950 5700 30  0001 C CNN
+F 0 "#PWR060" H 7950 5700 30  0001 C CNN
 F 1 "GND" H 7950 5630 30  0001 C CNN
 F 2 "" H 7950 5700 60  0000 C CNN
@@
 Connection ~ 2250 1750
 $Comp
-L 3V3 #PWR?
+L 3V3 #PWR061
 U 1 1 54723FF2
 P 2250 750
-F 0 "#PWR?" H 2250 850 40  0001 C CNN
+F 0 "#PWR061" H 2250 850 40  0001 C CNN
 F 1 "3V3" H 2250 875 40  0000 C CNN
 F 2 "" H 2250 750 60  0000 C CNN
@@
 	2250 850  2250 750
 $Comp
-L CONN_10X2 P?
+L CONN_10X2 P11
 U 1 1 547257ED
 P 8350 3150
-F 0 "P?" H 8350 3700 60  0000 C CNN
+F 0 "P11" H 8350 3700 60  0000 C CNN
 F 1 "CC_ISO" V 8350 3050 50  0000 C CNN
 F 2 "" H 8350 3150 60  0000 C CNN
@@
 	8950 3100 8750 3100
 Text GLabel 2000 6850 0    60   Input ~ 0
-GPIO_A0_LP
+GLCD_A0_LP
 Text GLabel 3600 6850 2    60   Input ~ 0
-GPIO_A0
+GLCD_A0
 Wire Wire Line
 	3600 6850 3350 6850
@@
 	2000 6850 2450 6850
 $Comp
-L 74LS126 U?
+L 74LS126 U5
 U 1 1 547262C6
 P 2900 6850
-F 0 "U?" H 3000 7050 60  0000 C CNN
+F 0 "U5" H 3000 7050 60  0000 C CNN
 F 1 "74ALVC126" H 3150 6700 60  0000 C CNN
 F 2 "~" H 2900 6850 60  0000 C CNN

Commit message: Finished first draft of rev 1 board
Parts:
- removed P11: CC_ISO, symbol CONN_10X2
Connections:
- wire segments 90 -> 84
Changed lines of the file:
@@
 $Descr A4 11693 8268
 encoding utf-8
-Sheet 6 7
+Sheet 6 8
 Title ""
-Date "24 nov 2014"
+Date "25 nov 2014"
 Rev ""
 Comp ""
@@
 $EndComp
 $Comp
-L 3V3 #PWR059
+L 3V3 #PWR060
 U 1 1 54723DBD
 P 7950 4900
-F 0 "#PWR059" H 7950 5000 40  0001 C CNN
+F 0 "#PWR060" H 7950 5000 40  0001 C CNN
 F 1 "3V3" H 7950 5025 40  0000 C CNN
 F 2 "" H 7950 4900 60  0000 C CNN
@@
 	7950 5350 8050 5350
 $Comp
-L GND #PWR060
+L GND #PWR061
 U 1 1 54723E16
 P 7950 5700
-F 0 "#PWR060" H 7950 5700 30  0001 C CNN
+F 0 "#PWR061" H 7950 5700 30  0001 C CNN
 F 1 "GND" H 7950 5630 30  0001 C CNN
 F 2 "" H 7950 5700 60  0000 C CNN
@@
 Connection ~ 2250 1750
 $Comp
-L 3V3 #PWR061
+L 3V3 #PWR062
 U 1 1 54723FF2
 P 2250 750
-F 0 "#PWR061" H 2250 850 40  0001 C CNN
+F 0 "#PWR062" H 2250 850 40  0001 C CNN
 F 1 "3V3" H 2250 875 40  0000 C CNN
 F 2 "" H 2250 750 60  0000 C CNN
@@
 Wire Wire Line
 	2250 850  2250 750
-$Comp
-L CONN_10X2 P11
-U 1 1 547257ED
-P 8350 3150
-F 0 "P11" H 8350 3700 60  0000 C CNN
-F 1 "CC_ISO" V 8350 3050 50  0000 C CNN
-F 2 "" H 8350 3150 60  0000 C CNN
-F 3 "" H 8350 3150 60  0000 C CNN
-	1    8350 3150
-	1    0    0    -1
-$EndComp
 Wire Wire Line
 	7550 2450 7950 2450
@@
 	7900 2600 7900 2800
 Wire Wire Line
-	7900 2800 7950 2800
+	7900 2800 8800 2800
 Wire Wire Line
 	7550 2750 7850 2750
@@
 	7850 2750 7850 2900
 Wire Wire Line
-	7850 2900 7950 2900
+	7850 2900 8850 2900
 Wire Wire Line
 	7550 2900 7800 2900
@@
 	7800 2900 7800 3000
 Wire Wire Line
-	7800 3000 7950 3000
-Wire Wire Line
-	7550 3200 7950 3200
+	7800 3000 8900 3000
+Wire Wire Line
+	7550 3200 9200 3200
 Wire Wire Line
 	7550 3050 7750 3050
@@
 	7750 3050 7750 3100
 Wire Wire Line
-	7750 3100 7950 3100
+	7750 3100 8950 3100
 Wire Wire Line
 	7550 3800 7950 3800
@@
 	7900 3650 7900 3500
 Wire Wire Line
-	7900 3500 7950 3500
+	7900 3500 8800 3500
 Wire Wire Line
 	7550 3500 7850 3500
@@
 	7850 3500 7850 3400
 Wire Wire Line
-	7850 3400 7950 3400
+	7850 3400 8850 3400
 Wire Wire Line
 	7550 3350 7800 3350
@@
 	7800 3350 7800 3300
 Wire Wire Line
-	7800 3300 7950 3300
+	7800 3300 8900 3300
 Wire Wire Line
 	9200 3800 8750 3800
@@
 	8800 3650 8800 3500
 Wire Wire Line
-	8800 3500 8750 3500
-Wire Wire Line
 	9200 3500 8850 3500
 Wire Wire Line
 	8850 3500 8850 3400
 Wire Wire Line
-	8850 3400 8750 3400
-Wire Wire Line
 	9200 3350 8900 3350
 Wire Wire Line
 	8900 3350 8900 3300
 Wire Wire Line
-	8900 3300 8750 3300
-Wire Wire Line
-	9200 3200 8750 3200
-Wire Wire Line
 	9200 2450 8750 2450
 Wire Wire Line
@@
 	8800 2600 8800 2800
 Wire Wire Line
-	8800 2800 8750 2800
-Wire Wire Line
 	9200 2750 8850 2750
 Wire Wire Line
 	8850 2750 8850 2900
 Wire Wire Line
-	8850 2900 8750 2900
-Wire Wire Line
 	9200 2900 8900 2900
 Wire Wire Line
 	8900 2900 8900 3000
 Wire Wire Line
-	8900 3000 8750 3000
-Wire Wire Line
 	9200 3050 8950 3050
 Wire Wire Line
 	8950 3050 8950 3100
-Wire Wire Line
-	8950 3100 8750 3100
 Text GLabel 2000 6850 0    60   Input ~ 0
 GLCD_A0_LP
@@
 Wire Wire Line
 	2250 7150 2250 1350
+Wire Wire Line
+	8750 2700 7950 2700
+Wire Wire Line
+	8750 3600 7950 3600
 $EndSCHEMATC

Commit message: Replaced buffers with CPLD
Parts:
- removed R27: 47K, ~, symbol R
- removed U3, U4, U5: 74ALVC126, ~, symbol 74LS126
- added U?: XC2C32A, ~, symbol XC2C32A
Connections:
- net labels added: 1V8, CPLD_TCK, CPLD_TDI, CPLD_TDO, CPLD_TMS, SPI_CS1, SPI_CS2, SPI_CS3, SPI_CS4, SPI_CS5, SPI_CS6, SPI_CS7, SPI_CS_CC
- net labels removed: SPI_SEL0, SPI_SEL1, SPI_SEL2
- wire segments 84 -> 117
- no-connect marks 0 -> 5

Commit message: Various fixes to schematics and footprints:
* Added pullup resistors to bumpers
* Changed value of RLED resistor
* Added resistor to GLED
* Changed SPI pullup resistors to 47k
* Added JTAG header for CPLD
* Changed motor driver footprint to MSOP
Parts:
- added P?: CPLD_JTAG, symbol CONN_6
- gave numbers to parts that had none: 1
Connections:
- wire segments 117 -> 128
Changed lines of the file:
@@
 $EndComp
 $Comp
-L 3V3 #PWR053
+L 3V3 #PWR051
 U 1 1 54723DBD
 P 7950 4900
-F 0 "#PWR053" H 7950 5000 40  0001 C CNN
+F 0 "#PWR051" H 7950 5000 40  0001 C CNN
 F 1 "3V3" H 7950 5025 40  0000 C CNN
 F 2 "" H 7950 4900 60  0000 C CNN
@@
 	7950 5350 8050 5350
 $Comp
-L GND #PWR054
+L GND #PWR052
 U 1 1 54723E16
 P 7950 5700
-F 0 "#PWR054" H 7950 5700 30  0001 C CNN
+F 0 "#PWR052" H 7950 5700 30  0001 C CNN
 F 1 "GND" H 7950 5630 30  0001 C CNN
 F 2 "" H 7950 5700 60  0000 C CNN
@@
 	8250 3150 8550 3150
 $Comp
-L XC2C32A U?
+L XC2C32A U1
 U 1 1 54DD81D8
 P 4000 4150
-F 0 "U?" H 4000 4150 60  0000 C CNN
+F 0 "U1" H 4000 4150 60  0000 C CNN
 F 1 "XC2C32A" H 4000 5400 60  0000 C CNN
 F 2 "~" H 4000 4800 60  0000 C CNN
@@
 	4900 5000 4800 5000
 $Comp
-L 3V3 #PWR?
+L 3V3 #PWR053
 U 1 1 54DD88EA
 P 4850 2750
-F 0 "#PWR?" H 4850 2850 40  0001 C CNN
+F 0 "#PWR053" H 4850 2850 40  0001 C CNN
 F 1 "3V3" H 4850 2875 40  0000 C CNN
 F 2 "" H 4850 2750 60  0000 C CNN
@@
 	4850 4300 4800 4300
 Wire Wire Line
-	4850 2750 4850 2800
-Wire Wire Line
-	4850 2800 4850 3400
-Wire Wire Line
-	4850 3400 4850 4300
+	4850 2750 4850 4300
 Wire Wire Line
 	4800 3400 4850 3400
 Connection ~ 4850 3400
 $Comp
-L GND #PWR?
+L GND #PWR054
 U 1 1 54DD89FD
 P 6100 3500
-F 0 "#PWR?" H 6100 3500 30  0001 C CNN
+F 0 "#PWR054" H 6100 3500 30  0001 C CNN
 F 1 "GND" H 6100 3430 30  0001 C CNN
 F 2 "" H 6100 3500 60  0000 C CNN
@@
 	2850 3400 3200 3400
 $Comp
-L GND #PWR?
+L GND #PWR055
 U 1 1 54DD8C2C
 P 1950 4950
-F 0 "#PWR?" H 1950 4950 30  0001 C CNN
+F 0 "#PWR055" H 1950 4950 30  0001 C CNN
 F 1 "GND" H 1950 4880 30  0001 C CNN
 F 2 "" H 1950 4950 60  0000 C CNN
@@
 	1950 4850 1950 4950
 $Comp
-L 1V8 #PWR?
+L 1V8 #PWR056
 U 1 1 54DD8CFA
 P 1950 4550
-F 0 "#PWR?" H 1950 4690 20  0001 C CNN
+F 0 "#PWR056" H 1950 4690 20  0001 C CNN
 F 1 "1V8" H 1950 4660 30  0000 C CNN
 F 2 "" H 1950 4550 60  0000 C CNN
@@
 	2850 4700 3200 4700
 Wire Wire Line
-	2850 3400 2850 4700
-Wire Wire Line
-	2850 4700 2850 4850
+	2850 3400 2850 4850
 Wire Wire Line
 	2850 4850 1950 4850
@@
 Wire Wire Line
 	8250 3000 8550 3000
+Text GLabel 5950 1400 0    60   Input ~ 0
+CPLD_TDO
+Text GLabel 5950 1550 0    60   Input ~ 0
+CPLD_TDI
+Text GLabel 5950 1700 0    60   Input ~ 0
+CPLD_TMS
+Text GLabel 5950 1250 0    60   Input ~ 0
+CPLD_TCK
+$Comp
+L CONN_6 P?
+U 1 1 54DE1CE8
+P 6800 1450
+F 0 "P?" V 6750 1450 60  0000 C CNN
+F 1 "CPLD_JTAG" V 6850 1450 60  0000 C CNN
+F 2 "" H 6800 1450 60  0000 C CNN
+F 3 "" H 6800 1450 60  0000 C CNN
+	1    6800 1450
+	1    0    0    -1
+$EndComp
+Wire Wire Line
+	5950 1700 6450 1700
+Wire Wire Line
+	5950 1550 6050 1550
+Wire Wire Line
+	6050 1550 6050 1600
+Wire Wire Line
+	6050 1600 6450 1600
+Wire Wire Line
+	5950 1400 6100 1400
+Wire Wire Line
+	6100 1400 6100 1500
+Wire Wire Line
+	6100 1500 6450 1500
+Wire Wire Line
+	5950 1250 6150 1250
+Wire Wire Line
+	6150 1250 6150 1400
+Wire Wire Line
+	6150 1400 6450 1400
+$Comp
+L GND #PWR?
+U 1 1 54DE1EE6
+P 6400 1950
+F 0 "#PWR?" H 6400 1950 30  0001 C CNN
+F 1 "GND" H 6400 1880 30  0001 C CNN
+F 2 "" H 6400 1950 60  0000 C CNN
+F 3 "" H 6400 1950 60  0000 C CNN
+	1    6400 1950
+	1    0    0    -1
+$EndComp
+Wire Wire Line
+	6400 1950 6400 1300
+Wire Wire Line
+	6400 1300 6450 1300
+$Comp
+L 3V3 #PWR?
+U 1 1 54DE1F75
+P 6400 900
+F 0 "#PWR?" H 6400 1000 40  0001 C CNN
+F 1 "3V3" H 6400 1025 40  0000 C CNN
+F 2 "" H 6400 900 60  0000 C CNN
+F 3 "" H 6400 900 60  0000 C CNN
+	1    6400 900
+	1    0    0    -1
+$EndComp
+Wire Wire Line
+	6450 1200 6400 1200
+Wire Wire Line
+	6400 1200 6400 900
 $EndSCHEMATC

Commit message: Added power LED, removed Codec Peripheral pin
Parts:
- gave numbers to parts that had none: 1
Changed lines of the file:
@@
 Sheet 5 7
 Title ""
-Date "13 feb 2015"
+Date "16 feb 2015"
 Rev ""
 Comp ""
@@
 $EndComp
 $Comp
-L 3V3 #PWR051
+L 3V3 #PWR60
 U 1 1 54723DBD
 P 7950 4900
-F 0 "#PWR051" H 7950 5000 40  0001 C CNN
+F 0 "#PWR60" H 7950 5000 40  0001 C CNN
 F 1 "3V3" H 7950 5025 40  0000 C CNN
 F 2 "" H 7950 4900 60  0000 C CNN
@@
 	7950 5350 8050 5350
 $Comp
-L GND #PWR052
+L GND #PWR61
 U 1 1 54723E16
 P 7950 5700
-F 0 "#PWR052" H 7950 5700 30  0001 C CNN
+F 0 "#PWR61" H 7950 5700 30  0001 C CNN
 F 1 "GND" H 7950 5630 30  0001 C CNN
 F 2 "" H 7950 5700 60  0000 C CNN
@@
 	4900 5000 4800 5000
 $Comp
-L 3V3 #PWR053
+L 3V3 #PWR56
 U 1 1 54DD88EA
 P 4850 2750
-F 0 "#PWR053" H 4850 2850 40  0001 C CNN
+F 0 "#PWR56" H 4850 2850 40  0001 C CNN
 F 1 "3V3" H 4850 2875 40  0000 C CNN
 F 2 "" H 4850 2750 60  0000 C CNN
@@
 Connection ~ 4850 3400
 $Comp
-L GND #PWR054
+L GND #PWR57
 U 1 1 54DD89FD
 P 6100 3500
-F 0 "#PWR054" H 6100 3500 30  0001 C CNN
+F 0 "#PWR57" H 6100 3500 30  0001 C CNN
 F 1 "GND" H 6100 3430 30  0001 C CNN
 F 2 "" H 6100 3500 60  0000 C CNN
@@
 	2850 3400 3200 3400
 $Comp
-L GND #PWR055
+L GND #PWR55
 U 1 1 54DD8C2C
 P 1950 4950
-F 0 "#PWR055" H 1950 4950 30  0001 C CNN
+F 0 "#PWR55" H 1950 4950 30  0001 C CNN
 F 1 "GND" H 1950 4880 30  0001 C CNN
 F 2 "" H 1950 4950 60  0000 C CNN
@@
 	1950 4850 1950 4950
 $Comp
-L 1V8 #PWR056
+L 1V8 #PWR54
 U 1 1 54DD8CFA
 P 1950 4550
-F 0 "#PWR056" H 1950 4690 20  0001 C CNN
+F 0 "#PWR54" H 1950 4690 20  0001 C CNN
 F 1 "1V8" H 1950 4660 30  0000 C CNN
 F 2 "" H 1950 4550 60  0000 C CNN
@@
 CPLD_TCK
 $Comp
-L CONN_6 P?
+L CONN_6 P11
 U 1 1 54DE1CE8
 P 6800 1450
-F 0 "P?" V 6750 1450 60  0000 C CNN
+F 0 "P11" V 6750 1450 60  0000 C CNN
 F 1 "CPLD_JTAG" V 6850 1450 60  0000 C CNN
 F 2 "" H 6800 1450 60  0000 C CNN
@@
 	6150 1400 6450 1400
 $Comp
-L GND #PWR?
+L GND #PWR59
 U 1 1 54DE1EE6
 P 6400 1950
-F 0 "#PWR?" H 6400 1950 30  0001 C CNN
+F 0 "#PWR59" H 6400 1950 30  0001 C CNN
 F 1 "GND" H 6400 1880 30  0001 C CNN
 F 2 "" H 6400 1950 60  0000 C CNN
@@
 	6400 1300 6450 1300
 $Comp
-L 3V3 #PWR?
+L 3V3 #PWR58
 U 1 1 54DE1F75
 P 6400 900
-F 0 "#PWR?" H 6400 1000 40  0001 C CNN
+F 0 "#PWR58" H 6400 1000 40  0001 C CNN
 F 1 "3V3" H 6400 1025 40  0000 C CNN
 F 2 "" H 6400 900 60  0000 C CNN

Commit message: Various changes
* Began Rev2 Layout
* Added Pullup Resistors to LP I2C
* Added IrDA Module
Parts:
- added R22, R23, R3, R4: 4.7k, ~, symbol R
Connections:
- wire segments 128 -> 142
- no-connect marks 5 -> 6

Commit message: Further work on the rev2 layout
Changed lines of the file:
@@
 Text GLabel 2750 4500 0    60   Input ~ 0
 UART_TX_LP
-Text GLabel 5250 3400 2    60   Input ~ 0
+Text GLabel 5250 4300 2    60   Input ~ 0
 SPI_SCK
-Text GLabel 5250 3550 2    60   Input ~ 0
+Text GLabel 5250 4150 2    60   Input ~ 0
 SPI_MOSI
-Text GLabel 5250 3700 2    60   Input ~ 0
+Text GLabel 5250 4000 2    60   Input ~ 0
 SPI_MISO
 Text GLabel 5250 5500 2    60   Input ~ 0
@@
 Text GLabel 5250 5650 2    60   Input ~ 0
 UART_TX
-Text GLabel 5250 4300 2    60   Input ~ 0
+Text GLabel 5250 3850 2    60   Input ~ 0
 CC_CONTROL
 Text GLabel 8250 3450 0    60   Input ~ 0
@@
 Text GLabel 8250 3750 0    60   Input ~ 0
 SPI_MISO_CC
-Text GLabel 5250 3850 2    60   Input ~ 0
+Text GLabel 5250 3400 2    60   Input ~ 0
 SPI_SEL0_CC
-Text GLabel 5250 4000 2    60   Input ~ 0
+Text GLabel 5250 3550 2    60   Input ~ 0
 SPI_SEL1_CC
-Text GLabel 5250 4150 2    60   Input ~ 0
+Text GLabel 5250 3700 2    60   Input ~ 0
 SPI_SEL2_CC
 Text GLabel 8250 3900 0    60   Input ~ 0
