File: board/mainboard/BusSplitter.sch (KiCad schematic (older format))
At the start: 7 parts, among them P11 CPLD_JTAG, U1 XC2C32A, U6 PCA9515B

Commit message: Finished draft 1 of Rev 2 layout
Connections:
- wire segments 142 -> 138
- no-connect marks 6 -> 7
Changed lines of the file:
@@
 $Descr A4 11693 8268
 encoding utf-8
-Sheet 5 7
+Sheet 5 8
 Title ""
-Date "26 feb 2015"
+Date "1 mar 2015"
 Rev ""
 Comp ""
@@
 Text GLabel 2750 4200 0    60   Input ~ 0
 CPLD_TCK
-NoConn ~ 4500 6000
 NoConn ~ 3200 3800
 NoConn ~ 3200 4800
@@
 	2950 3500 3200 3500
 Wire Wire Line
-	2900 5200 3200 5200
-Wire Wire Line
-	3200 5100 2950 5100
-Wire Wire Line
-	2950 5100 2950 5050
-Wire Wire Line
-	2950 5050 2900 5050
-Wire Wire Line
 	4800 3700 5250 3700
 Wire Wire Line
@@
 Wire Wire Line
 	4850 5100 4800 5100
+NoConn ~ 3200 5200
+NoConn ~ 3200 5100
 $EndSCHEMATC

Commit message: fixed DRC errors on schematic
Connections:
- no-connect marks 7 -> 8
Changed lines of the file:
@@
 Sheet 5 8
 Title ""
-Date "1 mar 2015"
+Date "2 mar 2015"
 Rev ""
 Comp ""
@@
 NoConn ~ 3200 5200
 NoConn ~ 3200 5100
+NoConn ~ 3200 4600
 $EndSCHEMATC

Commit message: Rebuilt power section to support switching, new buck converter for 3V3 net.
Parts:
- P11: symbol CONN_6 -> CONN_01X06
Changed lines of the file:
@@
 LIBS:valves
 LIBS:mainboard-cache
-EELAYER 27 0
+EELAYER 25 0
 EELAYER END
 $Descr A4 11693 8268
@@
 $EndComp
 $Comp
-L 3V3 #PWR69
+L 3V3 #PWR66
 U 1 1 54723DBD
 P 7950 4900
-F 0 "#PWR69" H 7950 5000 40  0001 C CNN
+F 0 "#PWR66" H 7950 5000 40  0001 C CNN
 F 1 "3V3" H 7950 5025 40  0000 C CNN
 F 2 "" H 7950 4900 60  0000 C CNN
@@
 $EndComp
 $Comp
-L GND #PWR70
+L GND #PWR67
 U 1 1 54723E16
 P 7950 5700
-F 0 "#PWR70" H 7950 5700 30  0001 C CNN
+F 0 "#PWR67" H 7950 5700 30  0001 C CNN
 F 1 "GND" H 7950 5630 30  0001 C CNN
 F 2 "" H 7950 5700 60  0000 C CNN
@@
 $EndComp
 $Comp
-L 3V3 #PWR63
+L 3V3 #PWR60
 U 1 1 54DD88EA
 P 4850 2750
-F 0 "#PWR63" H 4850 2850 40  0001 C CNN
+F 0 "#PWR60" H 4850 2850 40  0001 C CNN
 F 1 "3V3" H 4850 2875 40  0000 C CNN
 F 2 "" H 4850 2750 60  0000 C CNN
@@
 $EndComp
 $Comp
-L GND #PWR64
+L GND #PWR61
 U 1 1 54DD89FD
 P 6100 3500
-F 0 "#PWR64" H 6100 3500 30  0001 C CNN
+F 0 "#PWR61" H 6100 3500 30  0001 C CNN
 F 1 "GND" H 6100 3430 30  0001 C CNN
 F 2 "" H 6100 3500 60  0000 C CNN
@@
 $EndComp
 $Comp
-L GND #PWR62
+L GND #PWR59
 U 1 1 54DD8C2C
 P 1950 4950
-F 0 "#PWR62" H 1950 4950 30  0001 C CNN
+F 0 "#PWR59" H 1950 4950 30  0001 C CNN
 F 1 "GND" H 1950 4880 30  0001 C CNN
 F 2 "" H 1950 4950 60  0000 C CNN
@@
 $EndComp
 $Comp
-L 1V8 #PWR61
+L 1V8 #PWR58
 U 1 1 54DD8CFA
 P 1950 4550
-F 0 "#PWR61" H 1950 4690 20  0001 C CNN
+F 0 "#PWR58" H 1950 4690 20  0001 C CNN
 F 1 "1V8" H 1950 4660 30  0000 C CNN
 F 2 "" H 1950 4550 60  0000 C CNN
@@
 CPLD_TCK
 $Comp
-L CONN_6 P11
+L CONN_01X06 P11
 U 1 1 54DE1CE8
 P 6800 1450
@@
 $EndComp
 $Comp
-L GND #PWR66
+L GND #PWR63
 U 1 1 54DE1EE6
 P 6400 1950
-F 0 "#PWR66" H 6400 1950 30  0001 C CNN
+F 0 "#PWR63" H 6400 1950 30  0001 C CNN
 F 1 "GND" H 6400 1880 30  0001 C CNN
 F 2 "" H 6400 1950 60  0000 C CNN
@@
 $EndComp
 $Comp
-L 3V3 #PWR65
+L 3V3 #PWR62
 U 1 1 54DE1F75
 P 6400 900
-F 0 "#PWR65" H 6400 1000 40  0001 C CNN
+F 0 "#PWR62" H 6400 1000 40  0001 C CNN
 F 1 "3V3" H 6400 1025 40  0000 C CNN
 F 2 "" H 6400 900 60  0000 C CNN
@@
 	8250 3000 8550 3000
 Wire Wire Line
-	5950 1700 6450 1700
+	5950 1700 6600 1700
 Wire Wire Line
 	5950 1550 6050 1550
@@
 	6050 1550 6050 1600
 Wire Wire Line
-	6050 1600 6450 1600
+	6050 1600 6600 1600
 Wire Wire Line
 	5950 1400 6100 1400
@@
 	6100 1400 6100 1500
 Wire Wire Line
-	6100 1500 6450 1500
+	6100 1500 6600 1500
 Wire Wire Line
 	5950 1250 6150 1250
@@
 	6150 1250 6150 1400
 Wire Wire Line
-	6150 1400 6450 1400
+	6150 1400 6600 1400
 Wire Wire Line
 	6400 1950 6400 1300
 Wire Wire Line
-	6400 1300 6450 1300
-Wire Wire Line
-	6450 1200 6400 1200
+	6400 1300 6600 1300
+Wire Wire Line
+	6400 1200 6600 1200
 Wire Wire Line
 	6400 1200 6400 900
@@
 $EndComp
 $Comp
-L 3V3 #PWR71
+L 3V3 #PWR68
 U 1 1 54EE9CD1
 P 9100 4400
-F 0 "#PWR71" H 9100 4500 40  0001 C CNN
+F 0 "#PWR68" H 9100 4500 40  0001 C CNN
 F 1 "3V3" H 9100 4525 40  0000 C CNN
 F 2 "" H 9100 4400 60  0000 C CNN
@@
 $EndComp
 $Comp
-L 3V3 #PWR72
+L 3V3 #PWR69
 U 1 1 54EE9CDD
 P 9300 4400
-F 0 "#PWR72" H 9300 4500 40  0001 C CNN
+F 0 "#PWR69" H 9300 4500 40  0001 C CNN
 F 1 "3V3" H 9300 4525 40  0000 C CNN
 F 2 "" H 9300 4400 60  0000 C CNN
@@
 $EndComp
 $Comp
-L 3V3 #PWR67
+L 3V3 #PWR64
 U 1 1 54EE9E9C
 P 7500 4450
-F 0 "#PWR67" H 7500 4550 40  0001 C CNN
+F 0 "#PWR64" H 7500 4550 40  0001 C CNN
 F 1 "3V3" H 7500 4575 40  0000 C CNN
 F 2 "" H 7500 4450 60  0000 C CNN
@@
 $EndComp
 $Comp
-L 3V3 #PWR68
+L 3V3 #PWR65
 U 1 1 54EE9EA8
 P 7700 4450
-F 0 "#PWR68" H 7700 4550 40  0001 C CNN
+F 0 "#PWR65" H 7700 4550 40  0001 C CNN
 F 1 "3V3" H 7700 4575 40  0000 C CNN
 F 2 "" H 7700 4450 60  0000 C CNN

Commit message: Completed rev 3.0 schematics.
1) Replaced MPU with STM Accelerometer
Parts:
- R22, R23: footprint ~ -> (none)
- R3, R4: footprint ~ -> Resistors_SMD:R_0603
- U1: footprint ~ -> footprints:CoolrunnerII
Connections:
- wire segments 138 -> 140
Changed lines of the file:
@@
 F 0 "U6" H 8500 5350 60  0000 C CNN
 F 1 "PCA9515B" H 8500 5700 60  0000 C CNN
-F 2 "" H 8500 5700 60  0000 C CNN
+F 2 "" H 8500 5700 60  0001 C CNN
 F 3 "" H 8500 5700 60  0000 C CNN
 	1    8500 5300
@@
 $EndComp
 $Comp
-L 3V3 #PWR66
+L 3V3 #PWR054
 U 1 1 54723DBD
 P 7950 4900
-F 0 "#PWR66" H 7950 5000 40  0001 C CNN
+F 0 "#PWR054" H 7950 5000 40  0001 C CNN
 F 1 "3V3" H 7950 5025 40  0000 C CNN
 F 2 "" H 7950 4900 60  0000 C CNN
@@
 $EndComp
 $Comp
-L GND #PWR67
+L GND #PWR055
 U 1 1 54723E16
 P 7950 5700
-F 0 "#PWR67" H 7950 5700 30  0001 C CNN
+F 0 "#PWR055" H 7950 5700 30  0001 C CNN
 F 1 "GND" H 7950 5630 30  0001 C CNN
 F 2 "" H 7950 5700 60  0000 C CNN
@@
 F 0 "U1" H 4000 4150 60  0000 C CNN
 F 1 "XC2C32A" H 4000 5400 60  0000 C CNN
-F 2 "~" H 4000 4800 60  0000 C CNN
+F 2 "footprints:CoolrunnerII" H 4000 4800 60  0000 C CNN
 F 3 "~" H 4000 4800 60  0000 C CNN
 	1    4000 4150
@@
 $EndComp
 $Comp
-L 3V3 #PWR60
+L 3V3 #PWR056
 U 1 1 54DD88EA
 P 4850 2750
-F 0 "#PWR60" H 4850 2850 40  0001 C CNN
+F 0 "#PWR056" H 4850 2850 40  0001 C CNN
 F 1 "3V3" H 4850 2875 40  0000 C CNN
 F 2 "" H 4850 2750 60  0000 C CNN
@@
 $EndComp
 $Comp
-L GND #PWR61
-U 1 1 54DD89FD
-P 6100 3500
-F 0 "#PWR61" H 6100 3500 30  0001 C CNN
-F 1 "GND" H 6100 3430 30  0001 C CNN
-F 2 "" H 6100 3500 60  0000 C CNN
-F 3 "" H 6100 3500 60  0000 C CNN
-	1    6100 3500
-	1    0    0    -1
-$EndComp
-$Comp
-L GND #PWR59
-U 1 1 54DD8C2C
-P 1950 4950
-F 0 "#PWR59" H 1950 4950 30  0001 C CNN
-F 1 "GND" H 1950 4880 30  0001 C CNN
-F 2 "" H 1950 4950 60  0000 C CNN
-F 3 "" H 1950 4950 60  0000 C CNN
-	1    1950 4950
-	1    0    0    -1
-$EndComp
-$Comp
-L 1V8 #PWR58
+L 1V8 #PWR057
 U 1 1 54DD8CFA
 P 1950 4550
-F 0 "#PWR58" H 1950 4690 20  0001 C CNN
+F 0 "#PWR057" H 1950 4690 20  0001 C CNN
 F 1 "1V8" H 1950 4660 30  0000 C CNN
 F 2 "" H 1950 4550 60  0000 C CNN
@@
 F 0 "P11" V 6750 1450 60  0000 C CNN
 F 1 "CPLD_JTAG" V 6850 1450 60  0000 C CNN
-F 2 "" H 6800 1450 60  0000 C CNN
+F 2 "" H 6800 1450 60  0001 C CNN
 F 3 "" H 6800 1450 60  0000 C CNN
 	1    6800 1450
@@
 $EndComp
 $Comp
-L GND #PWR63
-U 1 1 54DE1EE6
-P 6400 1950
-F 0 "#PWR63" H 6400 1950 30  0001 C CNN
-F 1 "GND" H 6400 1880 30  0001 C CNN
-F 2 "" H 6400 1950 60  0000 C CNN
-F 3 "" H 6400 1950 60  0000 C CNN
-	1    6400 1950
-	1    0    0    -1
-$EndComp
-$Comp
-L 3V3 #PWR62
+L 3V3 #PWR058
 U 1 1 54DE1F75
 P 6400 900
-F 0 "#PWR62" H 6400 1000 40  0001 C CNN
+F 0 "#PWR058" H 6400 1000 40  0001 C CNN
 F 1 "3V3" H 6400 1025 40  0000 C CNN
 F 2 "" H 6400 900 60  0000 C CNN
@@
 Connection ~ 4850 3400
 Wire Wire Line
-	4800 3300 6100 3300
-Wire Wire Line
-	6100 3300 6100 3500
-Wire Wire Line
 	3200 3700 3150 3700
 Wire Wire Line
@@
 	6150 1400 6600 1400
 Wire Wire Line
-	6400 1950 6400 1300
-Wire Wire Line
-	6400 1300 6600 1300
+	6350 1300 6600 1300
 Wire Wire Line
 	6400 1200 6600 1200
@@
 F 0 "R4" V 9180 4700 40  0000 C CNN
 F 1 "4.7k" V 9107 4701 40  0000 C CNN
-F 2 "~" V 9030 4700 30  0000 C CNN
+F 2 "Resistors_SMD:R_0603" V 9030 4700 30  0001 C CNN
 F 3 "~" H 9100 4700 30  0000 C CNN
 	1    9100 4700
@@
 $EndComp
 $Comp
-L 3V3 #PWR68
+L 3V3 #PWR059
 U 1 1 54EE9CD1
 P 9100 4400
-F 0 "#PWR68" H 9100 4500 40  0001 C CNN
+F 0 "#PWR059" H 9100 4500 40  0001 C CNN
 F 1 "3V3" H 9100 4525 40  0000 C CNN
 F 2 "" H 9100 4400 60  0000 C CNN
@@
 F 0 "R3" V 9380 4700 40  0000 C CNN
 F 1 "4.7k" V 9307 4701 40  0000 C CNN
-F 2 "~" V 9230 4700 30  0000 C CNN
+F 2 "Resistors_SMD:R_0603" V 9230 4700 30  0001 C CNN
 F 3 "~" H 9300 4700 30  0000 C CNN
 	1    9300 4700
@@
 $EndComp
 $Comp
-L 3V3 #PWR69
+L 3V3 #PWR060
 U 1 1 54EE9CDD
 P 9300 4400
-F 0 "#PWR69" H 9300 4500 40  0001 C CNN
+F 0 "#PWR060" H 9300 4500 40  0001 C CNN
 F 1 "3V3" H 9300 4525 40  0000 C CNN
 F 2 "" H 9300 4400 60  0000 C CNN
@@
 F 0 "R22" V 7580 4750 40  0000 C CNN
 F 1 "4.7k" V 7507 4751 40  0000 C CNN
-F 2 "~" V 7430 4750 30  0000 C CNN
+F 2 "" V 7430 4750 30  0001 C CNN
 F 3 "~" H 7500 4750 30  0000 C CNN
 	1    7500 4750
@@
 $EndComp
 $Comp
-L 3V3 #PWR64
+L 3V3 #PWR061
 U 1 1 54EE9E9C
 P 7500 4450
-F 0 "#PWR64" H 7500 4550 40  0001 C CNN
+F 0 "#PWR061" H 7500 4550 40  0001 C CNN
 F 1 "3V3" H 7500 4575 40  0000 C CNN
 F 2 "" H 7500 4450 60  0000 C CNN
@@
 F 0 "R23" V 7780 4750 40  0000 C CNN
 F 1 "4.7k" V 7707 4751 40  0000 C CNN
-F 2 "~" V 7630 4750 30  0000 C CNN
+F 2 "" V 7630 4750 30  0001 C CNN
 F 3 "~" H 7700 4750 30  0000 C CNN
 	1    7700 4750
@@
 $EndComp
 $Comp
-L 3V3 #PWR65
+L 3V3 #PWR062
 U 1 1 54EE9EA8
 P 7700 4450
-F 0 "#PWR65" H 7700 4550 40  0001 C CNN
+F 0 "#PWR062" H 7700 4550 40  0001 C CNN
 F 1 "3V3" H 7700 4575 40  0000 C CNN
 F 2 "" H 7700 4450 60  0000 C CNN
@@
 NoConn ~ 3200 5100
 NoConn ~ 3200 4600
+$Comp
+L GND #PWR063
+U 1 1 55A8C1A3
+P 6250 1300
+F 0 "#PWR063" H 6250 1300 30  0001 C CNN
+F 1 "GND" H 6250 1230 30  0001 C CNN
+F 2 "" H 6250 1300 60  0000 C CNN
+F 3 "" H 6250 1300 60  0000 C CNN
+	1    6250 1300
+	1    0    0    -1
+$EndComp
+Wire Wire Line
+	6350 1300 6350 1250
+Wire Wire Line
+	6350 1250 6250 1250
+Wire Wire Line
+	6250 1250 6250 1300
+$Comp
+L GND #PWR064
+U 1 1 55A8CDE3
+P 6200 3450
+F 0 "#PWR064" H 6200 3450 30  0001 C CNN
+F 1 "GND" H 6200 3380 30  0001 C CNN
+F 2 "" H 6200 3450 60  0000 C CNN
+F 3 "" H 6200 3450 60  0000 C CNN
+	1    6200 3450
+	1    0    0    -1
+$EndComp
+Wire Wire Line
+	4800 3300 6200 3300
+Wire Wire Line
+	6200 3300 6200 3450
+$Comp
+L GND #PWR065
+U 1 1 55A8D239
+P 1950 4950
+F 0 "#PWR065" H 1950 4950 30  0001 C CNN
+F 1 "GND" H 1950 4880 30  0001 C CNN
+F 2 "" H 1950 4950 60  0000 C CNN
+F 3 "" H 1950 4950 60  0000 C CNN
+	1    1950 4950
+	1    0    0    -1
+$EndComp
 $EndSCHEMATC
