File: board/mainboard/LaunchpadConnection.sch (KiCad schematic (older format))
At the start: 1 part

Commit message: Added simple peripherals to launchpad schematic
Parts:
- added D?: RLED, ~, symbol LED
- added D?: GLED, ~, symbol LED
- added P? (x2): CONN_2, symbol CONN_2
- added PR? (x2): 500K, ~, symbol R
- added R? (x2): 100K, ~, symbol R
- added R?: 560, ~, symbol R
- added RV? (x2): 10K, ~, symbol POT
- added SW? (x4): SW_PUSH, ~, symbol SW_PUSH
Connections:
- wire segments 32 -> 81

Commit message: Named some default named connectors, fixed incorrect pull down
Parts:
- P?: value CONN_2 -> ANALOG
- P?: value CONN_2 -> BUMPERS
Changed lines of the file:
@@
 P 1500 3700
 F 0 "P?" V 1450 3700 40  0000 C CNN
-F 1 "CONN_2" V 1550 3700 40  0000 C CNN
+F 1 "ANALOG" V 1550 3700 40  0000 C CNN
 F 2 "" H 1500 3700 60  0000 C CNN
 F 3 "" H 1500 3700 60  0000 C CNN
@@
 P 10300 3650
 F 0 "P?" V 10250 3650 40  0000 C CNN
-F 1 "CONN_2" V 10350 3650 40  0000 C CNN
+F 1 "BUMPERS" V 10350 3650 40  0000 C CNN
 F 2 "" H 10300 3650 60  0000 C CNN
 F 3 "" H 10300 3650 60  0000 C CNN

Commit message: Added connector for Line Sensors, and fixed pots/photsensors
Parts:
- removed PR? (x2): 500K, ~, symbol R
- removed R? (x2): 100K, ~, symbol R
- removed RV?: 10K, ~, symbol POT
- added P?: CONN_5, symbol CONN_5
Connections:
- net labels added: LINE_SENSOR_C, LINE_SENSOR_L, LINE_SENSOR_R, POT
- net labels removed: PHOTO1, PHOTO2, POT1, POT2
- wire segments 81 -> 73
Changed lines of the file:
@@
 Sheet 4 5
 Title ""
-Date "18 nov 2014"
+Date "19 nov 2014"
 Rev ""
 Comp ""
@@
 	1    0    0    -1
 $EndComp
-Text GLabel 4050 4800 0    60   Input ~ 0
-POT1
 Text GLabel 4050 4950 0    60   Input ~ 0
-POT2
+POT
 Text GLabel 4050 4500 0    60   Input ~ 0
-PHOTO1
+LINE_SENSOR_L
 Text GLabel 4050 4650 0    60   Input ~ 0
-PHOTO2
+LINE_SENSOR_R
 Text GLabel 4050 2400 0    60   Input ~ 0
 AIN1
@@
 L 3V3 #PWR?
 U 1 1 546A82AF
-P 1900 6350
-F 0 "#PWR?" H 1900 6450 40  0001 C CNN
-F 1 "3V3" H 1900 6475 40  0000 C CNN
-F 2 "" H 1900 6350 60  0000 C CNN
-F 3 "" H 1900 6350 60  0000 C CNN
-	1    1900 6350
+P 2000 4650
+F 0 "#PWR?" H 2000 4750 40  0001 C CNN
+F 1 "3V3" H 2000 4775 40  0000 C CNN
+F 2 "" H 2000 4650 60  0000 C CNN
+F 3 "" H 2000 4650 60  0000 C CNN
+	1    2000 4650
 	1    0    0    -1
 $EndComp
@@
 L GND #PWR?
 U 1 1 546A82BC
-P 1900 7050
-F 0 "#PWR?" H 1900 7050 30  0001 C CNN
-F 1 "GND" H 1900 6980 30  0001 C CNN
-F 2 "" H 1900 7050 60  0000 C CNN
-F 3 "" H 1900 7050 60  0000 C CNN
-	1    1900 7050
+P 2000 5350
+F 0 "#PWR?" H 2000 5350 30  0001 C CNN
+F 1 "GND" H 2000 5280 30  0001 C CNN
+F 2 "" H 2000 5350 60  0000 C CNN
+F 3 "" H 2000 5350 60  0000 C CNN
+	1    2000 5350
 	1    0    0    -1
 $EndComp
@@
 L POT RV?
 U 1 1 546A82C5
-P 1700 6700
-F 0 "RV?" H 1700 6600 50  0000 C CNN
-F 1 "10K" H 1700 6700 50  0000 C CNN
-F 2 "~" H 1700 6700 60  0000 C CNN
-F 3 "~" H 1700 6700 60  0000 C CNN
-	1    1700 6700
+P 2000 5000
+F 0 "RV?" H 2000 4900 50  0000 C CNN
+F 1 "10K" H 2000 5000 50  0000 C CNN
+F 2 "~" H 2000 5000 60  0000 C CNN
+F 3 "~" H 2000 5000 60  0000 C CNN
+	1    2000 5000
 	0    -1   -1   0
 $EndComp
-$Comp
-L POT RV?
-U 1 1 546A82D2
-P 2100 6700
-F 0 "RV?" H 2100 6600 50  0000 C CNN
-F 1 "10K" H 2100 6700 50  0000 C CNN
-F 2 "~" H 2100 6700 60  0000 C CNN
-F 3 "~" H 2100 6700 60  0000 C CNN
-	1    2100 6700
-	0    1    1    0
-$EndComp
-Text GLabel 1400 6700 0    60   Input ~ 0
-POT1
-Text GLabel 2400 6700 2    60   Input ~ 0
-POT2
-$Comp
-L R PR?
-U 1 1 546A8635
-P 2050 4850
-F 0 "PR?" V 2130 4850 40  0000 C CNN
-F 1 "500K" V 2057 4851 40  0000 C CNN
-F 2 "~" V 1980 4850 30  0000 C CNN
-F 3 "~" H 2050 4850 30  0000 C CNN
-	1    2050 4850
-	1    0    0    -1
-$EndComp
-$Comp
-L R R?
-U 1 1 546A865D
-P 2050 5500
-F 0 "R?" V 2130 5500 40  0000 C CNN
-F 1 "100K" V 2057 5501 40  0000 C CNN
-F 2 "~" V 1980 5500 30  0000 C CNN
-F 3 "~" H 2050 5500 30  0000 C CNN
-	1    2050 5500
-	1    0    0    -1
-$EndComp
-$Comp
-L 3V3 #PWR?
-U 1 1 546A866B
-P 1900 4500
-F 0 "#PWR?" H 1900 4600 40  0001 C CNN
-F 1 "3V3" H 1900 4625 40  0000 C CNN
-F 2 "" H 1900 4500 60  0000 C CNN
-F 3 "" H 1900 4500 60  0000 C CNN
-	1    1900 4500
-	1    0    0    -1
-$EndComp
-$Comp
-L R PR?
-U 1 1 546A8673
-P 1750 4850
-F 0 "PR?" V 1830 4850 40  0000 C CNN
-F 1 "500K" V 1757 4851 40  0000 C CNN
-F 2 "~" V 1680 4850 30  0000 C CNN
-F 3 "~" H 1750 4850 30  0000 C CNN
-	1    1750 4850
-	1    0    0    -1
-$EndComp
-$Comp
-L R R?
-U 1 1 546A8679
-P 1750 5500
-F 0 "R?" V 1830 5500 40  0000 C CNN
-F 1 "100K" V 1757 5501 40  0000 C CNN
-F 2 "~" V 1680 5500 30  0000 C CNN
-F 3 "~" H 1750 5500 30  0000 C CNN
-	1    1750 5500
-	1    0    0    -1
-$EndComp
+Text GLabel 1700 5000 0    60   Input ~ 0
+POT
 $Comp
 L GND #PWR?
 U 1 1 546A8777
-P 1900 7050
-F 0 "#PWR?" H 1900 7050 30  0001 C CNN
-F 1 "GND" H 1900 6980 30  0001 C CNN
-F 2 "" H 1900 7050 60  0000 C CNN
-F 3 "" H 1900 7050 60  0000 C CNN
-	1    1900 7050
+P 2000 5350
+F 0 "#PWR?" H 2000 5350 30  0001 C CNN
+F 1 "GND" H 2000 5280 30  0001 C CNN
+F 2 "" H 2000 5350 60  0000 C CNN
+F 3 "" H 2000 5350 60  0000 C CNN
+	1    2000 5350
 	1    0    0    -1
 $EndComp
@@
 L GND #PWR?
 U 1 1 546A877E
-P 1900 7050
-F 0 "#PWR?" H 1900 7050 30  0001 C CNN
-F 1 "GND" H 1900 6980 30  0001 C CNN
-F 2 "" H 1900 7050 60  0000 C CNN
-F 3 "" H 1900 7050 60  0000 C CNN
-	1    1900 7050
+P 2000 5350
+F 0 "#PWR?" H 2000 5350 30  0001 C CNN
+F 1 "GND" H 2000 5280 30  0001 C CNN
+F 2 "" H 2000 5350 60  0000 C CNN
+F 3 "" H 2000 5350 60  0000 C CNN
+	1    2000 5350
 	1    0    0    -1
 $EndComp
@@
 L GND #PWR?
 U 1 1 546A8785
-P 1900 7050
-F 0 "#PWR?" H 1900 7050 30  0001 C CNN
-F 1 "GND" H 1900 6980 30  0001 C CNN
-F 2 "" H 1900 7050 60  0000 C CNN
-F 3 "" H 1900 7050 60  0000 C CNN
-	1    1900 7050
-	1    0    0    -1
-$EndComp
-$Comp
-L GND #PWR?
-U 1 1 546A878E
-P 1900 5900
-F 0 "#PWR?" H 1900 5900 30  0001 C CNN
-F 1 "GND" H 1900 5830 30  0001 C CNN
-F 2 "" H 1900 5900 60  0000 C CNN
-F 3 "" H 1900 5900 60  0000 C CNN
-	1    1900 5900
-	1    0    0    -1
-$EndComp
-Text GLabel 1500 5200 0    60   Input ~ 0
-PHOTO1
-Text GLabel 2300 5200 2    60   Input ~ 0
-PHOTO2
+P 2000 5350
+F 0 "#PWR?" H 2000 5350 30  0001 C CNN
+F 1 "GND" H 2000 5280 30  0001 C CNN
+F 2 "" H 2000 5350 60  0000 C CNN
+F 3 "" H 2000 5350 60  0000 C CNN
+	1    2000 5350
+	1    0    0    -1
+$EndComp
 $Comp
 L CONN_2 P?
@@
 	6850 2700 7150 2700
 Wire Wire Line
-	2250 6700 2400 6700
-Wire Wire Line
-	1400 6700 1550 6700
-Wire Wire Line
-	1700 6950 1700 7000
-Wire Wire Line
-	1700 7000 2100 7000
-Wire Wire Line
-	1900 7000 1900 7050
-Wire Wire Line
-	2100 7000 2100 6950
-Connection ~ 1900 7000
-Wire Wire Line
-	1900 6350 1900 6400
-Wire Wire Line
-	1700 6400 2100 6400
-Wire Wire Line
-	1700 6400 1700 6450
-Wire Wire Line
-	2100 6400 2100 6450
-Connection ~ 1900 6400
-Wire Wire Line
-	1900 4500 1900 4550
-Wire Wire Line
-	1750 4550 2050 4550
-Wire Wire Line
-	1750 4550 1750 4600
-Wire Wire Line
-	2050 4550 2050 4600
-Connection ~ 1900 4550
-Wire Wire Line
-	1750 5100 1750 5250
-Wire Wire Line
-	2050 5100 2050 5250
-Wire Wire Line
-	1750 5750 1750 5800
-Wire Wire Line
-	1750 5800 2050 5800
-Wire Wire Line
-	2050 5800 2050 5750
-Wire Wire Line
-	1900 5800 1900 5900
-Connection ~ 1900 5800
-Wire Wire Line
-	1500 5200 1750 5200
-Connection ~ 1750 5200
-Wire Wire Line
-	2050 5200 2300 5200
-Connection ~ 2050 5200
+	1700 5000 1850 5000
 Wire Wire Line
 	2050 3800 1850 3800
@@
 Wire Wire Line
 	9750 3750 9950 3750
+$Comp
+L CONN_5 P?
+U 1 1 546BE6CC
+P 1350 2600
+F 0 "P?" V 1300 2600 50  0000 C CNN
+F 1 "CONN_5" V 1400 2600 50  0000 C CNN
+F 2 "" H 1350 2600 60  0000 C CNN
+F 3 "" H 1350 2600 60  0000 C CNN
+	1    1350 2600
+	-1   0    0    1
+$EndComp
+$Comp
+L GND #PWR?
+U 1 1 546BE7D1
+P 1950 3000
+F 0 "#PWR?" H 1950 3000 30  0001 C CNN
+F 1 "GND" H 1950 2930 30  0001 C CNN
+F 2 "" H 1950 3000 60  0000 C CNN
+F 3 "" H 1950 3000 60  0000 C CNN
+	1    1950 3000
+	1    0    0    -1
+$EndComp
+Wire Wire Line
+	1750 2800 1950 2800
+Wire Wire Line
+	1950 2800 1950 3000
+$Comp
+L 3V3 #PWR?
+U 1 1 546BE83D
+P 1950 2250
+F 0 "#PWR?" H 1950 2350 40  0001 C CNN
+F 1 "3V3" H 1950 2375 40  0000 C CNN
+F 2 "" H 1950 2250 60  0000 C CNN
+F 3 "" H 1950 2250 60  0000 C CNN
+	1    1950 2250
+	1    0    0    -1
+$EndComp
+Wire Wire Line
+	1750 2400 1950 2400
+Wire Wire Line
+	1950 2400 1950 2250
+Text GLabel 2200 2400 2    60   Input ~ 0
+LINE_SENSOR_R
+Text GLabel 2200 2600 2    60   Input ~ 0
+LINE_SENSOR_C
+Text GLabel 2200 2800 2    60   Input ~ 0
+LINE_SENSOR_L
+Wire Wire Line
+	1750 2600 2200 2600
+Wire Wire Line
+	1750 2500 2050 2500
+Wire Wire Line
+	2050 2500 2050 2400
+Wire Wire Line
+	2050 2400 2200 2400
+Wire Wire Line
+	1750 2700 2050 2700
+Wire Wire Line
+	2050 2700 2050 2800
+Wire Wire Line
+	2050 2800 2200 2800
+Text GLabel 4050 4800 0    60   Input ~ 0
+LINE_SENSOR_C
+Wire Wire Line
+	2000 4650 2000 4750
+Wire Wire Line
+	2000 5250 2000 5350
 $EndSCHEMATC

Commit message: Added CC3200 bus cutoff schematics
Parts:
- added R? (x2): 10K, ~, symbol R
Connections:
- net labels added: I2C_CL_LP, I2C_DA_LP, SPI_MISO_LP, SPI_MOSI_LP, SPI_SCK_LP, SPI_SEL0_LP, SPI_SEL1_LP, SPI_SEL2_LP, UART_RX_LP, UART_TX_LP
- net labels removed: I2C_CL, I2C_DA, SPI_MISO, SPI_MOSI, SPI_SCK, SPI_SEL0, SPI_SEL1, SPI_SEL2, UART_RX, UART_TX
- wire segments 73 -> 77

Commit message: Added header containing all interrupt pins
Parts:
- added P?: INT_GPIO, symbol CONN_6
Connections:
- net labels added: MOTOR1F, MOTOR2F, MPUINT, RTCINT1, RTCINT2, SD_SWITCH
- wire segments 77 -> 93
Changed lines of the file:
@@
 L CONN_2 P?
 U 1 1 546A9114
-P 10300 2900
-F 0 "P?" V 10250 2900 40  0000 C CNN
-F 1 "BUMPERS" V 10350 2900 40  0000 C CNN
-F 2 "" H 10300 2900 60  0000 C CNN
-F 3 "" H 10300 2900 60  0000 C CNN
-	1    10300 2900
+P 10250 2250
+F 0 "P?" V 10200 2250 40  0000 C CNN
+F 1 "BUMPERS" V 10300 2250 40  0000 C CNN
+F 2 "" H 10250 2250 60  0000 C CNN
+F 3 "" H 10250 2250 60  0000 C CNN
+	1    10250 2250
 	1    0    0    -1
 $EndComp
-Text GLabel 9750 2800 0    60   Input ~ 0
+Text GLabel 9700 2150 0    60   Input ~ 0
 BUMP1
-Text GLabel 9750 3000 0    60   Input ~ 0
+Text GLabel 9700 2350 0    60   Input ~ 0
 BUMP2
 Wire Wire Line
-	9750 2800 9950 2800
+	9700 2150 9900 2150
 Wire Wire Line
-	9750 3000 9950 3000
+	9700 2350 9900 2350
 $Comp
 L CONN_5 P?
@@
 Wire Wire Line
 	8050 1250 8050 1350
-Text GLabel 3550 5400 0    60   Input ~ 0
-SPI_MISO_LP
-Text GLabel 3550 5250 0    60   Input ~ 0
-SPI_MOSI_LP
-Text GLabel 3550 5850 0    60   Input ~ 0
-SPI_SEL0_LP
-Text GLabel 3550 5700 0    60   Input ~ 0
-SPI_SEL1_LP
-Text GLabel 3550 5550 0    60   Input ~ 0
-SPI_SEL2_LP
-Text GLabel 3550 5100 0    60   Input ~ 0
-SPI_SCK_LP
-Text GLabel 3550 6000 0    60   Input ~ 0
-I2C_CL_LP
-Text GLabel 3550 6150 0    60   Input ~ 0
-I2C_DA_LP
+Text GLabel 4900 5350 0    60   Input ~ 0
+RTCINT1
+Text GLabel 4900 5500 0    60   Input ~ 0
+RTCINT2
+Text GLabel 4900 5650 0    60   Input ~ 0
+MPUINT
+Text GLabel 4900 5800 0    60   Input ~ 0
+SD_SWITCH
+$Comp
+L CONN_6 P?
+U 1 1 54724B44
+P 5700 5750
+F 0 "P?" V 5650 5750 60  0000 C CNN
+F 1 "INT_GPIO" V 5750 5750 60  0000 C CNN
+F 2 "" H 5700 5750 60  0000 C CNN
+F 3 "" H 5700 5750 60  0000 C CNN
+	1    5700 5750
+	1    0    0    -1
+$EndComp
+Text GLabel 4900 5950 0    60   Input ~ 0
+MOTOR1F
+Text GLabel 4900 6100 0    60   Input ~ 0
+MOTOR2F
+Wire Wire Line
+	4900 5350 5300 5350
+Wire Wire Line
+	5300 5350 5300 5500
+Wire Wire Line
+	5300 5500 5350 5500
+Wire Wire Line
+	4900 5500 5200 5500
+Wire Wire Line
+	5200 5500 5200 5600
+Wire Wire Line
+	5200 5600 5350 5600
+Wire Wire Line
+	4900 5650 5100 5650
+Wire Wire Line
+	5100 5650 5100 5700
+Wire Wire Line
+	5100 5700 5350 5700
+Wire Wire Line
+	4900 5800 5350 5800
+Wire Wire Line
+	4900 5950 5100 5950
+Wire Wire Line
+	5100 5950 5100 5900
+Wire Wire Line
+	5100 5900 5350 5900
+Wire Wire Line
+	4900 6100 5200 6100
+Wire Wire Line
+	5200 6100 5200 6000
+Wire Wire Line
+	5200 6000 5350 6000
 $EndSCHEMATC

Commit message: Connected GLCD_A0 to Launchpad and buffered it
Connections:
- net labels added: GPIO_A0_LP
- wire segments 93 -> 94
- no-connect marks 11 -> 10
Changed lines of the file:
@@
 $Descr A4 11693 8268
 encoding utf-8
-Sheet 4 6
+Sheet 4 7
 Title ""
 Date "23 nov 2014"
@@
 NoConn ~ 4550 4250
 NoConn ~ 6850 4250
-NoConn ~ 6850 3800
 NoConn ~ 6850 3350
 $Comp
@@
 Wire Wire Line
 	5200 6000 5350 6000
+Text GLabel 7150 3800 2    60   Input ~ 0
+GPIO_A0_LP
+Wire Wire Line
+	6850 3800 7150 3800
 $EndSCHEMATC

Commit message: Added header for remaining GPIOs on Launchpad
Parts:
- removed P?: INT_GPIO, symbol CONN_6
- added P?: INT_SRC, symbol CONN_7
- added P?: GPIO, symbol CONN_5
Connections:
- net labels added: PA5, PC4, PE0, PE4, PF4, WIFI_INT
- wire segments 94 -> 113
- no-connect marks 10 -> 5
Changed lines of the file:
@@
 Text GLabel 7150 2300 2    60   Input ~ 0
 SPI_SEL2_LP
-NoConn ~ 6850 1550
-NoConn ~ 4550 1850
-NoConn ~ 4550 2300
 NoConn ~ 4550 2900
 NoConn ~ 4550 3200
@@
 NoConn ~ 4550 4100
 NoConn ~ 4550 4250
-NoConn ~ 6850 4250
-NoConn ~ 6850 3350
 $Comp
 L GND #PWR?
@@
 Wire Wire Line
 	8050 1250 8050 1350
-Text GLabel 4900 5350 0    60   Input ~ 0
+Text GLabel 3500 5150 0    60   Input ~ 0
 RTCINT1
-Text GLabel 4900 5500 0    60   Input ~ 0
+Text GLabel 3500 5300 0    60   Input ~ 0
 RTCINT2
-Text GLabel 4900 5650 0    60   Input ~ 0
+Text GLabel 3500 5450 0    60   Input ~ 0
 MPUINT
-Text GLabel 4900 5800 0    60   Input ~ 0
+Text GLabel 3500 5600 0    60   Input ~ 0
 SD_SWITCH
-$Comp
-L CONN_6 P?
-U 1 1 54724B44
-P 5700 5750
-F 0 "P?" V 5650 5750 60  0000 C CNN
-F 1 "INT_GPIO" V 5750 5750 60  0000 C CNN
-F 2 "" H 5700 5750 60  0000 C CNN
-F 3 "" H 5700 5750 60  0000 C CNN
-	1    5700 5750
-	1    0    0    -1
-$EndComp
-Text GLabel 4900 5950 0    60   Input ~ 0
+Text GLabel 3500 5750 0    60   Input ~ 0
 MOTOR1F
-Text GLabel 4900 6100 0    60   Input ~ 0
+Text GLabel 3500 5900 0    60   Input ~ 0
 MOTOR2F
 Wire Wire Line
-	4900 5350 5300 5350
-Wire Wire Line
-	5300 5350 5300 5500
-Wire Wire Line
-	5300 5500 5350 5500
-Wire Wire Line
-	4900 5500 5200 5500
-Wire Wire Line
-	5200 5500 5200 5600
-Wire Wire Line
-	5200 5600 5350 5600
-Wire Wire Line
-	4900 5650 5100 5650
-Wire Wire Line
-	5100 5650 5100 5700
-Wire Wire Line
-	5100 5700 5350 5700
-Wire Wire Line
-	4900 5800 5350 5800
-Wire Wire Line
-	4900 5950 5100 5950
-Wire Wire Line
-	5100 5950 5100 5900
-Wire Wire Line
-	5100 5900 5350 5900
-Wire Wire Line
-	4900 6100 5200 6100
-Wire Wire Line
-	5200 6100 5200 6000
-Wire Wire Line
-	5200 6000 5350 6000
+	3500 5150 3900 5150
+Wire Wire Line
+	3900 5150 3900 5300
+Wire Wire Line
+	3900 5300 3950 5300
+Wire Wire Line
+	3500 5300 3800 5300
+Wire Wire Line
+	3800 5300 3800 5400
+Wire Wire Line
+	3800 5400 3950 5400
+Wire Wire Line
+	3500 5450 3700 5450
+Wire Wire Line
+	3700 5450 3700 5500
+Wire Wire Line
+	3700 5500 3950 5500
+Wire Wire Line
+	3500 5600 3950 5600
+Wire Wire Line
+	3500 5750 3700 5750
+Wire Wire Line
+	3700 5750 3700 5700
+Wire Wire Line
+	3700 5700 3950 5700
+Wire Wire Line
+	3500 5900 3800 5900
+Wire Wire Line
+	3800 5900 3800 5800
+Wire Wire Line
+	3800 5800 3950 5800
 Text GLabel 7150 3800 2    60   Input ~ 0
 GPIO_A0_LP
 Wire Wire Line
 	6850 3800 7150 3800
+$Comp
+L CONN_7 P?
+U 1 1 547268C8
+P 4300 5600
+F 0 "P?" V 4270 5600 60  0000 C CNN
+F 1 "INT_SRC" V 4370 5600 60  0000 C CNN
+F 2 "" H 4300 5600 60  0000 C CNN
+F 3 "" H 4300 5600 60  0000 C CNN
+	1    4300 5600
+	1    0    0    -1
+$EndComp
+Text GLabel 3500 6050 0    60   Input ~ 0
+WIFI_INT
+Wire Wire Line
+	3500 6050 3900 6050
+Wire Wire Line
+	3900 6050 3900 5900
+Wire Wire Line
+	3900 5900 3950 5900
+Text GLabel 7150 1550 2    60   Input ~ 0
+PE0
+Wire Wire Line
+	6850 1550 7150 1550
+Text GLabel 7150 3350 2    60   Input ~ 0
+PC4
+Wire Wire Line
+	6850 3350 7150 3350
+Text GLabel 7150 4250 2    60   Input ~ 0
+PF4
+Wire Wire Line
+	6850 4250 7150 4250
+Text GLabel 4050 1850 0    60   Input ~ 0
+PE4
+Wire Wire Line
+	4050 1850 4550 1850
+Text GLabel 4050 2300 0    60   Input ~ 0
+PA5
+Wire Wire Line
+	4050 2300 4550 2300
+$Comp
+L CONN_5 P?
+U 1 1 54726AA3
+P 6850 5650
+F 0 "P?" V 6800 5650 50  0000 C CNN
+F 1 "GPIO" V 6900 5650 50  0000 C CNN
+F 2 "" H 6850 5650 60  0000 C CNN
+F 3 "" H 6850 5650 60  0000 C CNN
+	1    6850 5650
+	1    0    0    -1
+$EndComp
+Text GLabel 6150 5350 0    60   Input ~ 0
+PA5
+Text GLabel 6150 5500 0    60   Input ~ 0
+PC4
+Text GLabel 6150 5650 0    60   Input ~ 0
+PE0
+Text GLabel 6150 5800 0    60   Input ~ 0
+PE4
+Text GLabel 6150 5950 0    60   Input ~ 0
+PF4
+Wire Wire Line
+	6150 5350 6450 5350
+Wire Wire Line
+	6450 5350 6450 5450
+Wire Wire Line
+	6150 5500 6400 5500
+Wire Wire Line
+	6400 5500 6400 5550
+Wire Wire Line
+	6400 5550 6450 5550
+Wire Wire Line
+	6150 5650 6450 5650
+Wire Wire Line
+	6150 5800 6400 5800
+Wire Wire Line
+	6400 5800 6400 5750
+Wire Wire Line
+	6400 5750 6450 5750
+Wire Wire Line
+	6150 5950 6450 5950
+Wire Wire Line
+	6450 5950 6450 5850
 $EndSCHEMATC
