File: board/mainboard/LaunchpadConnection.sch (KiCad schematic (older format))
At the start: 16 parts

Commit message: Added net names, fixed misnamed GLCD_A0
Parts:
- gave numbers to parts that had none: 16
Connections:
- net labels added: GLCD_A0_LP
- net labels removed: GPIO_A0_LP
Changed lines of the file:
@@
 $EndDescr
 $Comp
-L TIVALAUNCHPAD LP?
+L TIVALAUNCHPAD LP1
 U 1 1 5467DA7D
 P 5700 2750
-F 0 "LP?" H 5700 2600 60  0000 C CNN
+F 0 "LP1" H 5700 2600 60  0000 C CNN
 F 1 "TIVALAUNCHPAD" H 5700 2750 60  0000 C CNN
 F 2 "~" H 5700 2750 60  0000 C CNN
@@
 $EndComp
 $Comp
-L 3V3 #PWR?
+L 3V3 #PWR039
 U 1 1 5467DAD5
 P 4300 1050
-F 0 "#PWR?" H 4300 1150 40  0001 C CNN
+F 0 "#PWR039" H 4300 1150 40  0001 C CNN
 F 1 "3V3" H 4300 1175 40  0000 C CNN
 F 2 "" H 4300 1050 60  0000 C CNN
@@
 NoConn ~ 4550 4250
 $Comp
-L GND #PWR?
+L GND #PWR040
 U 1 1 5468095A
 P 8050 1350
-F 0 "#PWR?" H 8050 1350 30  0001 C CNN
+F 0 "#PWR040" H 8050 1350 30  0001 C CNN
 F 1 "GND" H 8050 1280 30  0001 C CNN
 F 2 "" H 8050 1350 60  0000 C CNN
@@
 AIN2
 $Comp
-L GND #PWR?
+L GND #PWR041
 U 1 1 546A7E28
 P 4300 3200
-F 0 "#PWR?" H 4300 3200 30  0001 C CNN
+F 0 "#PWR041" H 4300 3200 30  0001 C CNN
 F 1 "GND" H 4300 3130 30  0001 C CNN
 F 2 "" H 4300 3200 60  0000 C CNN
@@
 NMI
 $Comp
-L 3V3 #PWR?
+L 3V3 #PWR042
 U 1 1 546A82AF
 P 2000 4650
-F 0 "#PWR?" H 2000 4750 40  0001 C CNN
+F 0 "#PWR042" H 2000 4750 40  0001 C CNN
 F 1 "3V3" H 2000 4775 40  0000 C CNN
 F 2 "" H 2000 4650 60  0000 C CNN
@@
 $EndComp
 $Comp
-L GND #PWR?
+L GND #PWR043
 U 1 1 546A82BC
 P 2000 5350
-F 0 "#PWR?" H 2000 5350 30  0001 C CNN
+F 0 "#PWR043" H 2000 5350 30  0001 C CNN
 F 1 "GND" H 2000 5280 30  0001 C CNN
 F 2 "" H 2000 5350 60  0000 C CNN
@@
 $EndComp
 $Comp
-L POT RV?
+L POT RV1
 U 1 1 546A82C5
 P 2000 5000
-F 0 "RV?" H 2000 4900 50  0000 C CNN
+F 0 "RV1" H 2000 4900 50  0000 C CNN
 F 1 "10K" H 2000 5000 50  0000 C CNN
 F 2 "~" H 2000 5000 60  0000 C CNN
@@
 POT
 $Comp
-L GND #PWR?
+L GND #PWR044
 U 1 1 546A8777
 P 2000 5350
-F 0 "#PWR?" H 2000 5350 30  0001 C CNN
+F 0 "#PWR044" H 2000 5350 30  0001 C CNN
 F 1 "GND" H 2000 5280 30  0001 C CNN
 F 2 "" H 2000 5350 60  0000 C CNN
@@
 $EndComp
 $Comp
-L GND #PWR?
+L GND #PWR045
 U 1 1 546A877E
 P 2000 5350
-F 0 "#PWR?" H 2000 5350 30  0001 C CNN
+F 0 "#PWR045" H 2000 5350 30  0001 C CNN
 F 1 "GND" H 2000 5280 30  0001 C CNN
 F 2 "" H 2000 5350 60  0000 C CNN
@@
 $EndComp
 $Comp
-L GND #PWR?
+L GND #PWR046
 U 1 1 546A8785
 P 2000 5350
-F 0 "#PWR?" H 2000 5350 30  0001 C CNN
+F 0 "#PWR046" H 2000 5350 30  0001 C CNN
 F 1 "GND" H 2000 5280 30  0001 C CNN
 F 2 "" H 2000 5350 60  0000 C CNN
@@
 $EndComp
 $Comp
-L CONN_2 P?
+L CONN_2 P7
 U 1 1 546A885A
 P 1500 3700
-F 0 "P?" V 1450 3700 40  0000 C CNN
+F 0 "P7" V 1450 3700 40  0000 C CNN
 F 1 "ANALOG" V 1550 3700 40  0000 C CNN
 F 2 "" H 1500 3700 60  0000 C CNN
@@
 LED1
 $Comp
-L LED D?
+L LED D2
 U 1 1 546A8A5B
 P 10550 3500
-F 0 "D?" H 10550 3600 50  0000 C CNN
+F 0 "D2" H 10550 3600 50  0000 C CNN
 F 1 "RLED" H 10550 3400 50  0000 C CNN
 F 2 "~" H 10550 3500 60  0000 C CNN
@@
 $EndComp
 $Comp
-L LED D?
+L LED D1
 U 1 1 546A8A77
 P 10250 3650
-F 0 "D?" H 10250 3750 50  0000 C CNN
+F 0 "D1" H 10250 3750 50  0000 C CNN
 F 1 "GLED" H 10250 3550 50  0000 C CNN
 F 2 "~" H 10250 3650 60  0000 C CNN
@@
 $EndComp
 $Comp
-L R R?
+L R R17
 U 1 1 546A8AAA
 P 9700 3300
-F 0 "R?" V 9780 3300 40  0000 C CNN
+F 0 "R17" V 9780 3300 40  0000 C CNN
 F 1 "560" V 9707 3301 40  0000 C CNN
 F 2 "~" V 9630 3300 30  0000 C CNN
@@
 $EndComp
 $Comp
-L GND #PWR?
+L GND #PWR047
 U 1 1 546A8BD2
 P 10400 4000
-F 0 "#PWR?" H 10400 4000 30  0001 C CNN
+F 0 "#PWR047" H 10400 4000 30  0001 C CNN
 F 1 "GND" H 10400 3930 30  0001 C CNN
 F 2 "" H 10400 4000 60  0000 C CNN
@@
 Connection ~ 10400 3900
 $Comp
-L SW_PUSH SW?
+L SW_PUSH SW1
 U 1 1 546A8D80
 P 9200 5100
-F 0 "SW?" H 9350 5210 50  0000 C CNN
+F 0 "SW1" H 9350 5210 50  0000 C CNN
 F 1 "SW_PUSH" H 9200 5020 50  0000 C CNN
 F 2 "~" H 9200 5100 60  0000 C CNN
@@
 $EndComp
 $Comp
-L SW_PUSH SW?
+L SW_PUSH SW3
 U 1 1 546A8D8D
 P 10100 5100
-F 0 "SW?" H 10250 5210 50  0000 C CNN
+F 0 "SW3" H 10250 5210 50  0000 C CNN
 F 1 "SW_PUSH" H 10100 5020 50  0000 C CNN
 F 2 "~" H 10100 5100 60  0000 C CNN
@@
 $EndComp
 $Comp
-L SW_PUSH SW?
+L SW_PUSH SW2
 U 1 1 546A8D93
 P 9200 5700
-F 0 "SW?" H 9350 5810 50  0000 C CNN
+F 0 "SW2" H 9350 5810 50  0000 C CNN
 F 1 "SW_PUSH" H 9200 5620 50  0000 C CNN
 F 2 "~" H 9200 5700 60  0000 C CNN
@@
 $EndComp
 $Comp
-L SW_PUSH SW?
+L SW_PUSH SW4
 U 1 1 546A8D99
 P 10100 5700
-F 0 "SW?" H 10250 5810 50  0000 C CNN
+F 0 "SW4" H 10250 5810 50  0000 C CNN
 F 1 "SW_PUSH" H 10100 5620 50  0000 C CNN
 F 2 "~" H 10100 5700 60  0000 C CNN
@@
 	9550 4650 9550 6150
 $Comp
-L CONN_2 P?
+L CONN_2 P10
 U 1 1 546A9114
 P 10250 2250
-F 0 "P?" V 10200 2250 40  0000 C CNN
+F 0 "P10" V 10200 2250 40  0000 C CNN
 F 1 "BUMPERS" V 10300 2250 40  0000 C CNN
 F 2 "" H 10250 2250 60  0000 C CNN
@@
 	9700 2350 9900 2350
 $Comp
-L CONN_5 P?
+L CONN_5 P6
 U 1 1 546BE6CC
 P 1350 2600
-F 0 "P?" V 1300 2600 50  0000 C CNN
+F 0 "P6" V 1300 2600 50  0000 C CNN
 F 1 "CONN_5" V 1400 2600 50  0000 C CNN
 F 2 "" H 1350 2600 60  0000 C CNN
@@
 $EndComp
 $Comp
-L GND #PWR?
+L GND #PWR048
 U 1 1 546BE7D1
 P 1950 3000
-F 0 "#PWR?" H 1950 3000 30  0001 C CNN
+F 0 "#PWR048" H 1950 3000 30  0001 C CNN
 F 1 "GND" H 1950 2930 30  0001 C CNN
 F 2 "" H 1950 3000 60  0000 C CNN
@@
 	1950 2800 1950 3000
 $Comp
-L 3V3 #PWR?
+L 3V3 #PWR049
 U 1 1 546BE83D
 P 1950 2250
-F 0 "#PWR?" H 1950 2350 40  0001 C CNN
+F 0 "#PWR049" H 1950 2350 40  0001 C CNN
 F 1 "3V3" H 1950 2375 40  0000 C CNN
 F 2 "" H 1950 2250 60  0000 C CNN
@@
 	2000 5250 2000 5350
 $Comp
-L R R?
+L R R16
 U 1 1 547220E2
 P 9550 6400
-F 0 "R?" V 9630 6400 40  0000 C CNN
+F 0 "R16" V 9630 6400 40  0000 C CNN
 F 1 "10K" V 9557 6401 40  0000 C CNN
 F 2 "~" V 9480 6400 30  0000 C CNN
@@
 $EndComp
 $Comp
-L R R?
+L R R18
 U 1 1 547220F8
 P 10450 6400
-F 0 "R?" V 10530 6400 40  0000 C CNN
+F 0 "R18" V 10530 6400 40  0000 C CNN
 F 1 "10K" V 10457 6401 40  0000 C CNN
 F 2 "~" V 10380 6400 30  0000 C CNN
@@
 	10450 6700 10450 6650
 $Comp
-L GND #PWR?
+L GND #PWR050
 U 1 1 547221EF
 P 10400 4000
-F 0 "#PWR?" H 10400 4000 30  0001 C CNN
+F 0 "#PWR050" H 10400 4000 30  0001 C CNN
 F 1 "GND" H 10400 3930 30  0001 C CNN
 F 2 "" H 10400 4000 60  0000 C CNN
@@
 $EndComp
 $Comp
-L GND #PWR?
+L GND #PWR051
 U 1 1 547221F6
 P 10000 6850
-F 0 "#PWR?" H 10000 6850 30  0001 C CNN
+F 0 "#PWR051" H 10000 6850 30  0001 C CNN
 F 1 "GND" H 10000 6780 30  0001 C CNN
 F 2 "" H 10000 6850 60  0000 C CNN
@@
 	3800 5800 3950 5800
 Text GLabel 7150 3800 2    60   Input ~ 0
-GPIO_A0_LP
+GLCD_A0_LP
 Wire Wire Line
 	6850 3800 7150 3800
 $Comp
-L CONN_7 P?
+L CONN_7 P8
 U 1 1 547268C8
 P 4300 5600
-F 0 "P?" V 4270 5600 60  0000 C CNN
+F 0 "P8" V 4270 5600 60  0000 C CNN
 F 1 "INT_SRC" V 4370 5600 60  0000 C CNN
 F 2 "" H 4300 5600 60  0000 C CNN
@@
 	4050 2300 4550 2300
 $Comp
-L CONN_5 P?
+L CONN_5 P9
 U 1 1 54726AA3
 P 6850 5650
-F 0 "P?" V 6800 5650 50  0000 C CNN
+F 0 "P9" V 6800 5650 50  0000 C CNN
 F 1 "GPIO" V 6900 5650 50  0000 C CNN
 F 2 "" H 6850 5650 60  0000 C CNN

Commit message: Added Audio coded net to optional peripherals header
Parts:
- removed P8: INT_SRC, symbol CONN_7
- added P8: OPTIONAL_PERIPH, symbol CONN_8
Connections:
- net labels added: AUD_DAC_CL
- wire segments 113 -> 115
Changed lines of the file:
@@
 $Descr A4 11693 8268
 encoding utf-8
-Sheet 4 7
+Sheet 4 8
 Title ""
-Date "24 nov 2014"
+Date "25 nov 2014"
 Rev ""
 Comp ""
@@
 Wire Wire Line
 	6850 3800 7150 3800
-$Comp
-L CONN_7 P8
-U 1 1 547268C8
-P 4300 5600
-F 0 "P8" V 4270 5600 60  0000 C CNN
-F 1 "INT_SRC" V 4370 5600 60  0000 C CNN
-F 2 "" H 4300 5600 60  0000 C CNN
-F 3 "" H 4300 5600 60  0000 C CNN
-	1    4300 5600
-	1    0    0    -1
-$EndComp
 Text GLabel 3500 6050 0    60   Input ~ 0
 WIFI_INT
-Wire Wire Line
-	3500 6050 3900 6050
-Wire Wire Line
-	3900 6050 3900 5900
-Wire Wire Line
-	3900 5900 3950 5900
 Text GLabel 7150 1550 2    60   Input ~ 0
 PE0
@@
 Wire Wire Line
 	6450 5950 6450 5850
+$Comp
+L CONN_8 P8
+U 1 1 5473C1EB
+P 4300 5650
+F 0 "P8" V 4250 5650 60  0000 C CNN
+F 1 "OPTIONAL_PERIPH" V 4350 5650 60  0000 C CNN
+F 2 "" H 4300 5650 60  0000 C CNN
+F 3 "" H 4300 5650 60  0000 C CNN
+	1    4300 5650
+	1    0    0    -1
+$EndComp
+Wire Wire Line
+	3500 6050 3900 6050
+Text GLabel 3500 6200 0    60   Input ~ 0
+AUD_DAC_CL
+Wire Wire Line
+	3500 6200 3950 6200
+Wire Wire Line
+	3950 6200 3950 6000
+Wire Wire Line
+	3950 5900 3900 5900
+Wire Wire Line
+	3900 5900 3900 6050
 $EndSCHEMATC

Commit message: Finished first draft of rev 1 board
Parts:
- removed P10: BUMPERS, symbol CONN_2
- added P10: BUMPERS, symbol CONN_4
Connections:
- wire segments 115 -> 118
Changed lines of the file:
@@
 Wire Wire Line
 	9550 4650 9550 6150
-$Comp
-L CONN_2 P10
-U 1 1 546A9114
-P 10250 2250
-F 0 "P10" V 10200 2250 40  0000 C CNN
-F 1 "BUMPERS" V 10300 2250 40  0000 C CNN
-F 2 "" H 10250 2250 60  0000 C CNN
-F 3 "" H 10250 2250 60  0000 C CNN
-	1    10250 2250
-	1    0    0    -1
-$EndComp
 Text GLabel 9700 2150 0    60   Input ~ 0
 BUMP1
@@
 Wire Wire Line
 	8050 1250 8050 1350
+Text GLabel 3500 5450 0    60   Input ~ 0
+RTCINT1
+Text GLabel 3500 5600 0    60   Input ~ 0
+RTCINT2
 Text GLabel 3500 5150 0    60   Input ~ 0
-RTCINT1
-Text GLabel 3500 5300 0    60   Input ~ 0
-RTCINT2
-Text GLabel 3500 5450 0    60   Input ~ 0
 MPUINT
-Text GLabel 3500 5600 0    60   Input ~ 0
+Text GLabel 3500 5750 0    60   Input ~ 0
 SD_SWITCH
-Text GLabel 3500 5750 0    60   Input ~ 0
+Text GLabel 3500 5900 0    60   Input ~ 0
 MOTOR1F
-Text GLabel 3500 5900 0    60   Input ~ 0
+Text GLabel 3500 6050 0    60   Input ~ 0
 MOTOR2F
 Wire Wire Line
@@
 Wire Wire Line
 	6850 3800 7150 3800
-Text GLabel 3500 6050 0    60   Input ~ 0
+Text GLabel 3500 5300 0    60   Input ~ 0
 WIFI_INT
 Text GLabel 7150 1550 2    60   Input ~ 0
@@
 Wire Wire Line
 	3900 5900 3900 6050
+$Comp
+L CONN_4 P10
+U 1 1 54741374
+P 10250 2300
+F 0 "P10" V 10200 2300 50  0000 C CNN
+F 1 "BUMPERS" V 10300 2300 50  0000 C CNN
+F 2 "" H 10250 2300 60  0000 C CNN
+F 3 "" H 10250 2300 60  0000 C CNN
+	1    10250 2300
+	1    0    0    -1
+$EndComp
+$Comp
+L GND #PWR052
+U 1 1 54741383
+P 9800 2600
+F 0 "#PWR052" H 9800 2600 30  0001 C CNN
+F 1 "GND" H 9800 2530 30  0001 C CNN
+F 2 "" H 9800 2600 60  0000 C CNN
+F 3 "" H 9800 2600 60  0000 C CNN
+	1    9800 2600
+	1    0    0    -1
+$EndComp
+Wire Wire Line
+	9900 2250 9800 2250
+Wire Wire Line
+	9800 2250 9800 2600
+Wire Wire Line
+	9900 2450 9800 2450
+Connection ~ 9800 2450
 $EndSCHEMATC

Commit message: Various fixes to schematics and footprints:
* Added pullup resistors to bumpers
* Changed value of RLED resistor
* Added resistor to GLED
* Changed SPI pullup resistors to 47k
* Added JTAG header for CPLD
* Changed motor driver footprint to MSOP
Parts:
- added D?: POWER, ~, symbol LED
- added R? (x2): 220, ~, symbol R
- added R? (x2): 47k, ~, symbol R
- R17: value 560 -> 220
Connections:
- wire segments 118 -> 127

Commit message: Added power LED, removed Codec Peripheral pin
Parts:
- gave numbers to parts that had none: 5
Connections:
- net labels removed: AUD_DAC_CL
- wire segments 127 -> 125
Changed lines of the file:
@@
 Sheet 4 7
 Title ""
-Date "13 feb 2015"
+Date "16 feb 2015"
 Rev ""
 Comp ""
@@
 $EndComp
 $Comp
-L 3V3 #PWR037
+L 3V3 #PWR44
 U 1 1 5467DAD5
 P 4300 1050
-F 0 "#PWR037" H 4300 1150 40  0001 C CNN
+F 0 "#PWR44" H 4300 1150 40  0001 C CNN
 F 1 "3V3" H 4300 1175 40  0000 C CNN
 F 2 "" H 4300 1050 60  0000 C CNN
@@
 NoConn ~ 4550 4250
 $Comp
-L GND #PWR038
+L GND #PWR46
 U 1 1 5468095A
 P 8050 1350
-F 0 "#PWR038" H 8050 1350 30  0001 C CNN
+F 0 "#PWR46" H 8050 1350 30  0001 C CNN
 F 1 "GND" H 8050 1280 30  0001 C CNN
 F 2 "" H 8050 1350 60  0000 C CNN
@@
 AIN2
 $Comp
-L GND #PWR039
+L GND #PWR45
 U 1 1 546A7E28
 P 4300 3200
-F 0 "#PWR039" H 4300 3200 30  0001 C CNN
+F 0 "#PWR45" H 4300 3200 30  0001 C CNN
 F 1 "GND" H 4300 3130 30  0001 C CNN
 F 2 "" H 4300 3200 60  0000 C CNN
@@
 NMI
 $Comp
-L 3V3 #PWR040
+L 3V3 #PWR39
 U 1 1 546A82AF
 P 2000 4650
-F 0 "#PWR040" H 2000 4750 40  0001 C CNN
+F 0 "#PWR39" H 2000 4750 40  0001 C CNN
 F 1 "3V3" H 2000 4775 40  0000 C CNN
 F 2 "" H 2000 4650 60  0000 C CNN
@@
 $EndComp
 $Comp
-L GND #PWR041
+L GND #PWR40
 U 1 1 546A82BC
 P 2000 5350
-F 0 "#PWR041" H 2000 5350 30  0001 C CNN
+F 0 "#PWR40" H 2000 5350 30  0001 C CNN
 F 1 "GND" H 2000 5280 30  0001 C CNN
 F 2 "" H 2000 5350 60  0000 C CNN
@@
 POT
 $Comp
-L GND #PWR042
+L GND #PWR41
 U 1 1 546A8777
 P 2000 5350
-F 0 "#PWR042" H 2000 5350 30  0001 C CNN
+F 0 "#PWR41" H 2000 5350 30  0001 C CNN
 F 1 "GND" H 2000 5280 30  0001 C CNN
 F 2 "" H 2000 5350 60  0000 C CNN
@@
 $EndComp
 $Comp
-L GND #PWR043
+L GND #PWR42
 U 1 1 546A877E
 P 2000 5350
-F 0 "#PWR043" H 2000 5350 30  0001 C CNN
+F 0 "#PWR42" H 2000 5350 30  0001 C CNN
 F 1 "GND" H 2000 5280 30  0001 C CNN
 F 2 "" H 2000 5350 60  0000 C CNN
@@
 $EndComp
 $Comp
-L GND #PWR044
+L GND #PWR43
 U 1 1 546A8785
 P 2000 5350
-F 0 "#PWR044" H 2000 5350 30  0001 C CNN
+F 0 "#PWR43" H 2000 5350 30  0001 C CNN
 F 1 "GND" H 2000 5280 30  0001 C CNN
 F 2 "" H 2000 5350 60  0000 C CNN
@@
 $EndComp
 $Comp
-L GND #PWR045
+L GND #PWR52
 U 1 1 546A8BD2
 P 10400 4000
-F 0 "#PWR045" H 10400 4000 30  0001 C CNN
+F 0 "#PWR52" H 10400 4000 30  0001 C CNN
 F 1 "GND" H 10400 3930 30  0001 C CNN
 F 2 "" H 10400 4000 60  0000 C CNN
@@
 $EndComp
 $Comp
-L GND #PWR046
+L GND #PWR38
 U 1 1 546BE7D1
 P 1950 3000
-F 0 "#PWR046" H 1950 3000 30  0001 C CNN
+F 0 "#PWR38" H 1950 3000 30  0001 C CNN
 F 1 "GND" H 1950 2930 30  0001 C CNN
 F 2 "" H 1950 3000 60  0000 C CNN
@@
 $EndComp
 $Comp
-L 3V3 #PWR047
+L 3V3 #PWR37
 U 1 1 546BE83D
 P 1950 2250
-F 0 "#PWR047" H 1950 2350 40  0001 C CNN
+F 0 "#PWR37" H 1950 2350 40  0001 C CNN
 F 1 "3V3" H 1950 2375 40  0000 C CNN
 F 2 "" H 1950 2250 60  0000 C CNN
@@
 $EndComp
 $Comp
-L GND #PWR048
+L GND #PWR53
 U 1 1 547221EF
 P 10400 4000
-F 0 "#PWR048" H 10400 4000 30  0001 C CNN
+F 0 "#PWR53" H 10400 4000 30  0001 C CNN
 F 1 "GND" H 10400 3930 30  0001 C CNN
 F 2 "" H 10400 4000 60  0000 C CNN
@@
 $EndComp
 $Comp
-L GND #PWR049
+L GND #PWR51
 U 1 1 547221F6
 P 10000 6850
-F 0 "#PWR049" H 10000 6850 30  0001 C CNN
+F 0 "#PWR51" H 10000 6850 30  0001 C CNN
 F 1 "GND" H 10000 6780 30  0001 C CNN
 F 2 "" H 10000 6850 60  0000 C CNN
@@
 	1    0    0    -1
 $EndComp
-Text GLabel 3500 6200 0    60   Input ~ 0
-AUD_DAC_CL
 $Comp
 L CONN_4 P10
@@
 $EndComp
 $Comp
-L GND #PWR050
+L GND #PWR50
 U 1 1 54741383
 P 9800 2600
-F 0 "#PWR050" H 9800 2600 30  0001 C CNN
+F 0 "#PWR50" H 9800 2600 30  0001 C CNN
 F 1 "GND" H 9800 2530 30  0001 C CNN
 F 2 "" H 9800 2600 60  0000 C CNN
@@
 $EndComp
 $Comp
-L R R?
+L R R9
 U 1 1 54DE166E
 P 9700 3450
-F 0 "R?" V 9780 3450 40  0000 C CNN
+F 0 "R9" V 9780 3450 40  0000 C CNN
 F 1 "220" V 9707 3451 40  0000 C CNN
 F 2 "~" V 9630 3450 30  0000 C CNN
@@
 $EndComp
 $Comp
-L R R?
+L R R8
 U 1 1 54DE17F4
 P 9600 1800
-F 0 "R?" V 9680 1800 40  0000 C CNN
+F 0 "R8" V 9680 1800 40  0000 C CNN
 F 1 "47k" V 9607 1801 40  0000 C CNN
 F 2 "~" V 9530 1800 30  0000 C CNN
@@
 $EndComp
 $Comp
-L R R?
+L R R19
 U 1 1 54DE180D
 P 9750 1800
-F 0 "R?" V 9830 1800 40  0000 C CNN
+F 0 "R19" V 9830 1800 40  0000 C CNN
 F 1 "47k" V 9757 1801 40  0000 C CNN
 F 2 "~" V 9680 1800 30  0000 C CNN
@@
 	3500 6050 3900 6050
 Wire Wire Line
-	3500 6200 3950 6200
-Wire Wire Line
-	3950 6200 3950 6000
-Wire Wire Line
 	3950 5900 3900 5900
 Wire Wire Line
@@
 Connection ~ 9750 2350
 $Comp
-L 3V3 #PWR?
+L 3V3 #PWR49
 U 1 1 54DE19B8
 P 9600 1350
-F 0 "#PWR?" H 9600 1450 40  0001 C CNN
+F 0 "#PWR49" H 9600 1450 40  0001 C CNN
 F 1 "3V3" H 9600 1475 40  0000 C CNN
 F 2 "" H 9600 1350 60  0000 C CNN
@@
 Connection ~ 9600 1500
 $Comp
-L 3V3 #PWR?
+L 3V3 #PWR47
 U 1 1 54DE1AF6
 P 8600 2900
-F 0 "#PWR?" H 8600 3000 40  0001 C CNN
+F 0 "#PWR47" H 8600 3000 40  0001 C CNN
 F 1 "3V3" H 8600 3025 40  0000 C CNN
 F 2 "" H 8600 2900 60  0000 C CNN
@@
 $EndComp
 $Comp
-L GND #PWR?
+L GND #PWR48
 U 1 1 54DE1B05
 P 8600 4100
-F 0 "#PWR?" H 8600 4100 30  0001 C CNN
+F 0 "#PWR48" H 8600 4100 30  0001 C CNN
 F 1 "GND" H 8600 4030 30  0001 C CNN
 F 2 "" H 8600 4100 60  0000 C CNN
@@
 $EndComp
 $Comp
-L R R?
+L R R7
 U 1 1 54DE1B12
 P 8600 3250
-F 0 "R?" V 8680 3250 40  0000 C CNN
+F 0 "R7" V 8680 3250 40  0000 C CNN
 F 1 "220" V 8607 3251 40  0000 C CNN
 F 2 "~" V 8530 3250 30  0000 C CNN
@@
 	8600 4000 8600 4100
 $Comp
-L LED D?
+L LED D3
 U 1 1 54DE1CC5
 P 8600 3800
-F 0 "D?" H 8600 3900 50  0000 C CNN
+F 0 "D3" H 8600 3900 50  0000 C CNN
 F 1 "POWER" H 8600 3650 50  0000 C CNN
 F 2 "~" H 8600 3800 60  0000 C CNN

Commit message: Various changes
* Began Rev2 Layout
* Added Pullup Resistors to LP I2C
* Added IrDA Module
Parts:
- removed P8: OPTIONAL_PERIPH, symbol CONN_8
- added D4: CONTROL, ~, symbol LED
- added IR1: RPM841-H11, symbol RPM841-H11
- added K1: IRDA_EN, symbol CONN_3
- added P13: UART, symbol CONN_4
- added P8: OPTIONAL_PERIPH, symbol CONN_7
- added Q1: BSS84, ~, symbol MOS_P
- added R20: 220, ~, symbol R
- added R21: 3, ~, symbol R
Connections:
- net labels added: CC_CONTROL, UART_RX, UART_TX
- wire segments 125 -> 156

Commit message: Further work on the rev2 layout
Connections:
- wire segments 156 -> 158
Changed lines of the file:
@@
 L 3V3 #PWR058
 U 1 1 54EE0894
-P 1800 4350
-F 0 "#PWR058" H 1800 4450 40  0001 C CNN
-F 1 "3V3" H 1800 4475 40  0000 C CNN
-F 2 "" H 1800 4350 60  0000 C CNN
-F 3 "" H 1800 4350 60  0000 C CNN
-	1    1800 4350
+P 1600 4200
+F 0 "#PWR058" H 1600 4300 40  0001 C CNN
+F 1 "3V3" H 1600 4325 40  0000 C CNN
+F 2 "" H 1600 4200 60  0000 C CNN
+F 3 "" H 1600 4200 60  0000 C CNN
+	1    1600 4200
 	1    0    0    -1
 $EndComp
@@
 Wire Wire Line
 	1800 4750 1900 4750
+Text GLabel 1550 4350 0    60   Input ~ 0
+UART_RX
 Text GLabel 1550 4500 0    60   Input ~ 0
-UART_RX
-Text GLabel 1550 4650 0    60   Input ~ 0
 UART_TX
-Wire Wire Line
-	1550 4650 1900 4650
 Wire Wire Line
 	1900 4550 1700 4550
@@
 Wire Wire Line
 	3800 6300 3800 6400
+Wire Wire Line
+	1800 4350 1550 4350
+Wire Wire Line
+	1900 4650 1600 4650
+Wire Wire Line
+	1600 4650 1600 4200
 $EndSCHEMATC

Commit message: Finished draft 1 of Rev 2 layout
Changed lines of the file:
@@
 $Descr A4 11693 8268
 encoding utf-8
-Sheet 4 7
+Sheet 4 8
 Title ""
-Date "26 feb 2015"
+Date "1 mar 2015"
 Rev ""
 Comp ""
@@
 Wire Wire Line
 	1800 4750 1900 4750
+Text GLabel 1550 4500 0    60   Input ~ 0
+UART_RX
 Text GLabel 1550 4350 0    60   Input ~ 0
-UART_RX
-Text GLabel 1550 4500 0    60   Input ~ 0
 UART_TX
 Wire Wire Line
