File: board/mainboard/LaunchpadConnection.sch (KiCad schematic (older format))
At the start: 26 parts, among them K1 IRDA_EN, P10 BUMPERS, P13 UART, P8 OPTIONAL_PERIPH, P9 GPIO, Q1 BSS84, SW1 SW_PUSH, SW2 SW_PUSH, SW3 SW_PUSH, SW4 SW_PUSH

Commit message: Fixes for mainboard 1) Fixed IrDA module footprint, and UART lines. 2) Replaced SPI footprint with header for external LCD
Connections:
- wire segments 145 -> 159
Changed lines of the file:
@@
 	0    -1   -1   0
 $EndComp
-Text GLabel 6450 5550 2    60   Input ~ 0
+Text GLabel 6225 5700 2    60   Input ~ 0
 UART_RX
-Text GLabel 6450 5700 2    60   Input ~ 0
+Text GLabel 6225 5575 2    60   Input ~ 0
 UART_TX
 $Comp
@@
 	1    0    0    -1
 $EndComp
+Text GLabel 4050 1250 0    60   Input ~ 0
+3V3_LP
 Wire Wire Line
 	6850 1250 8050 1250
@@
 	10650 2950 10650 3000
 Wire Wire Line
-	10650 3000 10950 3000
+	10650 3000 10800 3000
+Wire Wire Line
+	10800 3000 10950 3000
 Wire Wire Line
 	10800 3000 10800 3100
@@
 Connection ~ 10800 3000
 Wire Wire Line
-	8500 5100 8900 5100
-Wire Wire Line
-	8500 5700 8900 5700
+	8500 5100 8800 5100
+Wire Wire Line
+	8800 5100 8900 5100
+Wire Wire Line
+	8500 5700 8800 5700
+Wire Wire Line
+	8800 5700 8900 5700
 Wire Wire Line
 	8800 5100 8800 5350
@@
 	10450 5700 10400 5700
 Wire Wire Line
-	10450 4650 10450 6150
+	10450 4650 10450 5100
+Wire Wire Line
+	10450 5100 10450 5700
+Wire Wire Line
+	10450 5700 10450 6150
 Wire Wire Line
 	10450 5100 10400 5100
@@
 Connection ~ 9550 5100
 Wire Wire Line
-	9550 4650 9550 6150
-Wire Wire Line
-	10150 1550 10650 1550
-Wire Wire Line
-	10150 1750 10650 1750
+	9550 4650 9550 5100
+Wire Wire Line
+	9550 5100 9550 5700
+Wire Wire Line
+	9550 5700 9550 6150
+Wire Wire Line
+	10150 1550 10200 1550
+Wire Wire Line
+	10200 1550 10650 1550
+Wire Wire Line
+	10150 1750 10350 1750
+Wire Wire Line
+	10350 1750 10650 1750
 Connection ~ 9550 5700
 Connection ~ 10450 5700
@@
 	9550 6650 9550 6700
 Wire Wire Line
-	9550 6700 10450 6700
+	9550 6700 10000 6700
+Wire Wire Line
+	10000 6700 10450 6700
 Wire Wire Line
 	10450 6700 10450 6650
@@
 	10400 1650 10650 1650
 Wire Wire Line
-	10400 1650 10400 2000
+	10400 1650 10400 1850
+Wire Wire Line
+	10400 1850 10400 2000
 Wire Wire Line
 	10400 1850 10650 1850
@@
 Connection ~ 10350 1750
 Wire Wire Line
-	10200 750  10200 950
+	10200 750  10200 900
+Wire Wire Line
+	10200 900  10200 950
 Wire Wire Line
 	10350 950  10350 900
@@
 	5000 6000 4850 6000
 Wire Wire Line
-	4850 6000 4850 6400
+	4850 6000 4850 6100
+Wire Wire Line
+	4850 6100 4850 6400
 Wire Wire Line
 	5000 6100 4850 6100
@@
 	5000 5600 4300 5600
 Wire Wire Line
-	4300 5250 4300 5700
+	4300 5250 4300 5600
+Wire Wire Line
+	4300 5600 4300 5700
 Wire Wire Line
 	4900 5700 5000 5700
@@
 Connection ~ 4300 5600
 Wire Wire Line
-	6450 5700 6100 5700
-Wire Wire Line
-	6100 5600 6250 5600
-Wire Wire Line
-	6250 5600 6250 5550
-Wire Wire Line
-	6250 5550 6450 5550
-Wire Wire Line
 	7100 5500 7100 5750
 Wire Wire Line
@@
 Wire Wire Line
 	2150 1400 2350 1400
-Text GLabel 4050 1250 0    60   Input ~ 0
-3V3_LP
+Wire Wire Line
+	6100 5700 6225 5700
+Wire Wire Line
+	6100 5600 6175 5600
+Wire Wire Line
+	6175 5600 6175 5575
+Wire Wire Line
+	6175 5575 6225 5575
 $EndSCHEMATC

Commit message: Completed rev 3.0 schematics.
1) Replaced MPU with STM Accelerometer
Parts:
- D1, D2, D3, D4: footprint ~ -> LEDs:LED-0805
- IR1: footprint (none) -> footprints:RPM973-H11
- K1: footprint (none) -> Pin_Headers:Pin_Header_Straight_1x03
- LP1: footprint ~ -> footprints:TivaC
- P10, P13: footprint (none) -> Pin_Headers:Pin_Header_Straight_1x04
- P8: footprint (none) -> Pin_Headers:Pin_Header_Straight_1x07
- P9: footprint (none) -> Pin_Headers:Pin_Header_Straight_1x05
- Q1, R20: footprint ~ -> (none)
- R10, R16, R17, R18, R19, R7, R8, R9: footprint ~ -> Resistors_SMD:R_0603
- R21: footprint ~ -> Resistors_SMD:R_0805
- SW1, SW2, SW3, SW4: footprint ~ -> footprints:PTS645
Connections:
- net labels added: ACCELINT1, ACCELINT2, PCINT
- net labels removed: MOTOR1F, MOTOR2F, MPUINT
- wire segments 159 -> 146

Commit message: Added most of the footprints needed to make this work
Parts:
- R20: footprint (none) -> Resistors_SMD:R_0603
Changed lines of the file:
@@
 NoConn ~ 4550 4250
 $Comp
-L GND #PWR037
+L GND #PWR038
 U 1 1 5468095A
 P 8050 1350
-F 0 "#PWR037" H 8050 1350 30  0001 C CNN
+F 0 "#PWR038" H 8050 1350 30  0001 C CNN
 F 1 "GND" H 8050 1280 30  0001 C CNN
 F 2 "" H 8050 1350 60  0000 C CNN
@@
 AIN2
 $Comp
-L GND #PWR038
+L GND #PWR039
 U 1 1 546A7E28
 P 4300 3200
-F 0 "#PWR038" H 4300 3200 30  0001 C CNN
+F 0 "#PWR039" H 4300 3200 30  0001 C CNN
 F 1 "GND" H 4300 3130 30  0001 C CNN
 F 2 "" H 4300 3200 60  0000 C CNN
@@
 $EndComp
 $Comp
-L GND #PWR039
+L GND #PWR040
 U 1 1 546A8BD2
 P 10800 3100
-F 0 "#PWR039" H 10800 3100 30  0001 C CNN
+F 0 "#PWR040" H 10800 3100 30  0001 C CNN
 F 1 "GND" H 10800 3030 30  0001 C CNN
 F 2 "" H 10800 3100 60  0000 C CNN
@@
 $EndComp
 $Comp
-L GND #PWR040
+L GND #PWR041
 U 1 1 547221EF
 P 10800 3100
-F 0 "#PWR040" H 10800 3100 30  0001 C CNN
+F 0 "#PWR041" H 10800 3100 30  0001 C CNN
 F 1 "GND" H 10800 3030 30  0001 C CNN
 F 2 "" H 10800 3100 60  0000 C CNN
@@
 $EndComp
 $Comp
-L GND #PWR041
+L GND #PWR042
 U 1 1 547221F6
 P 10000 6850
-F 0 "#PWR041" H 10000 6850 30  0001 C CNN
+F 0 "#PWR042" H 10000 6850 30  0001 C CNN
 F 1 "GND" H 10000 6780 30  0001 C CNN
 F 2 "" H 10000 6850 60  0000 C CNN
@@
 $EndComp
 $Comp
-L GND #PWR042
+L GND #PWR043
 U 1 1 54741383
 P 10400 2000
-F 0 "#PWR042" H 10400 2000 30  0001 C CNN
+F 0 "#PWR043" H 10400 2000 30  0001 C CNN
 F 1 "GND" H 10400 1930 30  0001 C CNN
 F 2 "" H 10400 2000 60  0000 C CNN
@@
 $EndComp
 $Comp
-L 3V3 #PWR043
+L 3V3 #PWR044
 U 1 1 54DE19B8
 P 10200 750
-F 0 "#PWR043" H 10200 850 40  0001 C CNN
+F 0 "#PWR044" H 10200 850 40  0001 C CNN
 F 1 "3V3" H 10200 875 40  0000 C CNN
 F 2 "" H 10200 750 60  0000 C CNN
@@
 $EndComp
 $Comp
-L 3V3 #PWR044
+L 3V3 #PWR045
 U 1 1 54DE1AF6
 P 9700 3300
-F 0 "#PWR044" H 9700 3400 40  0001 C CNN
+F 0 "#PWR045" H 9700 3400 40  0001 C CNN
 F 1 "3V3" H 9700 3425 40  0000 C CNN
 F 2 "" H 9700 3300 60  0000 C CNN
@@
 $EndComp
 $Comp
-L GND #PWR045
+L GND #PWR046
 U 1 1 54DE1B05
 P 10950 3550
-F 0 "#PWR045" H 10950 3550 30  0001 C CNN
+F 0 "#PWR046" H 10950 3550 30  0001 C CNN
 F 1 "GND" H 10950 3480 30  0001 C CNN
 F 2 "" H 10950 3550 60  0000 C CNN
@@
 F 0 "R20" V 3880 6050 40  0000 C CNN
 F 1 "220" V 3807 6051 40  0000 C CNN
-F 2 "" V 3730 6050 30  0001 C CNN
+F 2 "Resistors_SMD:R_0603" V 3730 6050 30  0001 C CNN
 F 3 "~" H 3800 6050 30  0000 C CNN
 	1    3800 6050
@@
 $EndComp
 $Comp
-L GND #PWR046
+L GND #PWR047
 U 1 1 54ED2BF4
 P 3800 7100
-F 0 "#PWR046" H 3800 7100 30  0001 C CNN
+F 0 "#PWR047" H 3800 7100 30  0001 C CNN
 F 1 "GND" H 3800 7030 30  0001 C CNN
 F 2 "" H 3800 7100 60  0000 C CNN
@@
 $EndComp
 $Comp
-L 3V3 #PWR047
+L 3V3 #PWR048
 U 1 1 54ED2C03
 P 3800 5050
-F 0 "#PWR047" H 3800 5150 40  0001 C CNN
+F 0 "#PWR048" H 3800 5150 40  0001 C CNN
 F 1 "3V3" H 3800 5175 40  0000 C CNN
 F 2 "" H 3800 5050 60  0000 C CNN
@@
 $EndComp
 $Comp
-L 3V3 #PWR048
+L 3V3 #PWR049
 U 1 1 54EE0127
 P 4300 5250
-F 0 "#PWR048" H 4300 5350 40  0001 C CNN
+F 0 "#PWR049" H 4300 5350 40  0001 C CNN
 F 1 "3V3" H 4300 5375 40  0000 C CNN
 F 2 "" H 4300 5250 60  0000 C CNN
@@
 $EndComp
 $Comp
-L GND #PWR049
+L GND #PWR050
 U 1 1 54EE0140
 P 4850 6400
-F 0 "#PWR049" H 4850 6400 30  0001 C CNN
+F 0 "#PWR050" H 4850 6400 30  0001 C CNN
 F 1 "GND" H 4850 6330 30  0001 C CNN
 F 2 "" H 4850 6400 60  0000 C CNN
@@
 $EndComp
 $Comp
-L 3V3 #PWR050
+L 3V3 #PWR051
 U 1 1 54EE05D1
 P 7100 5500
-F 0 "#PWR050" H 7100 5600 40  0001 C CNN
+F 0 "#PWR051" H 7100 5600 40  0001 C CNN
 F 1 "3V3" H 7100 5625 40  0000 C CNN
 F 2 "" H 7100 5500 60  0000 C CNN
@@
 $EndComp
 $Comp
-L GND #PWR051
+L GND #PWR052
 U 1 1 54EE05D7
 P 7100 6100
-F 0 "#PWR051" H 7100 6100 30  0001 C CNN
+F 0 "#PWR052" H 7100 6100 30  0001 C CNN
 F 1 "GND" H 7100 6030 30  0001 C CNN
 F 2 "" H 7100 6100 60  0000 C CNN
@@
 $EndComp
 $Comp
-L 3V3 #PWR052
+L 3V3 #PWR053
 U 1 1 54EE0894
 P 1600 4200
-F 0 "#PWR052" H 1600 4300 40  0001 C CNN
+F 0 "#PWR053" H 1600 4300 40  0001 C CNN
 F 1 "3V3" H 1600 4325 40  0000 C CNN
 F 2 "" H 1600 4200 60  0000 C CNN
@@
 $EndComp
 $Comp
-L GND #PWR053
+L GND #PWR054
 U 1 1 54EE093D
 P 1800 4950
-F 0 "#PWR053" H 1800 4950 30  0001 C CNN
+F 0 "#PWR054" H 1800 4950 30  0001 C CNN
 F 1 "GND" H 1800 4880 30  0001 C CNN
 F 2 "" H 1800 4950 60  0000 C CNN
@@
 RST
 $Comp
-L 3V3 #PWR054
+L 3V3 #PWR055
 U 1 1 54F5F6CD
 P 8900 1400
-F 0 "#PWR054" H 8900 1500 40  0001 C CNN
+F 0 "#PWR055" H 8900 1500 40  0001 C CNN
 F 1 "3V3" H 8900 1525 40  0000 C CNN
 F 2 "" H 8900 1400 60  0000 C CNN
@@
 	6175 5575 6225 5575
 $Comp
-L PWR_FLAG #FLG055
+L PWR_FLAG #FLG056
 U 1 1 55A8C7A5
 P 4325 1175
-F 0 "#FLG055" H 4325 1270 30  0001 C CNN
+F 0 "#FLG056" H 4325 1270 30  0001 C CNN
 F 1 "PWR_FLAG" H 4325 1355 30  0000 C CNN
 F 2 "" H 4325 1175 60  0000 C CNN
