File: board/mainboard/WifiConnections.sch (KiCad schematic (older format))
At the start: 1 part

Commit message: Added net names, fixed misnamed GLCD_A0
Parts:
- gave numbers to parts that had none: 1
Changed lines of the file:
@@
 $EndDescr
 $Comp
-L WIFI_BOARD WB?
+L WIFI_BOARD WB1
 U 1 1 54725F4B
 P 5700 3650
-F 0 "WB?" H 5700 3600 60  0000 C CNN
+F 0 "WB1" H 5700 3600 60  0000 C CNN
 F 1 "WIFI_BOARD" H 5700 4900 60  0000 C CNN
 F 2 "~" H 5700 3600 60  0000 C CNN
@@
 $EndComp
 $Comp
-L 3V3 #PWR?
+L 3V3 #PWR062
 U 1 1 54725F5A
 P 6600 2450
-F 0 "#PWR?" H 6600 2550 40  0001 C CNN
+F 0 "#PWR062" H 6600 2550 40  0001 C CNN
 F 1 "3V3" H 6600 2575 40  0000 C CNN
 F 2 "" H 6600 2450 60  0000 C CNN
@@
 	6600 2550 6600 2450
 $Comp
-L 3V3 #PWR?
+L 3V3 #PWR063
 U 1 1 54725F6C
 P 6600 3850
-F 0 "#PWR?" H 6600 3950 40  0001 C CNN
+F 0 "#PWR063" H 6600 3950 40  0001 C CNN
 F 1 "3V3" H 6600 3975 40  0000 C CNN
 F 2 "" H 6600 3850 60  0000 C CNN
@@
 	6600 3950 6600 3850
 $Comp
-L GND #PWR?
+L GND #PWR064
 U 1 1 54725F76
 P 6900 3750
-F 0 "#PWR?" H 6900 3750 30  0001 C CNN
+F 0 "#PWR064" H 6900 3750 30  0001 C CNN
 F 1 "GND" H 6900 3680 30  0001 C CNN
 F 2 "" H 6900 3750 60  0000 C CNN
@@
 	6900 3600 6900 3750
 $Comp
-L GND #PWR?
+L GND #PWR065
 U 1 1 54725F95
 P 6600 5150
-F 0 "#PWR?" H 6600 5150 30  0001 C CNN
+F 0 "#PWR065" H 6600 5150 30  0001 C CNN
 F 1 "GND" H 6600 5080 30  0001 C CNN
 F 2 "" H 6600 5150 60  0000 C CNN

Commit message: Various changes
* Began Rev2 Layout
* Added Pullup Resistors to LP I2C
* Added IrDA Module
Parts:
- added R27: 10K, ~, symbol R
Connections:
- wire segments 28 -> 31
Changed lines of the file:
@@
 Sheet 6 7
 Title ""
-Date "16 feb 2015"
+Date "26 feb 2015"
 Rev ""
 Comp ""
@@
 $EndComp
 $Comp
-L 3V3 #PWR62
+L 3V3 #PWR072
 U 1 1 54725F5A
-P 6600 2450
-F 0 "#PWR62" H 6600 2550 40  0001 C CNN
-F 1 "3V3" H 6600 2575 40  0000 C CNN
-F 2 "" H 6600 2450 60  0000 C CNN
-F 3 "" H 6600 2450 60  0000 C CNN
-	1    6600 2450
+P 6600 1750
+F 0 "#PWR072" H 6600 1850 40  0001 C CNN
+F 1 "3V3" H 6600 1875 40  0000 C CNN
+F 2 "" H 6600 1750 60  0000 C CNN
+F 3 "" H 6600 1750 60  0000 C CNN
+	1    6600 1750
 	1    0    0    -1
 $EndComp
@@
 	6450 2550 6600 2550
 Wire Wire Line
-	6600 2550 6600 2450
+	6600 2550 6600 1750
 $Comp
-L 3V3 #PWR63
+L 3V3 #PWR073
 U 1 1 54725F6C
 P 6600 3850
-F 0 "#PWR63" H 6600 3950 40  0001 C CNN
+F 0 "#PWR073" H 6600 3950 40  0001 C CNN
 F 1 "3V3" H 6600 3975 40  0000 C CNN
 F 2 "" H 6600 3850 60  0000 C CNN
@@
 	6600 3950 6600 3850
 $Comp
-L GND #PWR65
+L GND #PWR074
 U 1 1 54725F76
 P 6900 3750
-F 0 "#PWR65" H 6900 3750 30  0001 C CNN
+F 0 "#PWR074" H 6900 3750 30  0001 C CNN
 F 1 "GND" H 6900 3680 30  0001 C CNN
 F 2 "" H 6900 3750 60  0000 C CNN
@@
 	6900 3600 6900 3750
 $Comp
-L GND #PWR64
+L GND #PWR075
 U 1 1 54725F95
 P 6600 5150
-F 0 "#PWR64" H 6600 5150 30  0001 C CNN
+F 0 "#PWR075" H 6600 5150 30  0001 C CNN
 F 1 "GND" H 6600 5080 30  0001 C CNN
 F 2 "" H 6600 5150 60  0000 C CNN
@@
 Wire Wire Line
 	4550 3900 4950 3900
+$Comp
+L R R27
+U 1 1 54ED26EB
+P 6800 2300
+F 0 "R27" V 6880 2300 40  0000 C CNN
+F 1 "10K" V 6807 2301 40  0000 C CNN
+F 2 "~" V 6730 2300 30  0000 C CNN
+F 3 "~" H 6800 2300 30  0000 C CNN
+	1    6800 2300
+	1    0    0    -1
+$EndComp
+Wire Wire Line
+	6800 2050 6800 1850
+Wire Wire Line
+	6800 1850 6600 1850
+Connection ~ 6600 1850
+Wire Wire Line
+	6800 2550 6800 2700
+Connection ~ 6800 2700
 $EndSCHEMATC
