File: board/mainboard/WifiConnections.sch (KiCad schematic (older format))
At the start: 2 parts

Commit message: Completed rev 3.0 schematics.
1) Replaced MPU with STM Accelerometer
Parts:
- R27, WB1: footprint ~ -> (none)
Connections:
- net labels added: ACCELINT1, ACCELINT2, PCINT
- net labels removed: MOTOR1F, MOTOR2F, MPUINT
Changed lines of the file:
@@
 $Descr A4 11693 8268
 encoding utf-8
-Sheet 6 10
+Sheet 7 10
 Title ""
 Date "3 mar 2015"
@@
 F 0 "WB1" H 5700 3600 60  0000 C CNN
 F 1 "WIFI_BOARD" H 5700 4900 60  0000 C CNN
-F 2 "~" H 5700 3600 60  0000 C CNN
+F 2 "" H 5700 3600 60  0001 C CNN
 F 3 "~" H 5700 3600 60  0000 C CNN
 	1    5700 3650
@@
 $EndComp
 $Comp
-L 3V3 #PWR70
+L 3V3 #PWR066
 U 1 1 54725F5A
 P 6600 1750
-F 0 "#PWR70" H 6600 1850 40  0001 C CNN
+F 0 "#PWR066" H 6600 1850 40  0001 C CNN
 F 1 "3V3" H 6600 1875 40  0000 C CNN
 F 2 "" H 6600 1750 60  0000 C CNN
@@
 	6600 2550 6600 1750
 $Comp
-L 3V3 #PWR71
+L 3V3 #PWR067
 U 1 1 54725F6C
 P 6600 3850
-F 0 "#PWR71" H 6600 3950 40  0001 C CNN
+F 0 "#PWR067" H 6600 3950 40  0001 C CNN
 F 1 "3V3" H 6600 3975 40  0000 C CNN
 F 2 "" H 6600 3850 60  0000 C CNN
@@
 	6600 3950 6600 3850
 $Comp
-L GND #PWR73
+L GND #PWR068
 U 1 1 54725F76
 P 6900 3750
-F 0 "#PWR73" H 6900 3750 30  0001 C CNN
+F 0 "#PWR068" H 6900 3750 30  0001 C CNN
 F 1 "GND" H 6900 3680 30  0001 C CNN
 F 2 "" H 6900 3750 60  0000 C CNN
@@
 	6900 3600 6900 3750
 $Comp
-L GND #PWR72
+L GND #PWR069
 U 1 1 54725F95
 P 6600 5150
-F 0 "#PWR72" H 6600 5150 30  0001 C CNN
+F 0 "#PWR069" H 6600 5150 30  0001 C CNN
 F 1 "GND" H 6600 5080 30  0001 C CNN
 F 2 "" H 6600 5150 60  0000 C CNN
@@
 	6450 5000 6600 5000
 Text GLabel 6850 4700 2    60   Input ~ 0
-MOTOR1F
+ACCELINT1
 Text GLabel 6850 4850 2    60   Input ~ 0
-MOTOR2F
+ACCELINT2
 Wire Wire Line
 	6450 4850 6850 4850
@@
 	6850 4400 6450 4400
 Text GLabel 6850 4100 2    60   Input ~ 0
-MPUINT
+PCINT
 Text GLabel 6850 4250 2    60   Input ~ 0
 RTCINT1
@@
 F 0 "R27" V 6880 2300 40  0000 C CNN
 F 1 "10K" V 6807 2301 40  0000 C CNN
-F 2 "~" V 6730 2300 30  0000 C CNN
+F 2 "" V 6730 2300 30  0001 C CNN
 F 3 "~" H 6800 2300 30  0000 C CNN
 	1    6800 2300

Commit message: Added most of the footprints needed to make this work
Parts:
- R27: footprint (none) -> Resistors_SMD:R_0603
Changed lines of the file:
@@
 $EndComp
 $Comp
-L 3V3 #PWR068
+L 3V3 #PWR069
 U 1 1 54725F5A
 P 6600 1750
-F 0 "#PWR068" H 6600 1850 40  0001 C CNN
+F 0 "#PWR069" H 6600 1850 40  0001 C CNN
 F 1 "3V3" H 6600 1875 40  0000 C CNN
 F 2 "" H 6600 1750 60  0000 C CNN
@@
 	6600 2550 6600 1750
 $Comp
-L 3V3 #PWR069
+L 3V3 #PWR070
 U 1 1 54725F6C
 P 6600 3850
-F 0 "#PWR069" H 6600 3950 40  0001 C CNN
+F 0 "#PWR070" H 6600 3950 40  0001 C CNN
 F 1 "3V3" H 6600 3975 40  0000 C CNN
 F 2 "" H 6600 3850 60  0000 C CNN
@@
 	6600 3950 6600 3850
 $Comp
-L GND #PWR070
+L GND #PWR071
 U 1 1 54725F76
 P 6900 3750
-F 0 "#PWR070" H 6900 3750 30  0001 C CNN
+F 0 "#PWR071" H 6900 3750 30  0001 C CNN
 F 1 "GND" H 6900 3680 30  0001 C CNN
 F 2 "" H 6900 3750 60  0000 C CNN
@@
 	6900 3600 6900 3750
 $Comp
-L GND #PWR071
+L GND #PWR072
 U 1 1 54725F95
 P 6600 5150
-F 0 "#PWR071" H 6600 5150 30  0001 C CNN
+F 0 "#PWR072" H 6600 5150 30  0001 C CNN
 F 1 "GND" H 6600 5080 30  0001 C CNN
 F 2 "" H 6600 5150 60  0000 C CNN
@@
 F 0 "R27" V 6880 2300 40  0000 C CNN
 F 1 "10K" V 6807 2301 40  0000 C CNN
-F 2 "" V 6730 2300 30  0001 C CNN
+F 2 "Resistors_SMD:R_0603" V 6730 2300 30  0001 C CNN
 F 3 "~" H 6800 2300 30  0000 C CNN
 	1    6800 2300
