File: board/mainboard/Power.sch (KiCad schematic (older format))
At the start: 5 parts

Commit message: Annotations, DRC fixing, and first round of footprint matching
Parts:
- gave numbers to parts that had none: 5
Changed lines of the file:
@@
 $EndDescr
 $Comp
-L TPS63001 REG?
+L TPS63001 REG1
 U 1 1 5472BB01
 P 6000 3700
-F 0 "REG?" H 6000 3850 60  0000 C CNN
+F 0 "REG1" H 6000 3850 60  0000 C CNN
 F 1 "TPS63001" H 6000 4050 60  0000 C CNN
 F 2 "" H 6000 3850 60  0000 C CNN
@@
 $EndComp
 $Comp
-L INDUCTOR L?
+L INDUCTOR L2
 U 1 1 5472BB10
 P 6000 3150
-F 0 "L?" V 5950 3150 40  0000 C CNN
+F 0 "L2" V 5950 3150 40  0000 C CNN
 F 1 "2.2uH" V 6100 3150 40  0000 C CNN
 F 2 "~" H 6000 3150 60  0000 C CNN
@@
 Connection ~ 6100 4350
 $Comp
-L GND #PWR?
+L GND #PWR066
 U 1 1 5472BB7C
 P 6100 4500
-F 0 "#PWR?" H 6100 4500 30  0001 C CNN
+F 0 "#PWR066" H 6100 4500 30  0001 C CNN
 F 1 "GND" H 6100 4430 30  0001 C CNN
 F 2 "" H 6100 4500 60  0000 C CNN
@@
 $EndComp
 $Comp
-L 3V3 #PWR?
+L 3V3 #PWR067
 U 1 1 5472BBB1
 P 6750 3600
-F 0 "#PWR?" H 6750 3700 40  0001 C CNN
+F 0 "#PWR067" H 6750 3700 40  0001 C CNN
 F 1 "3V3" H 6750 3725 40  0000 C CNN
 F 2 "" H 6750 3600 60  0000 C CNN
@@
 Connection ~ 6600 3650
 $Comp
-L C C?
+L C C28
 U 1 1 5472BBE8
 P 6750 4000
-F 0 "C?" H 6750 4100 40  0000 L CNN
+F 0 "C28" H 6750 4100 40  0000 L CNN
 F 1 "10uF" H 6756 3915 40  0000 L CNN
 F 2 "~" H 6788 3850 30  0000 C CNN
@@
 Connection ~ 6200 4350
 $Comp
-L C C?
+L C C27
 U 1 1 5472BC2B
 P 5250 4000
-F 0 "C?" H 5250 4100 40  0000 L CNN
+F 0 "C27" H 5250 4100 40  0000 L CNN
 F 1 "10uF" H 5256 3915 40  0000 L CNN
 F 2 "~" H 5288 3850 30  0000 C CNN
@@
 Connection ~ 5500 3650
 $Comp
-L CONN_2 P?
+L CONN_2 P12
 U 1 1 5472BC89
 P 4450 3750
-F 0 "P?" V 4400 3750 40  0000 C CNN
+F 0 "P12" V 4400 3750 40  0000 C CNN
 F 1 "POWER" V 4500 3750 40  0000 C CNN
 F 2 "" H 4450 3750 60  0000 C CNN

Commit message: Finished first draft of rev 1 board
Connections:
- net labels added: VCC
- wire segments 24 -> 25
Changed lines of the file:
@@
 Sheet 8 8
 Title ""
-Date "24 nov 2014"
+Date "25 nov 2014"
 Rev ""
 Comp ""
@@
 Connection ~ 6100 4350
 $Comp
-L GND #PWR066
+L GND #PWR067
 U 1 1 5472BB7C
 P 6100 4500
-F 0 "#PWR066" H 6100 4500 30  0001 C CNN
+F 0 "#PWR067" H 6100 4500 30  0001 C CNN
 F 1 "GND" H 6100 4430 30  0001 C CNN
 F 2 "" H 6100 4500 60  0000 C CNN
@@
 $EndComp
 $Comp
-L 3V3 #PWR067
+L 3V3 #PWR068
 U 1 1 5472BBB1
 P 6750 3600
-F 0 "#PWR067" H 6750 3700 40  0001 C CNN
+F 0 "#PWR068" H 6750 3700 40  0001 C CNN
 F 1 "3V3" H 6750 3725 40  0000 C CNN
 F 2 "" H 6750 3600 60  0000 C CNN
@@
 $EndComp
 Wire Wire Line
-	6450 3650 6750 3650
+	6450 3650 6900 3650
 Wire Wire Line
 	6750 3600 6750 3800
@@
 	5000 3850 5000 4350
 Connection ~ 5250 3650
+$Comp
+L VCC #PWR069
+U 1 1 54740F55
+P 6900 3600
+F 0 "#PWR069" H 6900 3700 30  0001 C CNN
+F 1 "VCC" H 6900 3700 30  0000 C CNN
+F 2 "" H 6900 3600 60  0000 C CNN
+F 3 "" H 6900 3600 60  0000 C CNN
+	1    6900 3600
+	1    0    0    -1
+$EndComp
+Wire Wire Line
+	6900 3650 6900 3600
 $EndSCHEMATC

Commit message: Finished draft 1 of Rev 2 layout
Parts:
- added C16: 1uF, ~, symbol C
- added U2: TLV702, symbol TLV702
Connections:
- net labels added: 1V8
- wire segments 25 -> 32
Changed lines of the file:
@@
 $Descr A4 11693 8268
 encoding utf-8
-Sheet 7 7
+Sheet 7 8
 Title ""
-Date "26 feb 2015"
+Date "1 mar 2015"
 Rev ""
 Comp ""
@@
 	5000 4350 6750 4350
 Wire Wire Line
-	6200 4350 6200 4250
-Wire Wire Line
 	6100 4250 6100 4500
 Connection ~ 6100 4350
@@
 L GND #PWR076
 U 1 1 5472BB7C
-P 6100 4500
-F 0 "#PWR076" H 6100 4500 30  0001 C CNN
-F 1 "GND" H 6100 4430 30  0001 C CNN
-F 2 "" H 6100 4500 60  0000 C CNN
-F 3 "" H 6100 4500 60  0000 C CNN
-	1    6100 4500
+P 5450 5900
+F 0 "#PWR076" H 5450 5900 30  0001 C CNN
+F 1 "GND" H 5450 5830 30  0001 C CNN
+F 2 "" H 5450 5900 60  0000 C CNN
+F 3 "" H 5450 5900 60  0000 C CNN
+	1    5450 5900
 	1    0    0    -1
 $EndComp
@@
 Wire Wire Line
 	6750 4350 6750 4200
-Connection ~ 6200 4350
 $Comp
 L C C27
@@
 Wire Wire Line
 	6900 3650 6900 3600
+$Comp
+L TLV702 U2
+U 1 1 54F23A79
+P 6100 5500
+F 0 "U2" H 6100 5400 60  0000 C CNN
+F 1 "TLV702" H 6100 5750 60  0000 C CNN
+F 2 "" H 6100 5500 60  0000 C CNN
+F 3 "" H 6100 5500 60  0000 C CNN
+	1    6100 5500
+	1    0    0    -1
+$EndComp
+$Comp
+L 3V3 #PWR079
+U 1 1 54F23A86
+P 5450 5300
+F 0 "#PWR079" H 5450 5400 40  0001 C CNN
+F 1 "3V3" H 5450 5425 40  0000 C CNN
+F 2 "" H 5450 5300 60  0000 C CNN
+F 3 "" H 5450 5300 60  0000 C CNN
+	1    5450 5300
+	1    0    0    -1
+$EndComp
+Wire Wire Line
+	5600 5400 5450 5400
+Wire Wire Line
+	5450 5300 5450 5500
+Wire Wire Line
+	5450 5500 5600 5500
+Connection ~ 5450 5400
+Wire Wire Line
+	5600 5750 5450 5750
+Wire Wire Line
+	5450 5750 5450 5900
+$Comp
+L 1V8 #PWR080
+U 1 1 54F23B0C
+P 6800 5200
+F 0 "#PWR080" H 6800 5340 20  0001 C CNN
+F 1 "1V8" H 6800 5310 30  0000 C CNN
+F 2 "" H 6800 5200 60  0000 C CNN
+F 3 "" H 6800 5200 60  0000 C CNN
+	1    6800 5200
+	1    0    0    -1
+$EndComp
+Wire Wire Line
+	6600 5400 6800 5400
+Wire Wire Line
+	6800 5200 6800 5500
+$Comp
+L C C16
+U 1 1 54F23B41
+P 6800 5700
+F 0 "C16" H 6850 5800 40  0000 L CNN
+F 1 "1uF" H 6806 5615 40  0000 L CNN
+F 2 "~" H 6838 5550 30  0000 C CNN
+F 3 "~" H 6800 5700 60  0000 C CNN
+	1    6800 5700
+	1    0    0    -1
+$EndComp
+$Comp
+L GND #PWR081
+U 1 1 54F23B47
+P 6800 6050
+F 0 "#PWR081" H 6800 6050 30  0001 C CNN
+F 1 "GND" H 6800 5980 30  0001 C CNN
+F 2 "" H 6800 6050 60  0000 C CNN
+F 3 "" H 6800 6050 60  0000 C CNN
+	1    6800 6050
+	1    0    0    -1
+$EndComp
+Wire Wire Line
+	6800 5900 6800 6050
+Connection ~ 6800 5400
+$Comp
+L GND #PWR082
+U 1 1 54F23E17
+P 6100 4500
+F 0 "#PWR082" H 6100 4500 30  0001 C CNN
+F 1 "GND" H 6100 4430 30  0001 C CNN
+F 2 "" H 6100 4500 60  0000 C CNN
+F 3 "" H 6100 4500 60  0000 C CNN
+	1    6100 4500
+	1    0    0    -1
+$EndComp
 $EndSCHEMATC
