File: board/mainboard/Power.sch (KiCad schematic (older format))
At the start: 16 parts, among them P12 POWER, Q2 IRLML6402, Q3 IRLML6402, U2 TLV702, U4 TPS62142, U5 MCP6001R

Commit message: Completed work on I2C motor driver unit. 1) Added new motor drivers + I2C controller 2) Added headers for SWD for the KE40 device
Connections:
- wire segments 63 -> 85
Changed lines of the file:
@@
 $Descr A4 11693 8268
 encoding utf-8
-Sheet 7 9
+Sheet 7 10
 Title ""
 Date "3 mar 2015"
@@
 $EndDescr
 $Comp
-L GND #PWR72
+L GND #PWR79
 U 1 1 5472BB7C
 P 5450 5900
-F 0 "#PWR72" H 5450 5900 30  0001 C CNN
+F 0 "#PWR79" H 5450 5900 30  0001 C CNN
 F 1 "GND" H 5450 5830 30  0001 C CNN
 F 2 "" H 5450 5900 60  0000 C CNN
@@
 $EndComp
 $Comp
-L 3V3 #PWR71
+L 3V3 #PWR78
 U 1 1 54F23A86
 P 5450 5300
-F 0 "#PWR71" H 5450 5400 40  0001 C CNN
+F 0 "#PWR78" H 5450 5400 40  0001 C CNN
 F 1 "3V3" H 5450 5425 40  0000 C CNN
 F 2 "" H 5450 5300 60  0000 C CNN
@@
 $EndComp
 $Comp
-L 1V8 #PWR76
+L 1V8 #PWR83
 U 1 1 54F23B0C
 P 6800 5200
-F 0 "#PWR76" H 6800 5340 20  0001 C CNN
+F 0 "#PWR83" H 6800 5340 20  0001 C CNN
 F 1 "1V8" H 6800 5310 30  0000 C CNN
 F 2 "" H 6800 5200 60  0000 C CNN
@@
 $EndComp
 $Comp
-L GND #PWR77
+L GND #PWR84
 U 1 1 54F23B47
 P 6800 6050
-F 0 "#PWR77" H 6800 6050 30  0001 C CNN
+F 0 "#PWR84" H 6800 6050 30  0001 C CNN
 F 1 "GND" H 6800 5980 30  0001 C CNN
 F 2 "" H 6800 6050 60  0000 C CNN
@@
 VBAT
 $Comp
-L GND #PWR67
+L GND #PWR74
 U 1 1 55A31E2C
 P 1625 3875
-F 0 "#PWR67" H 1625 3875 30  0001 C CNN
+F 0 "#PWR74" H 1625 3875 30  0001 C CNN
 F 1 "GND" H 1625 3805 30  0001 C CNN
 F 2 "" H 1625 3875 60  0000 C CNN
@@
 $EndComp
 $Comp
-L GND #PWR75
+L GND #PWR82
 U 1 1 55A32978
 P 6050 5000
-F 0 "#PWR75" H 6050 5000 30  0001 C CNN
+F 0 "#PWR82" H 6050 5000 30  0001 C CNN
 F 1 "GND" H 6050 4930 30  0001 C CNN
 F 2 "" H 6050 5000 60  0000 C CNN
@@
 	5600 5400 5450 5400
 Wire Wire Line
-	5450 5300 5450 5500
+	5450 5300 5450 5400
+Wire Wire Line
+	5450 5400 5450 5500
 Wire Wire Line
 	5450 5500 5600 5500
@@
 	6600 5400 6800 5400
 Wire Wire Line
-	6800 5200 6800 5500
+	6800 5200 6800 5400
+Wire Wire Line
+	6800 5400 6800 5500
 Wire Wire Line
 	6800 5900 6800 6050
@@
 	5475 3575 5275 3575
 Wire Wire Line
-	5275 3450 5275 3775
+	5275 3450 5275 3575
+Wire Wire Line
+	5275 3575 5275 3675
+Wire Wire Line
+	5275 3675 5275 3775
 Connection ~ 5275 3450
 Wire Wire Line
@@
 	1525 3550 1625 3550
 Wire Wire Line
-	1625 3550 1625 3875
-Wire Wire Line
-	4925 3450 5475 3450
+	1625 3550 1625 3800
+Wire Wire Line
+	1625 3800 1625 3875
+Wire Wire Line
+	4925 3450 5050 3450
+Wire Wire Line
+	5050 3450 5275 3450
+Wire Wire Line
+	5275 3450 5475 3450
 Wire Wire Line
 	1600 3450 1525 3450
@@
 Connection ~ 1625 3800
 Wire Wire Line
-	2000 3450 2225 3450
+	2000 3450 2375 3450
 Wire Wire Line
 	6150 4825 6150 4650
 Wire Wire Line
-	5050 4825 7375 4825
-Wire Wire Line
-	6050 4650 6050 5000
+	5050 4825 5275 4825
+Wire Wire Line
+	5275 4825 5950 4825
+Wire Wire Line
+	5950 4825 6050 4825
+Wire Wire Line
+	6050 4825 6150 4825
+Wire Wire Line
+	6150 4825 6725 4825
+Wire Wire Line
+	6725 4825 6875 4825
+Wire Wire Line
+	6875 4825 7375 4825
+Wire Wire Line
+	6050 4650 6050 4825
+Wire Wire Line
+	6050 4825 6050 5000
 Wire Wire Line
 	5950 4825 5950 4650
@@
 $EndComp
 Wire Wire Line
-	7375 3975 6625 3975
+	7375 3975 6750 3975
+Wire Wire Line
+	6750 3975 6625 3975
 Connection ~ 6875 4825
 Wire Wire Line
-	7375 3425 7375 4200
+	7375 3425 7375 3650
+Wire Wire Line
+	7375 3650 7375 3975
+Wire Wire Line
+	7375 3975 7375 4200
 Wire Wire Line
 	6625 3850 6750 3850
@@
 $EndComp
 Wire Wire Line
-	6625 3650 6800 3650
+	6625 3650 6700 3650
+Wire Wire Line
+	6700 3650 6800 3650
 Wire Wire Line
 	6700 3750 6625 3750
 Wire Wire Line
-	6700 3550 6700 3750
+	6700 3550 6700 3650
+Wire Wire Line
+	6700 3650 6700 3750
 Connection ~ 6700 3650
 Wire Wire Line
 	6700 3550 6625 3550
 Wire Wire Line
-	7300 3650 7700 3650
+	7300 3650 7375 3650
+Wire Wire Line
+	7375 3650 7700 3650
 Connection ~ 7375 3975
 Wire Wire Line
@@
 Connection ~ 7375 3650
 $Comp
-L 3V3 #PWR79
+L 3V3 #PWR86
 U 1 1 55A33743
 P 7700 3650
-F 0 "#PWR79" H 7700 3750 40  0001 C CNN
+F 0 "#PWR86" H 7700 3750 40  0001 C CNN
 F 1 "3V3" H 7700 3775 40  0000 C CNN
 F 2 "" H 7700 3650 60  0000 C CNN
@@
 	6775 2225 6775 2325
 $Comp
-L 3V3 #PWR78
+L 3V3 #PWR85
 U 1 1 55A3575B
 P 7100 2150
-F 0 "#PWR78" H 7100 2250 40  0001 C CNN
+F 0 "#PWR85" H 7100 2250 40  0001 C CNN
 F 1 "3V3" H 7100 2275 40  0000 C CNN
 F 2 "" H 7100 2150 60  0000 C CNN
@@
 	7100 2325 7100 2150
 $Comp
-L 3V3 #PWR73
+L 3V3 #PWR80
 U 1 1 55A359B2
 P 5625 1575
-F 0 "#PWR73" H 5625 1675 40  0001 C CNN
+F 0 "#PWR80" H 5625 1675 40  0001 C CNN
 F 1 "3V3" H 5625 1700 40  0000 C CNN
 F 2 "" H 5625 1575 60  0000 C CNN
@@
 $EndComp
 $Comp
-L GND #PWR74
+L GND #PWR81
 U 1 1 55A35AB9
 P 5625 2575
-F 0 "#PWR74" H 5625 2575 30  0001 C CNN
+F 0 "#PWR81" H 5625 2575 30  0001 C CNN
 F 1 "GND" H 5625 2505 30  0001 C CNN
 F 2 "" H 5625 2575 60  0000 C CNN
@@
 $EndComp
 Wire Wire Line
-	4275 2825 4275 2950
+	4275 2825 4275 2900
+Wire Wire Line
+	4275 2900 4275 2950
 Connection ~ 4275 2900
 $Comp
-L 3V3 #PWR69
+L 3V3 #PWR76
 U 1 1 55A364F9
 P 4275 2250
-F 0 "#PWR69" H 4275 2350 40  0001 C CNN
+F 0 "#PWR76" H 4275 2350 40  0001 C CNN
 F 1 "3V3" H 4275 2375 40  0000 C CNN
 F 2 "" H 4275 2250 60  0000 C CNN
@@
 	4275 2325 4275 2250
 $Comp
-L GND #PWR70
+L GND #PWR77
 U 1 1 55A36665
 P 4275 3525
-F 0 "#PWR70" H 4275 3525 30  0001 C CNN
+F 0 "#PWR77" H 4275 3525 30  0001 C CNN
 F 1 "GND" H 4275 3455 30  0001 C CNN
 F 2 "" H 4275 3525 60  0000 C CNN
@@
 $EndComp
 Wire Wire Line
-	4275 1325 4275 1450
+	4275 1325 4275 1400
+Wire Wire Line
+	4275 1400 4275 1450
 Connection ~ 4275 1400
 Wire Wire Line
 	4275 825  4275 750
 $Comp
-L GND #PWR68
+L GND #PWR75
 U 1 1 55A36FC3
 P 4275 2025
-F 0 "#PWR68" H 4275 2025 30  0001 C CNN
+F 0 "#PWR75" H 4275 2025 30  0001 C CNN
 F 1 "GND" H 4275 1955 30  0001 C CNN
 F 2 "" H 4275 2025 60  0000 C CNN
@@
 Text Notes 1150 4075 0    60   ~ 0
 Reverse Battery Protection\n
+Text GLabel 2375 3450 2    60   Input ~ 0
+VBAT
 $EndSCHEMATC
