File: board/mainboard/Power.sch (KiCad schematic (older format))
At the start: 16 parts, among them P12 POWER, Q2 IRLML6402, Q3 IRLML6402, U2 TLV702, U4 TPS62142, U5 MCP6001R

Commit message: Completed rev 3.0 schematics.
1) Replaced MPU with STM Accelerometer
Parts:
- C16: footprint ~ -> (none)
- Q2, Q3: footprint SOT-23 -> Transistors_SMD:sot23
Connections:
- net labels added: CMP_VBAT
- wire segments 85 -> 65
Changed lines of the file:
@@
 $Descr A4 11693 8268
 encoding utf-8
-Sheet 7 10
+Sheet 8 10
 Title ""
 Date "3 mar 2015"
@@
 $EndDescr
 $Comp
-L GND #PWR79
+L GND #PWR070
 U 1 1 5472BB7C
 P 5450 5900
-F 0 "#PWR79" H 5450 5900 30  0001 C CNN
+F 0 "#PWR070" H 5450 5900 30  0001 C CNN
 F 1 "GND" H 5450 5830 30  0001 C CNN
 F 2 "" H 5450 5900 60  0000 C CNN
@@
 F 0 "P12" V 1275 3500 40  0000 C CNN
 F 1 "POWER" V 1375 3500 40  0000 C CNN
-F 2 "" H 1325 3500 60  0000 C CNN
+F 2 "" H 1325 3500 60  0001 C CNN
 F 3 "" H 1325 3500 60  0000 C CNN
 	1    1325 3500
@@
 F 0 "U2" H 6100 5400 60  0000 C CNN
 F 1 "TLV702" H 6100 5750 60  0000 C CNN
-F 2 "" H 6100 5500 60  0000 C CNN
+F 2 "" H 6100 5500 60  0001 C CNN
 F 3 "" H 6100 5500 60  0000 C CNN
 	1    6100 5500
@@
 $EndComp
 $Comp
-L 3V3 #PWR78
+L 3V3 #PWR071
 U 1 1 54F23A86
 P 5450 5300
-F 0 "#PWR78" H 5450 5400 40  0001 C CNN
+F 0 "#PWR071" H 5450 5400 40  0001 C CNN
 F 1 "3V3" H 5450 5425 40  0000 C CNN
 F 2 "" H 5450 5300 60  0000 C CNN
@@
 $EndComp
 $Comp
-L 1V8 #PWR83
+L 1V8 #PWR072
 U 1 1 54F23B0C
 P 6800 5200
-F 0 "#PWR83" H 6800 5340 20  0001 C CNN
+F 0 "#PWR072" H 6800 5340 20  0001 C CNN
 F 1 "1V8" H 6800 5310 30  0000 C CNN
 F 2 "" H 6800 5200 60  0000 C CNN
@@
 F 0 "C16" H 6850 5800 40  0000 L CNN
 F 1 "1uF" H 6806 5615 40  0000 L CNN
-F 2 "~" H 6838 5550 30  0000 C CNN
+F 2 "" H 6838 5550 30  0001 C CNN
 F 3 "~" H 6800 5700 60  0000 C CNN
 	1    6800 5700
@@
 $EndComp
 $Comp
-L GND #PWR84
+L GND #PWR073
 U 1 1 54F23B47
 P 6800 6050
-F 0 "#PWR84" H 6800 6050 30  0001 C CNN
+F 0 "#PWR073" H 6800 6050 30  0001 C CNN
 F 1 "GND" H 6800 5980 30  0001 C CNN
 F 2 "" H 6800 6050 60  0000 C CNN
@@
 F 0 "U4" H 5725 5775 60  0000 C CNN
 F 1 "TPS62142" H 6050 4925 60  0000 C CNN
-F 2 "" H 5950 4500 60  0000 C CNN
+F 2 "" H 5950 4500 60  0001 C CNN
 F 3 "" H 5950 4500 60  0000 C CNN
 	1    5875 4500
@@
 VBAT
 $Comp
-L GND #PWR74
+L GND #PWR074
 U 1 1 55A31E2C
 P 1625 3875
-F 0 "#PWR74" H 1625 3875 30  0001 C CNN
+F 0 "#PWR074" H 1625 3875 30  0001 C CNN
 F 1 "GND" H 1625 3805 30  0001 C CNN
 F 2 "" H 1625 3875 60  0000 C CNN
@@
 F 0 "Q2" H 1800 3402 40  0000 R CNN
 F 1 "IRLML6402" V 2025 3700 40  0000 R CNN
-F 2 "SOT-23" H 1560 3650 29  0000 C CNN
+F 2 "Transistors_SMD:sot23" H 1560 3650 29  0000 C CNN
 F 3 "" H 1800 3550 60  0000 C CNN
 	1    1800 3550
@@
 F 0 "C7" H 5275 4625 40  0000 L CNN
 F 1 "390pF" H 5281 4440 40  0000 L CNN
-F 2 "" H 5313 4375 30  0000 C CNN
+F 2 "" H 5313 4375 30  0001 C CNN
 F 3 "" H 5275 4525 60  0000 C CNN
 	1    5275 4525
@@
 $EndComp
 $Comp
-L GND #PWR82
+L GND #PWR075
 U 1 1 55A32978
 P 6050 5000
-F 0 "#PWR82" H 6050 5000 30  0001 C CNN
+F 0 "#PWR075" H 6050 5000 30  0001 C CNN
 F 1 "GND" H 6050 4930 30  0001 C CNN
 F 2 "" H 6050 5000 60  0000 C CNN
@@
 	5600 5400 5450 5400
 Wire Wire Line
-	5450 5300 5450 5400
-Wire Wire Line
-	5450 5400 5450 5500
+	5450 5300 5450 5500
 Wire Wire Line
 	5450 5500 5600 5500
@@
 	6600 5400 6800 5400
 Wire Wire Line
-	6800 5200 6800 5400
-Wire Wire Line
-	6800 5400 6800 5500
+	6800 5200 6800 5500
 Wire Wire Line
 	6800 5900 6800 6050
@@
 	5475 3575 5275 3575
 Wire Wire Line
-	5275 3450 5275 3575
-Wire Wire Line
-	5275 3575 5275 3675
-Wire Wire Line
-	5275 3675 5275 3775
+	5275 3450 5275 3775
 Connection ~ 5275 3450
 Wire Wire Line
@@
 	1525 3550 1625 3550
 Wire Wire Line
-	1625 3550 1625 3800
-Wire Wire Line
-	1625 3800 1625 3875
-Wire Wire Line
-	4925 3450 5050 3450
-Wire Wire Line
-	5050 3450 5275 3450
-Wire Wire Line
-	5275 3450 5475 3450
+	1625 3550 1625 3875
+Wire Wire Line
+	4925 3450 5475 3450
 Wire Wire Line
 	1600 3450 1525 3450
@@
 	6150 4825 6150 4650
 Wire Wire Line
-	5050 4825 5275 4825
-Wire Wire Line
-	5275 4825 5950 4825
-Wire Wire Line
-	5950 4825 6050 4825
-Wire Wire Line
-	6050 4825 6150 4825
-Wire Wire Line
-	6150 4825 6725 4825
-Wire Wire Line
-	6725 4825 6875 4825
-Wire Wire Line
-	6875 4825 7375 4825
-Wire Wire Line
-	6050 4650 6050 4825
-Wire Wire Line
-	6050 4825 6050 5000
+	5050 4825 7375 4825
+Wire Wire Line
+	6050 4650 6050 5000
 Wire Wire Line
 	5950 4825 5950 4650
@@
 F 0 "C6" H 5050 4625 40  0000 L CNN
 F 1 "10uF" H 5050 4425 40  0000 L CNN
-F 2 "" H 5088 4375 30  0000 C CNN
+F 2 "" H 5088 4375 30  0001 C CNN
 F 3 "" H 5050 4525 60  0000 C CNN
 	1    5050 4525
@@
 F 0 "C10" H 7375 4500 40  0000 L CNN
 F 1 "22uF" H 7381 4315 40  0000 L CNN
-F 2 "" H 7413 4250 30  0000 C CNN
+F 2 "" H 7413 4250 30  0001 C CNN
 F 3 "" H 7375 4400 60  0000 C CNN
 	1    7375 4400
@@
 $EndComp
 Wire Wire Line
-	7375 3975 6750 3975
-Wire Wire Line
-	6750 3975 6625 3975
+	7375 3975 6625 3975
 Connection ~ 6875 4825
 Wire Wire Line
-	7375 3425 7375 3650
-Wire Wire Line
-	7375 3650 7375 3975
-Wire Wire Line
-	7375 3975 7375 4200
+	7375 3425 7375 4200
 Wire Wire Line
 	6625 3850 6750 3850
@@
 F 0 "L1" H 7050 3750 50  0000 C CNN
 F 1 "2.2uH" H 7050 3600 50  0000 C CNN
-F 2 "" H 7050 3650 60  0000 C CNN
+F 2 "" H 7050 3650 60  0001 C CNN
 F 3 "" H 7050 3650 60  0000 C CNN
 	1    7050 3650
@@
 $EndComp
 Wire Wire Line
-	6625 3650 6700 3650
-Wire Wire Line
-	6700 3650 6800 3650
+	6625 3650 6800 3650
 Wire Wire Line
 	6700 3750 6625 3750
 Wire Wire Line
-	6700 3550 6700 3650
-Wire Wire Line
-	6700 3650 6700 3750
+	6700 3550 6700 3750
 Connection ~ 6700 3650
 Wire Wire Line
 	6700 3550 6625 3550
 Wire Wire Line
-	7300 3650 7375 3650
-Wire Wire Line
-	7375 3650 7700 3650
+	7300 3650 7700 3650
 Connection ~ 7375 3975
 Wire Wire Line
@@
 Connection ~ 7375 3650
 $Comp
-L 3V3 #PWR86
+L 3V3 #PWR076
 U 1 1 55A33743
 P 7700 3650
-F 0 "#PWR86" H 7700 3750 40  0001 C CNN
+F 0 "#PWR076" H 7700 3750 40  0001 C CNN
 F 1 "3V3" H 7700 3775 40  0000 C CNN
 F 2 "" H 7700 3650 60  0000 C CNN
@@
 F 0 "R34" V 6975 3425 40  0000 C CNN
 F 1 "100k" V 7057 3426 40  0000 C CNN
-F 2 "" V 6980 3425 30  0000 C CNN
+F 2 "" V 6980 3425 30  0001 C CNN
 F 3 "" H 7050 3425 30  0000 C CNN
 	1    7050 3425
@@
 F 0 "U5" H 5775 2700 60  0000 C CNN
 F 1 "MCP6001R" H 5950 2775 60  0000 C CNN
-F 2 "" H 5375 2550 60  0000 C CNN
+F 2 "" H 5375 2550 60  0001 C CNN
 F 3 "" H 5375 2550 60  0000 C CNN
 	1    5375 2550
@@
 F 0 "Q3" H 6675 1877 40  0000 R CNN
 F 1 "IRLML6402" H 6675 2174 40  0000 R CNN
-F 2 "SOT-23" H 6435 2125 29  0000 C CNN
+F 2 "Transistors_SMD:sot23" H 6435 2125 29  0000 C CNN
 F 3 "" H 6675 2025 60  0000 C CNN
 	1    6675 2025
@@
 	6775 2225 6775 2325
 $Comp
-L 3V3 #PWR85
+L 3V3 #PWR077
 U 1 1 55A3575B
 P 7100 2150
-F 0 "#PWR85" H 7100 2250 40  0001 C CNN
+F 0 "#PWR077" H 7100 2250 40  0001 C CNN
 F 1 "3V3" H 7100 2275 40  0000 C CNN
 F 2 "" H 7100 2150 60  0000 C CNN
@@
 	7100 2325 7100 2150
 $Comp
-L 3V3 #PWR80
+L 3V3 #PWR078
 U 1 1 55A359B2
 P 5625 1575
-F 0 "#PWR80" H 5625 1675 40  0001 C CNN
+F 0 "#PWR078" H 5625 1675 40  0001 C CNN
 F 1 "3V3" H 5625 1700 40  0000 C CNN
 F 2 "" H 5625 1575 60  0000 C CNN
@@
 $EndComp
 $Comp
-L GND #PWR81
+L GND #PWR079
 U 1 1 55A35AB9
 P 5625 2575
-F 0 "#PWR81" H 5625 2575 30  0001 C CNN
+F 0 "#PWR079" H 5625 2575 30  0001 C CNN
 F 1 "GND" H 5625 2505 30  0001 C CNN
 F 2 "" H 5625 2575 60  0000 C CNN
@@
 F 0 "R37" V 4200 2575 40  0000 C CNN
 F 1 "33k" V 4282 2576 40  0000 C CNN
-F 2 "" V 4205 2575 30  0000 C CNN
+F 2 "" V 4205 2575 30  0001 C CNN
 F 3 "" H 4275 2575 30  0000 C CNN
 	1    4275 2575
@@
 F 0 "R38" V 4200 3200 40  0000 C CNN
 F 1 "10k" V 4282 3201 40  0000 C CNN
-F 2 "" V 4205 3200 30  0000 C CNN
+F 2 "" V 4205 3200 30  0001 C CNN
 F 3 "" H 4275 3200 30  0000 C CNN
 	1    4275 3200
@@
 $EndComp
 Wire Wire Line
-	4275 2825 4275 2900
-Wire Wire Line
-	4275 2900 4275 2950
+	4275 2825 4275 2950
 Connection ~ 4275 2900
 $Comp
-L 3V3 #PWR76
+L 3V3 #PWR080
 U 1 1 55A364F9
 P 4275 2250
-F 0 "#PWR76" H 4275 2350 40  0001 C CNN
+F 0 "#PWR080" H 4275 2350 40  0001 C CNN
 F 1 "3V3" H 4275 2375 40  0000 C CNN
 F 2 "" H 4275 2250 60  0000 C CNN
@@
 	4275 2325 4275 2250
 $Comp
-L GND #PWR77
+L GND #PWR081
 U 1 1 55A36665
 P 4275 3525
-F 0 "#PWR77" H 4275 3525 30  0001 C CNN
+F 0 "#PWR081" H 4275 3525 30  0001 C CNN
 F 1 "GND" H 4275 3455 30  0001 C CNN
 F 2 "" H 4275 3525 60  0000 C CNN
@@
 F 0 "R35" V 4200 1075 40  0000 C CNN
 F 1 "33k" V 4282 1076 40  0000 C CNN
-F 2 "" V 4205 1075 30  0000 C CNN
+F 2 "" V 4205 1075 30  0001 C CNN
 F 3 "" H 4275 1075 30  0000 C CNN
 	1    4275 1075
@@
 F 0 "R36" V 4200 1700 40  0000 C CNN
 F 1 "10k" V 4282 1701 40  0000 C CNN
-F 2 "" V 4205 1700 30  0000 C CNN
+F 2 "" V 4205 1700 30  0001 C CNN
 F 3 "" H 4275 1700 30  0000 C CNN
 	1    4275 1700
@@
 $EndComp
 Wire Wire Line
-	4275 1325 4275 1400
-Wire Wire Line
-	4275 1400 4275 1450
+	4275 1325 4275 1450
 Connection ~ 4275 1400
 Wire Wire Line
 	4275 825  4275 750
 $Comp
-L GND #PWR75
+L GND #PWR082
 U 1 1 55A36FC3
 P 4275 2025
-F 0 "#PWR75" H 4275 2025 30  0001 C CNN
+F 0 "#PWR082" H 4275 2025 30  0001 C CNN
 F 1 "GND" H 4275 1955 30  0001 C CNN
 F 2 "" H 4275 2025 60  0000 C CNN
@@
 Wire Wire Line
 	4975 1950 4975 1400
-Wire Wire Line
-	4975 1400 4275 1400
 Text Notes 1150 4075 0    60   ~ 0
 Reverse Battery Protection\n
 Text GLabel 2375 3450 2    60   Input ~ 0
 VBAT
+Text Label 4875 1400 2    60   ~ 0
+CMP_VBAT
+Connection ~ 4975 1400
+Text GLabel 5025 1400 2    60   Input ~ 0
+CMP_VBAT
+Wire Wire Line
+	4275 1400 5025 1400
+$Comp
+L PWR_FLAG #FLG083
+U 1 1 55A90C84
+P 7525 3625
+F 0 "#FLG083" H 7525 3720 30  0001 C CNN
+F 1 "PWR_FLAG" H 7525 3805 30  0000 C CNN
+F 2 "" H 7525 3625 60  0000 C CNN
+F 3 "" H 7525 3625 60  0000 C CNN
+	1    7525 3625
+	1    0    0    -1
+$EndComp
+Wire Wire Line
+	7525 3625 7525 3650
+Connection ~ 7525 3650
+$Comp
+L PWR_FLAG #FLG084
+U 1 1 55A8BD1F
+P 2250 3300
+F 0 "#FLG084" H 2250 3395 30  0001 C CNN
+F 1 "PWR_FLAG" H 2250 3480 30  0000 C CNN
+F 2 "" H 2250 3300 60  0000 C CNN
+F 3 "" H 2250 3300 60  0000 C CNN
+	1    2250 3300
+	1    0    0    -1
+$EndComp
+Wire Wire Line
+	2250 3300 2250 3450
+Connection ~ 2250 3450
 $EndSCHEMATC

Commit message: Added most of the footprints needed to make this work
Parts:
- C10, C6: footprint (none) -> Capacitors_SMD:c_0805
- C16, C7: footprint (none) -> Capacitors_SMD:c_0603
- L1: footprint (none) -> footprints:SDR0403-2R2
- Q2, Q3: footprint Transistors_SMD:sot23 -> footprints:IRLML6402
- R34, R35, R36, R37, R38: footprint (none) -> Resistors_SMD:R_0603
- U4: footprint (none) -> footprints:TPS62142
- U5: footprint (none) -> footprints:MCP6001R
Connections:
- wire segments 65 -> 67
Changed lines of the file:
@@
 $EndDescr
 $Comp
-L GND #PWR072
+L GND #PWR073
 U 1 1 5472BB7C
 P 5450 5900
-F 0 "#PWR072" H 5450 5900 30  0001 C CNN
+F 0 "#PWR073" H 5450 5900 30  0001 C CNN
 F 1 "GND" H 5450 5830 30  0001 C CNN
 F 2 "" H 5450 5900 60  0000 C CNN
@@
 $EndComp
 $Comp
-L 3V3 #PWR073
+L 3V3 #PWR074
 U 1 1 54F23A86
 P 5450 5300
-F 0 "#PWR073" H 5450 5400 40  0001 C CNN
+F 0 "#PWR074" H 5450 5400 40  0001 C CNN
 F 1 "3V3" H 5450 5425 40  0000 C CNN
 F 2 "" H 5450 5300 60  0000 C CNN
@@
 $EndComp
 $Comp
-L 1V8 #PWR074
+L 1V8 #PWR075
 U 1 1 54F23B0C
 P 6800 5200
-F 0 "#PWR074" H 6800 5340 20  0001 C CNN
+F 0 "#PWR075" H 6800 5340 20  0001 C CNN
 F 1 "1V8" H 6800 5310 30  0000 C CNN
 F 2 "" H 6800 5200 60  0000 C CNN
@@
 F 0 "C16" H 6850 5800 40  0000 L CNN
 F 1 "1uF" H 6806 5615 40  0000 L CNN
-F 2 "" H 6838 5550 30  0001 C CNN
+F 2 "Capacitors_SMD:c_0603" H 6838 5550 30  0001 C CNN
 F 3 "~" H 6800 5700 60  0000 C CNN
 	1    6800 5700
@@
 $EndComp
 $Comp
-L GND #PWR075
+L GND #PWR076
 U 1 1 54F23B47
 P 6800 6050
-F 0 "#PWR075" H 6800 6050 30  0001 C CNN
+F 0 "#PWR076" H 6800 6050 30  0001 C CNN
 F 1 "GND" H 6800 5980 30  0001 C CNN
 F 2 "" H 6800 6050 60  0000 C CNN
@@
 F 0 "U4" H 5725 5775 60  0000 C CNN
 F 1 "TPS62142" H 6050 4925 60  0000 C CNN
-F 2 "" H 5950 4500 60  0001 C CNN
+F 2 "footprints:TPS62142" H 5950 4500 60  0001 C CNN
 F 3 "" H 5950 4500 60  0000 C CNN
 	1    5875 4500
@@
 VBAT
 $Comp
-L GND #PWR076
+L GND #PWR077
 U 1 1 55A31E2C
 P 1625 3875
-F 0 "#PWR076" H 1625 3875 30  0001 C CNN
+F 0 "#PWR077" H 1625 3875 30  0001 C CNN
 F 1 "GND" H 1625 3805 30  0001 C CNN
 F 2 "" H 1625 3875 60  0000 C CNN
@@
 F 0 "Q2" H 1800 3402 40  0000 R CNN
 F 1 "IRLML6402" V 2025 3700 40  0000 R CNN
-F 2 "Transistors_SMD:sot23" H 1560 3650 29  0000 C CNN
+F 2 "footprints:IRLML6402" H 1560 3650 29  0000 C CNN
 F 3 "" H 1800 3550 60  0000 C CNN
 	1    1800 3550
@@
 F 0 "C7" H 5275 4625 40  0000 L CNN
 F 1 "390pF" H 5281 4440 40  0000 L CNN
-F 2 "" H 5313 4375 30  0001 C CNN
+F 2 "Capacitors_SMD:c_0603" H 5313 4375 30  0001 C CNN
 F 3 "" H 5275 4525 60  0000 C CNN
 	1    5275 4525
@@
 $EndComp
 $Comp
-L GND #PWR077
+L GND #PWR078
 U 1 1 55A32978
 P 6050 5000
-F 0 "#PWR077" H 6050 5000 30  0001 C CNN
+F 0 "#PWR078" H 6050 5000 30  0001 C CNN
 F 1 "GND" H 6050 4930 30  0001 C CNN
 F 2 "" H 6050 5000 60  0000 C CNN
@@
 F 0 "C6" H 5050 4625 40  0000 L CNN
 F 1 "10uF" H 5050 4425 40  0000 L CNN
-F 2 "" H 5088 4375 30  0001 C CNN
+F 2 "Capacitors_SMD:c_0805" H 5088 4375 30  0001 C CNN
 F 3 "" H 5050 4525 60  0000 C CNN
 	1    5050 4525
@@
 F 0 "C10" H 7375 4500 40  0000 L CNN
 F 1 "22uF" H 7381 4315 40  0000 L CNN
-F 2 "" H 7413 4250 30  0001 C CNN
+F 2 "Capacitors_SMD:c_0805" H 7413 4250 30  0001 C CNN
 F 3 "" H 7375 4400 60  0000 C CNN
 	1    7375 4400
@@
 F 0 "L1" H 7050 3750 50  0000 C CNN
 F 1 "2.2uH" H 7050 3600 50  0000 C CNN
-F 2 "" H 7050 3650 60  0001 C CNN
+F 2 "footprints:SDR0403-2R2" H 7050 3650 60  0001 C CNN
 F 3 "" H 7050 3650 60  0000 C CNN
 	1    7050 3650
@@
 Connection ~ 7375 3650
 $Comp
-L 3V3 #PWR078
+L 3V3 #PWR079
 U 1 1 55A33743
 P 7700 3650
-F 0 "#PWR078" H 7700 3750 40  0001 C CNN
+F 0 "#PWR079" H 7700 3750 40  0001 C CNN
 F 1 "3V3" H 7700 3775 40  0000 C CNN
 F 2 "" H 7700 3650 60  0000 C CNN
@@
 F 0 "R34" V 6975 3425 40  0000 C CNN
 F 1 "100k" V 7057 3426 40  0000 C CNN
-F 2 "" V 6980 3425 30  0001 C CNN
+F 2 "Resistors_SMD:R_0603" V 6980 3425 30  0001 C CNN
 F 3 "" H 7050 3425 30  0000 C CNN
 	1    7050 3425
@@
 F 0 "U5" H 5775 2700 60  0000 C CNN
 F 1 "MCP6001R" H 5950 2775 60  0000 C CNN
-F 2 "" H 5375 2550 60  0001 C CNN
+F 2 "footprints:MCP6001R" H 5375 2550 60  0001 C CNN
 F 3 "" H 5375 2550 60  0000 C CNN
 	1    5375 2550
@@
 F 0 "Q3" H 6675 1877 40  0000 R CNN
 F 1 "IRLML6402" H 6675 2174 40  0000 R CNN
-F 2 "Transistors_SMD:sot23" H 6435 2125 29  0000 C CNN
+F 2 "footprints:IRLML6402" H 6435 2125 29  0000 C CNN
 F 3 "" H 6675 2025 60  0000 C CNN
 	1    6675 2025
@@
 	6775 2225 6775 2325
 $Comp
-L 3V3 #PWR079
+L 3V3 #PWR080
 U 1 1 55A3575B
 P 7100 2150
-F 0 "#PWR079" H 7100 2250 40  0001 C CNN
+F 0 "#PWR080" H 7100 2250 40  0001 C CNN
 F 1 "3V3" H 7100 2275 40  0000 C CNN
 F 2 "" H 7100 2150 60  0000 C CNN
@@
 	7100 2325 7100 2150
 $Comp
-L 3V3 #PWR080
+L 3V3 #PWR081
 U 1 1 55A359B2
 P 5625 1575
-F 0 "#PWR080" H 5625 1675 40  0001 C CNN
+F 0 "#PWR081" H 5625 1675 40  0001 C CNN
 F 1 "3V3" H 5625 1700 40  0000 C CNN
 F 2 "" H 5625 1575 60  0000 C CNN
@@
 $EndComp
 $Comp
-L GND #PWR081
+L GND #PWR082
 U 1 1 55A35AB9
 P 5625 2575
-F 0 "#PWR081" H 5625 2575 30  0001 C CNN
+F 0 "#PWR082" H 5625 2575 30  0001 C CNN
 F 1 "GND" H 5625 2505 30  0001 C CNN
 F 2 "" H 5625 2575 60  0000 C CNN
@@
 F 0 "R37" V 4200 2575 40  0000 C CNN
 F 1 "33k" V 4282 2576 40  0000 C CNN
-F 2 "" V 4205 2575 30  0001 C CNN
+F 2 "Resistors_SMD:R_0603" V 4205 2575 30  0001 C CNN
 F 3 "" H 4275 2575 30  0000 C CNN
 	1    4275 2575
@@
 F 0 "R38" V 4200 3200 40  0000 C CNN
 F 1 "10k" V 4282 3201 40  0000 C CNN
-F 2 "" V 4205 3200 30  0001 C CNN
+F 2 "Resistors_SMD:R_0603" V 4205 3200 30  0001 C CNN
 F 3 "" H 4275 3200 30  0000 C CNN
 	1    4275 3200
@@
 Connection ~ 4275 2900
 $Comp
-L 3V3 #PWR082
+L 3V3 #PWR083
 U 1 1 55A364F9
 P 4275 2250
-F 0 "#PWR082" H 4275 2350 40  0001 C CNN
+F 0 "#PWR083" H 4275 2350 40  0001 C CNN
 F 1 "3V3" H 4275 2375 40  0000 C CNN
 F 2 "" H 4275 2250 60  0000 C CNN
@@
 	4275 2325 4275 2250
 $Comp
-L GND #PWR083
+L GND #PWR084
 U 1 1 55A36665
 P 4275 3525
-F 0 "#PWR083" H 4275 3525 30  0001 C CNN
+F 0 "#PWR084" H 4275 3525 30  0001 C CNN
 F 1 "GND" H 4275 3455 30  0001 C CNN
 F 2 "" H 4275 3525 60  0000 C CNN
@@
 F 0 "R35" V 4200 1075 40  0000 C CNN
 F 1 "33k" V 4282 1076 40  0000 C CNN
-F 2 "" V 4205 1075 30  0001 C CNN
+F 2 "Resistors_SMD:R_0603" V 4205 1075 30  0001 C CNN
 F 3 "" H 4275 1075 30  0000 C CNN
 	1    4275 1075
@@
 F 0 "R36" V 4200 1700 40  0000 C CNN
 F 1 "10k" V 4282 1701 40  0000 C CNN
-F 2 "" V 4205 1700 30  0001 C CNN
+F 2 "Resistors_SMD:R_0603" V 4205 1700 30  0001 C CNN
 F 3 "" H 4275 1700 30  0000 C CNN
 	1    4275 1700
@@
 	4275 825  4275 750
 $Comp
-L GND #PWR084
+L GND #PWR085
 U 1 1 55A36FC3
 P 4275 2025
-F 0 "#PWR084" H 4275 2025 30  0001 C CNN
+F 0 "#PWR085" H 4275 2025 30  0001 C CNN
 F 1 "GND" H 4275 1955 30  0001 C CNN
 F 2 "" H 4275 2025 60  0000 C CNN
@@
 	4275 1400 5025 1400
 $Comp
-L PWR_FLAG #FLG085
+L PWR_FLAG #FLG086
 U 1 1 55A90C84
 P 7525 3625
-F 0 "#FLG085" H 7525 3720 30  0001 C CNN
+F 0 "#FLG086" H 7525 3720 30  0001 C CNN
 F 1 "PWR_FLAG" H 7525 3805 30  0000 C CNN
 F 2 "" H 7525 3625 60  0000 C CNN
@@
 Connection ~ 7525 3650
 $Comp
-L PWR_FLAG #FLG086
+L PWR_FLAG #FLG087
 U 1 1 55A8BD1F
 P 2250 3300
-F 0 "#FLG086" H 2250 3395 30  0001 C CNN
+F 0 "#FLG087" H 2250 3395 30  0001 C CNN
 F 1 "PWR_FLAG" H 2250 3480 30  0000 C CNN
 F 2 "" H 2250 3300 60  0000 C CNN
@@
 	2250 3300 2250 3450
 Connection ~ 2250 3450
+Wire Wire Line
+	6800 5925 6600 5925
+Wire Wire Line
+	6600 5925 6600 5750
+Connection ~ 6800 5925
 $EndSCHEMATC

Commit message: Saved last few changes before leaving
Parts:
- P12: footprint (none) -> Pin_Headers:Pin_Header_Straight_1x02
Changed lines of the file:
@@
 F 0 "P12" V 1275 3500 40  0000 C CNN
 F 1 "POWER" V 1375 3500 40  0000 C CNN
-F 2 "" H 1325 3500 60  0001 C CNN
+F 2 "Pin_Headers:Pin_Header_Straight_1x02" H 1325 3500 60  0001 C CNN
 F 3 "" H 1325 3500 60  0000 C CNN
 	1    1325 3500
