File: board/mainboard/Audio.sch (KiCad schematic (older format))
At the start: 15 parts

Commit message: First revision of mic and MAX9814, not finished
Parts:
- added 0.47uF, 0.68uF, 0.68uF?, 1uF, 2.2uF, 680nF: C, ~, symbol C
- added 2.2k, R? (x2): R, ~, symbol R
- added MIC?: CMA-4544PF-W, ~, symbol CMA-4544PF-W
- added U?: MAX9814, symbol MAX9814
Connections:
- wire segments 36 -> 67

Commit message: Finished draft 1 of Rev 2 layout
Parts:
- removed 0.68uF?: C, ~, symbol C
- added P15: MIC, symbol CONN_2
- C17: renamed from 0.47uF; value C -> 470nF
- C18: renamed from 0.68uF; value C -> 680nF
- C19: renamed from 680nF; value C -> 680nF
- C20: renamed from 2.2uF; value C -> 2.2uF
- C23: renamed from 1.0uF; value C -> 1.0uF
- C25: renamed from 1uF; value C -> 1uF
- R24: renamed from 2.2k; value R -> 2.2k
- R32, R33: renamed from R?; value R -> 150k
- gave numbers to parts that had none: 16
Connections:
- wire segments 67 -> 69

Commit message: fixed DRC errors on schematic
Changed lines of the file:
@@
 Sheet 8 8
 Title ""
-Date "1 mar 2015"
+Date "2 mar 2015"
 Rev ""
 Comp ""
@@
 	4100 5500 4000 5500
 Wire Wire Line
-	3550 6250 3350 6250
-Wire Wire Line
 	4100 6250 3950 6250
 Wire Wire Line
@@
 Wire Wire Line
 	6100 6600 6200 6600
+Wire Wire Line
+	3550 6250 3350 6250
+Connection ~ 3350 6250
 $EndSCHEMATC

Commit message: Rebuilt power section to support switching, new buck converter for 3V3 net.
Parts:
- P14, P15: symbol CONN_2 -> CONN_01X02
Connections:
- wire segments 69 -> 77
Changed lines of the file:
@@
 LIBS:valves
 LIBS:mainboard-cache
-EELAYER 27 0
+EELAYER 25 0
 EELAYER END
 $Descr A4 11693 8268
@@
 $EndComp
 $Comp
-L GND #PWR95
+L GND #PWR98
 U 1 1 54F15D3C
 P 5850 2950
-F 0 "#PWR95" H 5850 2950 30  0001 C CNN
+F 0 "#PWR98" H 5850 2950 30  0001 C CNN
 F 1 "GND" H 5850 2880 30  0001 C CNN
 F 2 "" H 5850 2950 60  0000 C CNN
@@
 $EndComp
 $Comp
-L 3V3 #PWR94
+L 3V3 #PWR97
 U 1 1 54F15D57
 P 5850 1150
-F 0 "#PWR94" H 5850 1250 40  0001 C CNN
+F 0 "#PWR97" H 5850 1250 40  0001 C CNN
 F 1 "3V3" H 5850 1275 40  0000 C CNN
 F 2 "" H 5850 1150 60  0000 C CNN
@@
 $EndComp
 $Comp
-L GND #PWR93
+L GND #PWR96
 U 1 1 54F15D90
 P 5250 1350
-F 0 "#PWR93" H 5250 1350 30  0001 C CNN
+F 0 "#PWR96" H 5250 1350 30  0001 C CNN
 F 1 "GND" H 5250 1280 30  0001 C CNN
 F 2 "" H 5250 1350 60  0000 C CNN
@@
 $EndComp
 $Comp
-L GND #PWR89
+L GND #PWR92
 U 1 1 54F15F26
 P 4500 2800
-F 0 "#PWR89" H 4500 2800 30  0001 C CNN
+F 0 "#PWR92" H 4500 2800 30  0001 C CNN
 F 1 "GND" H 4500 2730 30  0001 C CNN
 F 2 "" H 4500 2800 60  0000 C CNN
@@
 $EndComp
 $Comp
-L GND #PWR88
+L GND #PWR91
 U 1 1 54F15F53
 P 3950 2800
-F 0 "#PWR88" H 3950 2800 30  0001 C CNN
+F 0 "#PWR91" H 3950 2800 30  0001 C CNN
 F 1 "GND" H 3950 2730 30  0001 C CNN
 F 2 "" H 3950 2800 60  0000 C CNN
@@
 $EndComp
 $Comp
-L 3V3 #PWR87
+L 3V3 #PWR90
 U 1 1 54F15F81
 P 3950 1300
-F 0 "#PWR87" H 3950 1400 40  0001 C CNN
+F 0 "#PWR90" H 3950 1400 40  0001 C CNN
 F 1 "3V3" H 3950 1425 40  0000 C CNN
 F 2 "" H 3950 1300 60  0000 C CNN
@@
 $EndComp
 $Comp
-L CONN_2 P14
+L CONN_01X02 P14
 U 1 1 54F15FD1
 P 2700 2050
@@
 $EndComp
 $Comp
-L GND #PWR100
+L GND #PWR103
 U 1 1 54F16315
 P 7600 2400
-F 0 "#PWR100" H 7600 2400 30  0001 C CNN
+F 0 "#PWR103" H 7600 2400 30  0001 C CNN
 F 1 "GND" H 7600 2330 30  0001 C CNN
 F 2 "" H 7600 2400 60  0000 C CNN
@@
 $EndComp
 $Comp
-L 3V3 #PWR90
+L 3V3 #PWR93
 U 1 1 54F2495C
 P 5000 3950
-F 0 "#PWR90" H 5000 4050 40  0001 C CNN
+F 0 "#PWR93" H 5000 4050 40  0001 C CNN
 F 1 "3V3" H 5000 4075 40  0000 C CNN
 F 2 "" H 5000 3950 60  0000 C CNN
@@
 $EndComp
 $Comp
-L GND #PWR92
+L GND #PWR95
 U 1 1 54F249F7
 P 5200 4750
-F 0 "#PWR92" H 5200 4750 30  0001 C CNN
+F 0 "#PWR95" H 5200 4750 30  0001 C CNN
 F 1 "GND" H 5200 4680 30  0001 C CNN
 F 2 "" H 5200 4750 60  0000 C CNN
@@
 $EndComp
 $Comp
-L GND #PWR96
+L GND #PWR99
 U 1 1 54F24C7F
 P 6100 5350
-F 0 "#PWR96" H 6100 5350 30  0001 C CNN
+F 0 "#PWR99" H 6100 5350 30  0001 C CNN
 F 1 "GND" H 6100 5280 30  0001 C CNN
 F 2 "" H 6100 5350 60  0000 C CNN
@@
 $EndComp
 $Comp
-L GND #PWR86
+L GND #PWR89
 U 1 1 54F24D46
 P 3350 6400
-F 0 "#PWR86" H 3350 6400 30  0001 C CNN
+F 0 "#PWR89" H 3350 6400 30  0001 C CNN
 F 1 "GND" H 3350 6330 30  0001 C CNN
 F 2 "" H 3350 6400 60  0000 C CNN
@@
 	5050 1700 5050 750
 $Comp
-L GND #PWR84
+L GND #PWR87
 U 1 1 54F2512A
 P 2350 5800
-F 0 "#PWR84" H 2350 5800 30  0001 C CNN
+F 0 "#PWR87" H 2350 5800 30  0001 C CNN
 F 1 "GND" H 2350 5730 30  0001 C CNN
 F 2 "" H 2350 5800 60  0000 C CNN
@@
 	2350 5500 2350 5800
 $Comp
-L 3V3 #PWR97
+L 3V3 #PWR100
 U 1 1 54F2521B
 P 6100 5700
-F 0 "#PWR97" H 6100 5800 40  0001 C CNN
+F 0 "#PWR100" H 6100 5800 40  0001 C CNN
 F 1 "3V3" H 6100 5825 40  0000 C CNN
 F 2 "" H 6100 5700 60  0000 C CNN
@@
 	6100 5750 6100 5700
 $Comp
-L GND #PWR91
+L GND #PWR94
 U 1 1 54F252B5
 P 5000 6900
-F 0 "#PWR91" H 5000 6900 30  0001 C CNN
+F 0 "#PWR94" H 5000 6900 30  0001 C CNN
 F 1 "GND" H 5000 6830 30  0001 C CNN
 F 2 "" H 5000 6900 60  0000 C CNN
@@
 $EndComp
 $Comp
-L GND #PWR85
+L GND #PWR88
 U 1 1 54F2535D
 P 3350 5400
-F 0 "#PWR85" H 3350 5400 30  0001 C CNN
+F 0 "#PWR88" H 3350 5400 30  0001 C CNN
 F 1 "GND" H 3350 5330 30  0001 C CNN
 F 2 "" H 3350 5400 60  0000 C CNN
@@
 Connection ~ 6500 5500
 $Comp
-L GND #PWR99
+L GND #PWR102
 U 1 1 54F254FD
 P 6500 6300
-F 0 "#PWR99" H 6500 6300 30  0001 C CNN
+F 0 "#PWR102" H 6500 6300 30  0001 C CNN
 F 1 "GND" H 6500 6230 30  0001 C CNN
 F 2 "" H 6500 6300 60  0000 C CNN
@@
 	6500 6300 6500 6150
 $Comp
-L 3V3 #PWR98
+L 3V3 #PWR101
 U 1 1 54F25557
 P 6500 4700
-F 0 "#PWR98" H 6500 4800 40  0001 C CNN
+F 0 "#PWR101" H 6500 4800 40  0001 C CNN
 F 1 "3V3" H 6500 4825 40  0000 C CNN
 F 2 "" H 6500 4700 60  0000 C CNN
@@
 	6100 6000 6100 6600
 $Comp
-L CONN_2 P15
+L CONN_01X02 P15
 U 1 1 54F2A05E
 P 6550 6700
@@
 	3550 6250 3350 6250
 Connection ~ 3350 6250
+Wire Wire Line
+	2900 2000 3050 2000
+Wire Wire Line
+	3050 2000 3050 1950
+Wire Wire Line
+	3050 2150 3050 2100
+Wire Wire Line
+	3050 2100 2900 2100
+Wire Wire Line
+	6350 6650 6200 6650
+Wire Wire Line
+	6200 6650 6200 6600
+Wire Wire Line
+	6350 6750 6200 6750
+Wire Wire Line
+	6200 6750 6200 6800
 $EndSCHEMATC

Commit message: Completed rev 3.0 schematics.
1) Replaced MPU with STM Accelerometer
Parts:
- AUD1: footprint (none) -> footprints:LM4808
- C17, C18, C19, C20, C21, C22, C23, C24, C25, C26, C29, R24, R25, R26, R28, R29, R30, R31, R32, R33: footprint ~ -> (none)
- HP1: footprint ~ -> footprints:HeadphoneJack
- MIC1: footprint ~ -> footprints:CMA-4544
- P14, P15: footprint (none) -> Pin_Headers:Pin_Header_Straight_1x02
Changed lines of the file:
@@
 F 0 "AUD1" H 5850 2050 60  0000 C CNN
 F 1 "LM4808" H 5850 2200 60  0000 C CNN
-F 2 "" H 5850 2050 60  0000 C CNN
+F 2 "footprints:LM4808" H 5850 2050 60  0001 C CNN
 F 3 "" H 5850 2050 60  0000 C CNN
 	1    5850 2050
@@
 F 0 "C21" H 3950 850 40  0000 L CNN
 F 1 "2.2uF" H 3956 665 40  0000 L CNN
-F 2 "~" H 3988 600 30  0000 C CNN
+F 2 "" H 3988 600 30  0001 C CNN
 F 3 "~" H 3950 750 60  0000 C CNN
 	1    3950 750
@@
 F 0 "R28" V 4680 750 40  0000 C CNN
 F 1 "3.9k" V 4607 751 40  0000 C CNN
-F 2 "~" V 4530 750 30  0000 C CNN
+F 2 "" V 4530 750 30  0001 C CNN
 F 3 "~" H 4600 750 30  0000 C CNN
 	1    4600 750
@@
 F 0 "R30" V 5930 750 40  0000 C CNN
 F 1 "3.9k" V 5857 751 40  0000 C CNN
-F 2 "~" V 5780 750 30  0000 C CNN
+F 2 "" V 5780 750 30  0001 C CNN
 F 3 "~" H 5850 750 30  0000 C CNN
 	1    5850 750
@@
 F 0 "C26" H 7100 1950 40  0000 L CNN
 F 1 "100uF" H 7106 1765 40  0000 L CNN
-F 2 "~" H 7138 1700 30  0000 C CNN
+F 2 "" H 7138 1700 30  0001 C CNN
 F 3 "~" H 7100 1850 60  0000 C CNN
 	1    7100 1850
@@
 F 0 "R31" V 5930 3400 40  0000 C CNN
 F 1 "3.9k" V 5857 3401 40  0000 C CNN
-F 2 "~" V 5780 3400 30  0000 C CNN
+F 2 "" V 5780 3400 30  0001 C CNN
 F 3 "~" H 5850 3400 30  0000 C CNN
 	1    5850 3400
@@
 F 0 "R29" V 4680 3400 40  0000 C CNN
 F 1 "3.9k" V 4607 3401 40  0000 C CNN
-F 2 "~" V 4530 3400 30  0000 C CNN
+F 2 "" V 4530 3400 30  0001 C CNN
 F 3 "~" H 4600 3400 30  0000 C CNN
 	1    4600 3400
@@
 $EndComp
 $Comp
-L GND #PWR98
+L GND #PWR085
 U 1 1 54F15D3C
 P 5850 2950
-F 0 "#PWR98" H 5850 2950 30  0001 C CNN
+F 0 "#PWR085" H 5850 2950 30  0001 C CNN
 F 1 "GND" H 5850 2880 30  0001 C CNN
 F 2 "" H 5850 2950 60  0000 C CNN
@@
 $EndComp
 $Comp
-L 3V3 #PWR97
+L 3V3 #PWR086
 U 1 1 54F15D57
 P 5850 1150
-F 0 "#PWR97" H 5850 1250 40  0001 C CNN
+F 0 "#PWR086" H 5850 1250 40  0001 C CNN
 F 1 "3V3" H 5850 1275 40  0000 C CNN
 F 2 "" H 5850 1150 60  0000 C CNN
@@
 F 0 "C24" H 5550 1300 40  0000 L CNN
 F 1 "0.1uF" H 5556 1115 40  0000 L CNN
-F 2 "~" H 5588 1050 30  0000 C CNN
+F 2 "" H 5588 1050 30  0001 C CNN
 F 3 "~" H 5550 1200 60  0000 C CNN
 	1    5550 1200
@@
 $EndComp
 $Comp
-L GND #PWR96
+L GND #PWR087
 U 1 1 54F15D90
 P 5250 1350
-F 0 "#PWR96" H 5250 1350 30  0001 C CNN
+F 0 "#PWR087" H 5250 1350 30  0001 C CNN
 F 1 "GND" H 5250 1280 30  0001 C CNN
 F 2 "" H 5250 1350 60  0000 C CNN
@@
 F 0 "C29" H 7100 2350 40  0000 L CNN
 F 1 "100uF" H 7106 2165 40  0000 L CNN
-F 2 "~" H 7138 2100 30  0000 C CNN
+F 2 "" H 7138 2100 30  0001 C CNN
 F 3 "~" H 7100 2250 60  0000 C CNN
 	1    7100 2250
@@
 F 0 "C22" H 3950 3500 40  0000 L CNN
 F 1 "2.2uF" H 3956 3315 40  0000 L CNN
-F 2 "~" H 3988 3250 30  0000 C CNN
+F 2 "" H 3988 3250 30  0001 C CNN
 F 3 "~" H 3950 3400 60  0000 C CNN
 	1    3950 3400
@@
 F 0 "C23" H 4500 2500 40  0000 L CNN
 F 1 "1.0uF" H 4506 2315 40  0000 L CNN
-F 2 "~" H 4538 2250 30  0000 C CNN
+F 2 "" H 4538 2250 30  0001 C CNN
 F 3 "~" H 4500 2400 60  0000 C CNN
 	1    4500 2400
@@
 F 0 "R26" V 4030 2450 40  0000 C CNN
 F 1 "100k" V 3957 2451 40  0000 C CNN
-F 2 "~" V 3880 2450 30  0000 C CNN
+F 2 "" V 3880 2450 30  0001 C CNN
 F 3 "~" H 3950 2450 30  0000 C CNN
 	1    3950 2450
@@
 F 0 "R25" V 4030 1650 40  0000 C CNN
 F 1 "100k" V 3957 1651 40  0000 C CNN
-F 2 "~" V 3880 1650 30  0000 C CNN
+F 2 "" V 3880 1650 30  0001 C CNN
 F 3 "~" H 3950 1650 30  0000 C CNN
 	1    3950 1650
@@
 $EndComp
 $Comp
-L GND #PWR92
+L GND #PWR088
 U 1 1 54F15F26
 P 4500 2800
-F 0 "#PWR92" H 4500 2800 30  0001 C CNN
+F 0 "#PWR088" H 4500 2800 30  0001 C CNN
 F 1 "GND" H 4500 2730 30  0001 C CNN
 F 2 "" H 4500 2800 60  0000 C CNN
@@
 $EndComp
 $Comp
-L GND #PWR91
+L GND #PWR089
 U 1 1 54F15F53
 P 3950 2800
-F 0 "#PWR91" H 3950 2800 30  0001 C CNN
+F 0 "#PWR089" H 3950 2800 30  0001 C CNN
 F 1 "GND" H 3950 2730 30  0001 C CNN
 F 2 "" H 3950 2800 60  0000 C CNN
@@
 $EndComp
 $Comp
-L 3V3 #PWR90
+L 3V3 #PWR090
 U 1 1 54F15F81
 P 3950 1300
-F 0 "#PWR90" H 3950 1400 40  0001 C CNN
+F 0 "#PWR090" H 3950 1400 40  0001 C CNN
 F 1 "3V3" H 3950 1425 40  0000 C CNN
 F 2 "" H 3950 1300 60  0000 C CNN
@@
 F 0 "P14" V 2650 2050 40  0000 C CNN
 F 1 "AUDIO" V 2750 2050 40  0000 C CNN
-F 2 "" H 2700 2050 60  0000 C CNN
+F 2 "Pin_Headers:Pin_Header_Straight_1x02" H 2700 2050 60  0001 C CNN
 F 3 "" H 2700 2050 60  0000 C CNN
 	1    2700 2050
@@
 F 0 "HP1" H 8100 2300 60  0000 C CNN
 F 1 "HP_JACK" H 8100 1900 60  0000 C CNN
-F 2 "~" H 8100 2300 60  0000 C CNN
+F 2 "footprints:HeadphoneJack" H 8100 2300 60  0000 C CNN
 F 3 "~" H 8100 2300 60  0000 C CNN
 	1    8100 2100
@@
 $EndComp
 $Comp
-L GND #PWR103
+L GND #PWR091
 U 1 1 54F16315
 P 7600 2400
-F 0 "#PWR103" H 7600 2400 30  0001 C CNN
+F 0 "#PWR091" H 7600 2400 30  0001 C CNN
 F 1 "GND" H 7600 2330 30  0001 C CNN
 F 2 "" H 7600 2400 60  0000 C CNN
@@
 F 0 "U3" H 5000 5750 60  0000 C CNN
 F 1 "MAX9814" H 5000 5900 60  0000 C CNN
-F 2 "" H 5000 5750 60  0000 C CNN
+F 2 "" H 5000 5750 60  0001 C CNN
 F 3 "" H 5000 5750 60  0000 C CNN
 	1    5000 5750
@@
 F 0 "C25" H 5200 4450 40  0000 L CNN
 F 1 "1uF" H 5206 4265 40  0000 L CNN
-F 2 "~" H 5238 4200 30  0000 C CNN
+F 2 "" H 5238 4200 30  0001 C CNN
 F 3 "~" H 5200 4350 60  0000 C CNN
 	1    5200 4350
@@
 $EndComp
 $Comp
-L 3V3 #PWR93
+L 3V3 #PWR092
 U 1 1 54F2495C
 P 5000 3950
-F 0 "#PWR93" H 5000 4050 40  0001 C CNN
+F 0 "#PWR092" H 5000 4050 40  0001 C CNN
 F 1 "3V3" H 5000 4075 40  0000 C CNN
 F 2 "" H 5000 3950 60  0000 C CNN
@@
 $EndComp
 $Comp
-L GND #PWR95
+L GND #PWR093
 U 1 1 54F249F7
 P 5200 4750
-F 0 "#PWR95" H 5200 4750 30  0001 C CNN
+F 0 "#PWR093" H 5200 4750 30  0001 C CNN
 F 1 "GND" H 5200 4680 30  0001 C CNN
 F 2 "" H 5200 4750 60  0000 C CNN
@@
 $EndComp
 $Comp
-L GND #PWR99
+L GND #PWR094
 U 1 1 54F24C7F
 P 6100 5350
-F 0 "#PWR99" H 6100 5350 30  0001 C CNN
+F 0 "#PWR094" H 6100 5350 30  0001 C CNN
 F 1 "GND" H 6100 5280 30  0001 C CNN
 F 2 "" H 6100 5350 60  0000 C CNN
@@
 F 0 "C19" H 3750 6100 40  0000 L CNN
 F 1 "680nF" H 3756 5915 40  0000 L CNN
-F 2 "~" H 3788 5850 30  0000 C CNN
+F 2 "" H 3788 5850 30  0001 C CNN
 F 3 "~" H 3750 6000 60  0000 C CNN
 	1    3750 6000
@@
 $EndComp
 $Comp
-L GND #PWR89
+L GND #PWR095
 U 1 1 54F24D46
 P 3350 6400
-F 0 "#PWR89" H 3350 6400 30  0001 C CNN
+F 0 "#PWR095" H 3350 6400 30  0001 C CNN
 F 1 "GND" H 3350 6330 30  0001 C CNN
 F 2 "" H 3350 6400 60  0000 C CNN
@@
 F 0 "C20" H 3750 6350 40  0000 L CNN
 F 1 "2.2uF" H 3756 6165 40  0000 L CNN
-F 2 "~" H 3788 6100 30  0000 C CNN
+F 2 "" H 3788 6100 30  0001 C CNN
 F 3 "~" H 3750 6250 60  0000 C CNN
 	1    3750 6250
@@
 F 0 "R24" V 3830 5500 40  0000 C CNN
 F 1 "2.2k" V 3757 5501 40  0000 C CNN
-F 2 "~" V 3680 5500 30  0000 C CNN
+F 2 "" V 3680 5500 30  0001 C CNN
 F 3 "~" H 3750 5500 30  0000 C CNN
 	1    3750 5500
@@
 F 0 "C18" H 3750 5850 40  0000 L CNN
 F 1 "680nF" H 3756 5665 40  0000 L CNN
-F 2 "~" H 3788 5600 30  0000 C CNN
+F 2 "" H 3788 5600 30  0001 C CNN
 F 3 "~" H 3750 5750 60  0000 C CNN
 	1    3750 5750
@@
 F 0 "MIC1" H 2750 5200 60  0000 C CNN
 F 1 "CMA-4544PF-W" H 2700 5700 60  0001 C CNN
-F 2 "~" H 2700 5700 60  0000 C CNN
+F 2 "footprints:CMA-4544" H 2700 5700 60  0000 C CNN
 F 3 "~" H 2700 5700 60  0000 C CNN
 	1    2750 5450
@@
 	5050 1700 5050 750
 $Comp
-L GND #PWR87
+L GND #PWR096
 U 1 1 54F2512A
 P 2350 5800
-F 0 "#PWR87" H 2350 5800 30  0001 C CNN
+F 0 "#PWR096" H 2350 5800 30  0001 C CNN
 F 1 "GND" H 2350 5730 30  0001 C CNN
 F 2 "" H 2350 5800 60  0000 C CNN
@@
 	2350 5500 2350 5800
 $Comp
-L 3V3 #PWR100
+L 3V3 #PWR097
 U 1 1 54F2521B
 P 6100 5700
-F 0 "#PWR100" H 6100 5800 40  0001 C CNN
+F 0 "#PWR097" H 6100 5800 40  0001 C CNN
 F 1 "3V3" H 6100 5825 40  0000 C CNN
 F 2 "" H 6100 5700 60  0000 C CNN
@@
 	6100 5750 6100 5700
 $Comp
-L GND #PWR94
+L GND #PWR098
 U 1 1 54F252B5
 P 5000 6900
-F 0 "#PWR94" H 5000 6900 30  0001 C CNN
+F 0 "#PWR098" H 5000 6900 30  0001 C CNN
 F 1 "GND" H 5000 6830 30  0001 C CNN
 F 2 "" H 5000 6900 60  0000 C CNN
@@
 F 0 "C17" H 3750 5350 40  0000 L CNN
 F 1 "470nF" H 3756 5165 40  0000 L CNN
-F 2 "~" H 3788 5100 30  0000 C CNN
+F 2 "" H 3788 5100 30  0001 C CNN
 F 3 "~" H 3750 5250 60  0000 C CNN
 	1    3750 5250
@@
 $EndComp
 $Comp
-L GND #PWR88
+L GND #PWR099
 U 1 1 54F2535D
 P 3350 5400
-F 0 "#PWR88" H 3350 5400 30  0001 C CNN
+F 0 "#PWR099" H 3350 5400 30  0001 C CNN
 F 1 "GND" H 3350 5330 30  0001 C CNN
 F 2 "" H 3350 5400 60  0000 C CNN
@@
 F 0 "R32" V 6580 5100 40  0000 C CNN
 F 1 "150k" V 6507 5101 40  0000 C CNN
-F 2 "~" V 6430 5100 30  0000 C CNN
+F 2 "" V 6430 5100 30  0001 C CNN
 F 3 "~" H 6500 5100 30  0000 C CNN
 	1    6500 5100
@@
 F 0 "R33" V 6580 5900 40  0000 C CNN
 F 1 "150k" V 6507 5901 40  0000 C CNN
-F 2 "~" V 6430 5900 30  0000 C CNN
+F 2 "" V 6430 5900 30  0001 C CNN
 F 3 "~" H 6500 5900 30  0000 C CNN
 	1    6500 5900
@@
 Connection ~ 6500 5500
 $Comp
-L GND #PWR102
+L GND #PWR0100
 U 1 1 54F254FD
 P 6500 6300
-F 0 "#PWR102" H 6500 6300 30  0001 C CNN
+F 0 "#PWR0100" H 6500 6300 30  0001 C CNN
 F 1 "GND" H 6500 6230 30  0001 C CNN
 F 2 "" H 6500 6300 60  0000 C CNN
@@
 	6500 6300 6500 6150
 $Comp
-L 3V3 #PWR101
+L 3V3 #PWR0101
 U 1 1 54F25557
 P 6500 4700
-F 0 "#PWR101" H 6500 4800 40  0001 C CNN
+F 0 "#PWR0101" H 6500 4800 40  0001 C CNN
 F 1 "3V3" H 6500 4825 40  0000 C CNN
 F 2 "" H 6500 4700 60  0000 C CNN
@@
 F 0 "P15" V 6500 6700 40  0000 C CNN
 F 1 "MIC" V 6600 6700 40  0000 C CNN
-F 2 "" H 6550 6700 60  0000 C CNN
+F 2 "Pin_Headers:Pin_Header_Straight_1x02" H 6550 6700 60  0001 C CNN
 F 3 "" H 6550 6700 60  0000 C CNN
 	1    6550 6700
