File: board/mainboard/Audio.sch (KiCad schematic (older format))
At the start: 26 parts, among them P14 AUDIO, P15 MIC, U3 MAX9814

Commit message: Added most of the footprints needed to make this work
Parts:
- C17, C18, C19, C20, C21, C22, C23, C24, C25: footprint (none) -> Capacitors_SMD:c_0603
- C26, C29: footprint (none) -> footprints:CAP_SMD_100uF__; symbol C -> CPsmall
- R24, R25, R26, R28, R29, R30, R31, R32, R33: footprint (none) -> Resistors_SMD:R_0603
- U3: footprint (none) -> footprints:MAX9814
Connections:
- wire segments 77 -> 79
Changed lines of the file:
@@
 F 0 "C21" H 3950 850 40  0000 L CNN
 F 1 "2.2uF" H 3956 665 40  0000 L CNN
-F 2 "" H 3988 600 30  0001 C CNN
+F 2 "Capacitors_SMD:c_0603" H 3988 600 30  0001 C CNN
 F 3 "~" H 3950 750 60  0000 C CNN
 	1    3950 750
@@
 F 0 "R28" V 4680 750 40  0000 C CNN
 F 1 "3.9k" V 4607 751 40  0000 C CNN
-F 2 "" V 4530 750 30  0001 C CNN
+F 2 "Resistors_SMD:R_0603" V 4530 750 30  0001 C CNN
 F 3 "~" H 4600 750 30  0000 C CNN
 	1    4600 750
@@
 F 0 "R30" V 5930 750 40  0000 C CNN
 F 1 "3.9k" V 5857 751 40  0000 C CNN
-F 2 "" V 5780 750 30  0001 C CNN
+F 2 "Resistors_SMD:R_0603" V 5780 750 30  0001 C CNN
 F 3 "~" H 5850 750 30  0000 C CNN
 	1    5850 750
@@
 $EndComp
 $Comp
-L C C26
+L CPsmall C26
 U 1 1 54F15BD3
 P 7100 1850
 F 0 "C26" H 7100 1950 40  0000 L CNN
 F 1 "100uF" H 7106 1765 40  0000 L CNN
-F 2 "" H 7138 1700 30  0001 C CNN
+F 2 "footprints:CAP_SMD_100uF__" H 7138 1700 30  0001 C CNN
 F 3 "~" H 7100 1850 60  0000 C CNN
 	1    7100 1850
@@
 F 0 "R31" V 5930 3400 40  0000 C CNN
 F 1 "3.9k" V 5857 3401 40  0000 C CNN
-F 2 "" V 5780 3400 30  0001 C CNN
+F 2 "Resistors_SMD:R_0603" V 5780 3400 30  0001 C CNN
 F 3 "~" H 5850 3400 30  0000 C CNN
 	1    5850 3400
@@
 F 0 "R29" V 4680 3400 40  0000 C CNN
 F 1 "3.9k" V 4607 3401 40  0000 C CNN
-F 2 "" V 4530 3400 30  0001 C CNN
+F 2 "Resistors_SMD:R_0603" V 4530 3400 30  0001 C CNN
 F 3 "~" H 4600 3400 30  0000 C CNN
 	1    4600 3400
@@
 $EndComp
 $Comp
-L GND #PWR087
+L GND #PWR088
 U 1 1 54F15D3C
 P 5850 2950
-F 0 "#PWR087" H 5850 2950 30  0001 C CNN
+F 0 "#PWR088" H 5850 2950 30  0001 C CNN
 F 1 "GND" H 5850 2880 30  0001 C CNN
 F 2 "" H 5850 2950 60  0000 C CNN
@@
 $EndComp
 $Comp
-L 3V3 #PWR088
+L 3V3 #PWR089
 U 1 1 54F15D57
 P 5850 1150
-F 0 "#PWR088" H 5850 1250 40  0001 C CNN
+F 0 "#PWR089" H 5850 1250 40  0001 C CNN
 F 1 "3V3" H 5850 1275 40  0000 C CNN
 F 2 "" H 5850 1150 60  0000 C CNN
@@
 F 0 "C24" H 5550 1300 40  0000 L CNN
 F 1 "0.1uF" H 5556 1115 40  0000 L CNN
-F 2 "" H 5588 1050 30  0001 C CNN
+F 2 "Capacitors_SMD:c_0603" H 5588 1050 30  0001 C CNN
 F 3 "~" H 5550 1200 60  0000 C CNN
 	1    5550 1200
@@
 $EndComp
 $Comp
-L GND #PWR089
+L GND #PWR090
 U 1 1 54F15D90
 P 5250 1350
-F 0 "#PWR089" H 5250 1350 30  0001 C CNN
+F 0 "#PWR090" H 5250 1350 30  0001 C CNN
 F 1 "GND" H 5250 1280 30  0001 C CNN
 F 2 "" H 5250 1350 60  0000 C CNN
@@
 $EndComp
 $Comp
-L C C29
+L CPsmall C29
 U 1 1 54F15DDC
 P 7100 2250
 F 0 "C29" H 7100 2350 40  0000 L CNN
 F 1 "100uF" H 7106 2165 40  0000 L CNN
-F 2 "" H 7138 2100 30  0001 C CNN
+F 2 "footprints:CAP_SMD_100uF__" H 7138 2100 30  0001 C CNN
 F 3 "~" H 7100 2250 60  0000 C CNN
 	1    7100 2250
@@
 F 0 "C22" H 3950 3500 40  0000 L CNN
 F 1 "2.2uF" H 3956 3315 40  0000 L CNN
-F 2 "" H 3988 3250 30  0001 C CNN
+F 2 "Capacitors_SMD:c_0603" H 3988 3250 30  0001 C CNN
 F 3 "~" H 3950 3400 60  0000 C CNN
 	1    3950 3400
@@
 F 0 "C23" H 4500 2500 40  0000 L CNN
 F 1 "1.0uF" H 4506 2315 40  0000 L CNN
-F 2 "" H 4538 2250 30  0001 C CNN
+F 2 "Capacitors_SMD:c_0603" H 4538 2250 30  0001 C CNN
 F 3 "~" H 4500 2400 60  0000 C CNN
 	1    4500 2400
@@
 F 0 "R26" V 4030 2450 40  0000 C CNN
 F 1 "100k" V 3957 2451 40  0000 C CNN
-F 2 "" V 3880 2450 30  0001 C CNN
+F 2 "Resistors_SMD:R_0603" V 3880 2450 30  0001 C CNN
 F 3 "~" H 3950 2450 30  0000 C CNN
 	1    3950 2450
@@
 F 0 "R25" V 4030 1650 40  0000 C CNN
 F 1 "100k" V 3957 1651 40  0000 C CNN
-F 2 "" V 3880 1650 30  0001 C CNN
+F 2 "Resistors_SMD:R_0603" V 3880 1650 30  0001 C CNN
 F 3 "~" H 3950 1650 30  0000 C CNN
 	1    3950 1650
@@
 $EndComp
 $Comp
-L GND #PWR090
+L GND #PWR091
 U 1 1 54F15F26
 P 4500 2800
-F 0 "#PWR090" H 4500 2800 30  0001 C CNN
+F 0 "#PWR091" H 4500 2800 30  0001 C CNN
 F 1 "GND" H 4500 2730 30  0001 C CNN
 F 2 "" H 4500 2800 60  0000 C CNN
@@
 $EndComp
 $Comp
-L GND #PWR091
+L GND #PWR092
 U 1 1 54F15F53
 P 3950 2800
-F 0 "#PWR091" H 3950 2800 30  0001 C CNN
+F 0 "#PWR092" H 3950 2800 30  0001 C CNN
 F 1 "GND" H 3950 2730 30  0001 C CNN
 F 2 "" H 3950 2800 60  0000 C CNN
@@
 $EndComp
 $Comp
-L 3V3 #PWR092
+L 3V3 #PWR093
 U 1 1 54F15F81
 P 3950 1300
-F 0 "#PWR092" H 3950 1400 40  0001 C CNN
+F 0 "#PWR093" H 3950 1400 40  0001 C CNN
 F 1 "3V3" H 3950 1425 40  0000 C CNN
 F 2 "" H 3950 1300 60  0000 C CNN
@@
 $EndComp
 $Comp
-L GND #PWR093
+L GND #PWR094
 U 1 1 54F16315
 P 7600 2400
-F 0 "#PWR093" H 7600 2400 30  0001 C CNN
+F 0 "#PWR094" H 7600 2400 30  0001 C CNN
 F 1 "GND" H 7600 2330 30  0001 C CNN
 F 2 "" H 7600 2400 60  0000 C CNN
@@
 F 0 "U3" H 5000 5750 60  0000 C CNN
 F 1 "MAX9814" H 5000 5900 60  0000 C CNN
-F 2 "" H 5000 5750 60  0001 C CNN
+F 2 "footprints:MAX9814" H 5000 5750 60  0001 C CNN
 F 3 "" H 5000 5750 60  0000 C CNN
 	1    5000 5750
@@
 F 0 "C25" H 5200 4450 40  0000 L CNN
 F 1 "1uF" H 5206 4265 40  0000 L CNN
-F 2 "" H 5238 4200 30  0001 C CNN
+F 2 "Capacitors_SMD:c_0603" H 5238 4200 30  0001 C CNN
 F 3 "~" H 5200 4350 60  0000 C CNN
 	1    5200 4350
@@
 $EndComp
 $Comp
-L 3V3 #PWR094
+L 3V3 #PWR095
 U 1 1 54F2495C
 P 5000 3950
-F 0 "#PWR094" H 5000 4050 40  0001 C CNN
+F 0 "#PWR095" H 5000 4050 40  0001 C CNN
 F 1 "3V3" H 5000 4075 40  0000 C CNN
 F 2 "" H 5000 3950 60  0000 C CNN
@@
 $EndComp
 $Comp
-L GND #PWR095
+L GND #PWR096
 U 1 1 54F249F7
 P 5200 4750
-F 0 "#PWR095" H 5200 4750 30  0001 C CNN
+F 0 "#PWR096" H 5200 4750 30  0001 C CNN
 F 1 "GND" H 5200 4680 30  0001 C CNN
 F 2 "" H 5200 4750 60  0000 C CNN
@@
 $EndComp
 $Comp
-L GND #PWR096
+L GND #PWR097
 U 1 1 54F24C7F
 P 6100 5350
-F 0 "#PWR096" H 6100 5350 30  0001 C CNN
+F 0 "#PWR097" H 6100 5350 30  0001 C CNN
 F 1 "GND" H 6100 5280 30  0001 C CNN
 F 2 "" H 6100 5350 60  0000 C CNN
@@
 F 0 "C19" H 3750 6100 40  0000 L CNN
 F 1 "680nF" H 3756 5915 40  0000 L CNN
-F 2 "" H 3788 5850 30  0001 C CNN
+F 2 "Capacitors_SMD:c_0603" H 3788 5850 30  0001 C CNN
 F 3 "~" H 3750 6000 60  0000 C CNN
 	1    3750 6000
@@
 $EndComp
 $Comp
-L GND #PWR097
+L GND #PWR098
 U 1 1 54F24D46
 P 3350 6400
-F 0 "#PWR097" H 3350 6400 30  0001 C CNN
+F 0 "#PWR098" H 3350 6400 30  0001 C CNN
 F 1 "GND" H 3350 6330 30  0001 C CNN
 F 2 "" H 3350 6400 60  0000 C CNN
@@
 F 0 "C20" H 3750 6350 40  0000 L CNN
 F 1 "2.2uF" H 3756 6165 40  0000 L CNN
-F 2 "" H 3788 6100 30  0001 C CNN
+F 2 "Capacitors_SMD:c_0603" H 3788 6100 30  0001 C CNN
 F 3 "~" H 3750 6250 60  0000 C CNN
 	1    3750 6250
@@
 F 0 "R24" V 3830 5500 40  0000 C CNN
 F 1 "2.2k" V 3757 5501 40  0000 C CNN
-F 2 "" V 3680 5500 30  0001 C CNN
+F 2 "Resistors_SMD:R_0603" V 3680 5500 30  0001 C CNN
 F 3 "~" H 3750 5500 30  0000 C CNN
 	1    3750 5500
@@
 F 0 "C18" H 3750 5850 40  0000 L CNN
 F 1 "680nF" H 3756 5665 40  0000 L CNN
-F 2 "" H 3788 5600 30  0001 C CNN
+F 2 "Capacitors_SMD:c_0603" H 3788 5600 30  0001 C CNN
 F 3 "~" H 3750 5750 60  0000 C CNN
 	1    3750 5750
@@
 Connection ~ 6800 2250
 Wire Wire Line
-	6700 2250 6900 2250
+	6700 2250 7000 2250
 Wire Wire Line
 	6800 3400 6100 3400
@@
 Connection ~ 6800 1850
 Wire Wire Line
-	6700 1850 6900 1850
+	6700 1850 7000 1850
 Wire Wire Line
 	6800 750  6800 1850
@@
 	5050 1700 5050 750
 $Comp
-L GND #PWR098
+L GND #PWR099
 U 1 1 54F2512A
 P 2350 5800
-F 0 "#PWR098" H 2350 5800 30  0001 C CNN
+F 0 "#PWR099" H 2350 5800 30  0001 C CNN
 F 1 "GND" H 2350 5730 30  0001 C CNN
 F 2 "" H 2350 5800 60  0000 C CNN
@@
 	2350 5500 2350 5800
 $Comp
-L 3V3 #PWR099
+L 3V3 #PWR0100
 U 1 1 54F2521B
 P 6100 5700
-F 0 "#PWR099" H 6100 5800 40  0001 C CNN
+F 0 "#PWR0100" H 6100 5800 40  0001 C CNN
 F 1 "3V3" H 6100 5825 40  0000 C CNN
 F 2 "" H 6100 5700 60  0000 C CNN
@@
 	6100 5750 6100 5700
 $Comp
-L GND #PWR0100
+L GND #PWR0101
 U 1 1 54F252B5
 P 5000 6900
-F 0 "#PWR0100" H 5000 6900 30  0001 C CNN
+F 0 "#PWR0101" H 5000 6900 30  0001 C CNN
 F 1 "GND" H 5000 6830 30  0001 C CNN
 F 2 "" H 5000 6900 60  0000 C CNN
@@
 F 0 "C17" H 3750 5350 40  0000 L CNN
 F 1 "470nF" H 3756 5165 40  0000 L CNN
-F 2 "" H 3788 5100 30  0001 C CNN
+F 2 "Capacitors_SMD:c_0603" H 3788 5100 30  0001 C CNN
 F 3 "~" H 3750 5250 60  0000 C CNN
 	1    3750 5250
@@
 $EndComp
 $Comp
-L GND #PWR0101
+L GND #PWR0102
 U 1 1 54F2535D
 P 3350 5400
-F 0 "#PWR0101" H 3350 5400 30  0001 C CNN
+F 0 "#PWR0102" H 3350 5400 30  0001 C CNN
 F 1 "GND" H 3350 5330 30  0001 C CNN
 F 2 "" H 3350 5400 60  0000 C CNN
@@
 F 0 "R32" V 6580 5100 40  0000 C CNN
 F 1 "150k" V 6507 5101 40  0000 C CNN
-F 2 "" V 6430 5100 30  0001 C CNN
+F 2 "Resistors_SMD:R_0603" V 6430 5100 30  0001 C CNN
 F 3 "~" H 6500 5100 30  0000 C CNN
 	1    6500 5100
@@
 F 0 "R33" V 6580 5900 40  0000 C CNN
 F 1 "150k" V 6507 5901 40  0000 C CNN
-F 2 "" V 6430 5900 30  0001 C CNN
+F 2 "Resistors_SMD:R_0603" V 6430 5900 30  0001 C CNN
 F 3 "~" H 6500 5900 30  0000 C CNN
 	1    6500 5900
@@
 Connection ~ 6500 5500
 $Comp
-L GND #PWR0102
+L GND #PWR0103
 U 1 1 54F254FD
 P 6500 6300
-F 0 "#PWR0102" H 6500 6300 30  0001 C CNN
+F 0 "#PWR0103" H 6500 6300 30  0001 C CNN
 F 1 "GND" H 6500 6230 30  0001 C CNN
 F 2 "" H 6500 6300 60  0000 C CNN
@@
 	6500 6300 6500 6150
 $Comp
-L 3V3 #PWR0103
+L 3V3 #PWR0104
 U 1 1 54F25557
 P 6500 4700
-F 0 "#PWR0103" H 6500 4800 40  0001 C CNN
+F 0 "#PWR0104" H 6500 4800 40  0001 C CNN
 F 1 "3V3" H 6500 4825 40  0000 C CNN
 F 2 "" H 6500 4700 60  0000 C CNN
@@
 Wire Wire Line
 	6200 6750 6200 6800
+Wire Wire Line
+	7300 2250 7200 2250
+Wire Wire Line
+	7300 1850 7200 1850
 $EndSCHEMATC
