File: board/mainboard/Analog.sch (KiCad schematic (older format))
At the start: 12 parts, among them P6 CONN_5, P7 ANALOG

Commit message: Changed analog header to expose 3 analog inputs (freed up from removing potentiometer)
Parts:
- P7: symbol CONN_01X02 -> CONN_01X03
Connections:
- net labels added: AIN3
- wire segments 45 -> 39
Changed lines of the file:
@@
 Comment4 ""
 $EndDescr
-$Comp
-L CONN_01X02 P7
-U 1 1 55A47551
-P 3100 3775
-F 0 "P7" V 3050 3775 40  0000 C CNN
-F 1 "ANALOG" V 3150 3775 40  0000 C CNN
-F 2 "" H 3100 3775 60  0000 C CNN
-F 3 "" H 3100 3775 60  0000 C CNN
-	1    3100 3775
-	-1   0    0    1
-$EndComp
 Text GLabel 3650 3875 2    60   Input ~ 0
 AIN1
-Text GLabel 3650 3675 2    60   Input ~ 0
+Text GLabel 3650 3750 2    60   Input ~ 0
 AIN2
 $Comp
@@
 LINE_SENSOR_L
 Wire Wire Line
-	3300 3875 3650 3875
-Wire Wire Line
-	3300 3675 3650 3675
-Wire Wire Line
 	3150 2875 3550 2875
 Wire Wire Line
@@
 Wire Wire Line
 	3650 2875 3800 2875
-Wire Wire Line
-	3300 3675 3300 3725
-Wire Wire Line
-	3300 3875 3300 3825
 $Comp
 L CAP_TOUCH CAP1
@@
 $EndComp
 Wire Wire Line
-	6625 2375 6725 2375
-Wire Wire Line
-	6725 2375 6925 2375
-Wire Wire Line
-	6925 2375 9550 2375
+	6625 2375 9550 2375
 $Comp
 L C C11
@@
 	6725 2375 6725 2550
 Wire Wire Line
-	6725 3100 6825 3100
-Wire Wire Line
-	6825 3100 6925 3100
+	6725 3100 6925 3100
 Wire Wire Line
 	6725 3100 6725 2950
@@
 	8050 2625 8050 2775
 Wire Wire Line
-	8050 3325 8150 3325
-Wire Wire Line
-	8150 3325 8250 3325
+	8050 3325 8250 3325
 Wire Wire Line
 	8050 3325 8050 3175
@@
 	9475 3475 9475 3450
 Wire Wire Line
-	9275 3475 9375 3475
-Wire Wire Line
-	9375 3475 9475 3475
+	9275 3475 9475 3475
 Wire Wire Line
 	9275 3475 9275 3425
@@
 Connection ~ 9375 3475
 Wire Wire Line
-	7975 2625 8050 2625
-Wire Wire Line
-	8050 2625 8250 2625
-Wire Wire Line
-	8250 2625 9550 2625
+	7975 2625 9550 2625
 Wire Wire Line
 	8250 2625 8250 2700
@@
 LINE_SENSOR_L
 Wire Wire Line
-	9225 2850 9275 2850
-Wire Wire Line
-	9275 2850 9475 2850
-Wire Wire Line
-	9475 2850 9550 2850
+	9225 2850 9550 2850
 Connection ~ 9275 2850
 Wire Wire Line
@@
 	6825 3100 6825 3175
 Connection ~ 6825 3100
+Text GLabel 3650 3625 2    60   Input ~ 0
+AIN3
+$Comp
+L CONN_01X03 P7
+U 1 1 55A47551
+P 3100 3750
+F 0 "P7" V 3050 3750 40  0000 C CNN
+F 1 "ANALOG" V 3150 3750 40  0000 C CNN
+F 2 "" H 3100 3750 60  0000 C CNN
+F 3 "" H 3100 3750 60  0000 C CNN
+	1    3100 3750
+	-1   0    0    1
+$EndComp
+Wire Wire Line
+	3650 3750 3300 3750
+Wire Wire Line
+	3300 3650 3500 3650
+Wire Wire Line
+	3500 3650 3500 3625
+Wire Wire Line
+	3500 3625 3650 3625
+Wire Wire Line
+	3650 3875 3500 3875
+Wire Wire Line
+	3500 3875 3500 3850
+Wire Wire Line
+	3500 3850 3300 3850
 $EndSCHEMATC

Commit message: Completed rev 3.0 schematics.
1) Replaced MPU with STM Accelerometer
Parts:
- P6: value CONN_5 -> Line Sensors; footprint (none) -> Pin_Headers:Pin_Header_Straight_1x05
- P7: value ANALOG -> Analog In; footprint (none) -> Pin_Headers:Pin_Header_Straight_1x03
Changed lines of the file:
@@
 $Descr A4 11693 8268
 encoding utf-8
-Sheet 9 10
+Sheet 10 10
 Title ""
 Date ""
@@
 P 2950 2675
 F 0 "P6" V 2900 2675 50  0000 C CNN
-F 1 "CONN_5" V 3000 2675 50  0000 C CNN
-F 2 "" H 2950 2675 60  0000 C CNN
+F 1 "Line Sensors" V 3000 2675 50  0000 C CNN
+F 2 "Pin_Headers:Pin_Header_Straight_1x05" H 2950 2675 60  0001 C CNN
 F 3 "" H 2950 2675 60  0000 C CNN
 	1    2950 2675
@@
 $EndComp
 $Comp
-L GND #PWR105
+L GND #PWR0102
 U 1 1 55A47561
 P 3550 3075
-F 0 "#PWR105" H 3550 3075 30  0001 C CNN
+F 0 "#PWR0102" H 3550 3075 30  0001 C CNN
 F 1 "GND" H 3550 3005 30  0001 C CNN
 F 2 "" H 3550 3075 60  0000 C CNN
@@
 $EndComp
 $Comp
-L 3V3 #PWR104
+L 3V3 #PWR0103
 U 1 1 55A47567
 P 3550 2325
-F 0 "#PWR104" H 3550 2425 40  0001 C CNN
+F 0 "#PWR0103" H 3550 2425 40  0001 C CNN
 F 1 "3V3" H 3550 2450 40  0000 C CNN
 F 2 "" H 3550 2325 60  0000 C CNN
@@
 F 0 "CAP1" H 10425 2800 60  0000 C CNN
 F 1 "CAP_TOUCH" H 10425 1975 60  0000 C CNN
-F 2 "" H 10650 2250 60  0000 C CNN
+F 2 "" H 10650 2250 60  0001 C CNN
 F 3 "" H 10650 2250 60  0000 C CNN
 	1    10425 2500
@@
 F 0 "R42" V 9880 2375 40  0000 C CNN
 F 1 "5k" V 9807 2376 40  0000 C CNN
-F 2 "" V 9730 2375 30  0000 C CNN
+F 2 "" V 9730 2375 30  0001 C CNN
 F 3 "" H 9800 2375 30  0000 C CNN
 	1    9800 2375
@@
 F 0 "R43" V 9880 2625 40  0000 C CNN
 F 1 "5k" V 9807 2626 40  0000 C CNN
-F 2 "" V 9730 2625 30  0000 C CNN
+F 2 "" V 9730 2625 30  0001 C CNN
 F 3 "" H 9800 2625 30  0000 C CNN
 	1    9800 2625
@@
 F 0 "R44" V 9880 2850 40  0000 C CNN
 F 1 "5k" V 9807 2851 40  0000 C CNN
-F 2 "" V 9730 2850 30  0000 C CNN
+F 2 "" V 9730 2850 30  0001 C CNN
 F 3 "" H 9800 2850 30  0000 C CNN
 	1    9800 2850
@@
 F 0 "R39" V 7005 2725 40  0000 C CNN
 F 1 "50k" V 6932 2726 40  0000 C CNN
-F 2 "" V 6855 2725 30  0000 C CNN
+F 2 "" V 6855 2725 30  0001 C CNN
 F 3 "" H 6925 2725 30  0000 C CNN
 	1    6925 2725
@@
 F 0 "C11" H 6725 2850 40  0000 L CNN
 F 1 "10pF" H 6731 2665 40  0000 L CNN
-F 2 "" H 6763 2600 30  0000 C CNN
+F 2 "" H 6763 2600 30  0001 C CNN
 F 3 "" H 6725 2750 60  0000 C CNN
 	1    6725 2750
@@
 	6725 3100 6725 2950
 $Comp
-L GND #PWR106
+L GND #PWR0104
 U 1 1 55A489A5
 P 6825 3175
-F 0 "#PWR106" H 6825 3175 30  0001 C CNN
+F 0 "#PWR0104" H 6825 3175 30  0001 C CNN
 F 1 "GND" H 6825 3105 30  0001 C CNN
 F 2 "" H 6825 3175 60  0000 C CNN
@@
 F 0 "R40" V 8330 2950 40  0000 C CNN
 F 1 "50k" V 8257 2951 40  0000 C CNN
-F 2 "" V 8180 2950 30  0000 C CNN
+F 2 "" V 8180 2950 30  0001 C CNN
 F 3 "" H 8250 2950 30  0000 C CNN
 	1    8250 2950
@@
 F 0 "C12" H 8050 3075 40  0000 L CNN
 F 1 "10pF" H 8056 2890 40  0000 L CNN
-F 2 "" H 8088 2825 30  0000 C CNN
+F 2 "" H 8088 2825 30  0001 C CNN
 F 3 "" H 8050 2975 60  0000 C CNN
 	1    8050 2975
@@
 	8050 3325 8050 3175
 $Comp
-L GND #PWR107
+L GND #PWR0105
 U 1 1 55A48CCB
 P 8150 3425
-F 0 "#PWR107" H 8150 3425 30  0001 C CNN
+F 0 "#PWR0105" H 8150 3425 30  0001 C CNN
 F 1 "GND" H 8150 3355 30  0001 C CNN
 F 2 "" H 8150 3425 60  0000 C CNN
@@
 F 0 "R41" V 9555 3200 40  0000 C CNN
 F 1 "50k" V 9482 3201 40  0000 C CNN
-F 2 "" V 9405 3200 30  0000 C CNN
+F 2 "" V 9405 3200 30  0001 C CNN
 F 3 "" H 9475 3200 30  0000 C CNN
 	1    9475 3200
@@
 F 0 "C13" H 9275 3325 40  0000 L CNN
 F 1 "10pF" H 9281 3140 40  0000 L CNN
-F 2 "" H 9313 3075 30  0000 C CNN
+F 2 "" H 9313 3075 30  0001 C CNN
 F 3 "" H 9275 3225 60  0000 C CNN
 	1    9275 3225
@@
 	9275 3475 9275 3425
 $Comp
-L GND #PWR108
+L GND #PWR0106
 U 1 1 55A48F7B
 P 9375 3550
-F 0 "#PWR108" H 9375 3550 30  0001 C CNN
+F 0 "#PWR0106" H 9375 3550 30  0001 C CNN
 F 1 "GND" H 9375 3480 30  0001 C CNN
 F 2 "" H 9375 3550 60  0000 C CNN
@@
 P 3100 3750
 F 0 "P7" V 3050 3750 40  0000 C CNN
-F 1 "ANALOG" V 3150 3750 40  0000 C CNN
-F 2 "" H 3100 3750 60  0000 C CNN
+F 1 "Analog In" V 3150 3750 40  0000 C CNN
+F 2 "Pin_Headers:Pin_Header_Straight_1x03" H 3100 3750 60  0001 C CNN
 F 3 "" H 3100 3750 60  0000 C CNN
 	1    3100 3750

Commit message: Added most of the footprints needed to make this work
Parts:
- C11, C12, C13: footprint (none) -> Capacitors_SMD:c_0603
- R39, R40, R41, R42, R43, R44: footprint (none) -> Resistors_SMD:R_0603
Changed lines of the file:
@@
 $EndComp
 $Comp
-L GND #PWR0104
+L GND #PWR0105
 U 1 1 55A47561
 P 3550 3075
-F 0 "#PWR0104" H 3550 3075 30  0001 C CNN
+F 0 "#PWR0105" H 3550 3075 30  0001 C CNN
 F 1 "GND" H 3550 3005 30  0001 C CNN
 F 2 "" H 3550 3075 60  0000 C CNN
@@
 $EndComp
 $Comp
-L 3V3 #PWR0105
+L 3V3 #PWR0106
 U 1 1 55A47567
 P 3550 2325
-F 0 "#PWR0105" H 3550 2425 40  0001 C CNN
+F 0 "#PWR0106" H 3550 2425 40  0001 C CNN
 F 1 "3V3" H 3550 2450 40  0000 C CNN
 F 2 "" H 3550 2325 60  0000 C CNN
@@
 F 0 "R42" V 9880 2375 40  0000 C CNN
 F 1 "5k" V 9807 2376 40  0000 C CNN
-F 2 "" V 9730 2375 30  0001 C CNN
+F 2 "Resistors_SMD:R_0603" V 9730 2375 30  0001 C CNN
 F 3 "" H 9800 2375 30  0000 C CNN
 	1    9800 2375
@@
 F 0 "R43" V 9880 2625 40  0000 C CNN
 F 1 "5k" V 9807 2626 40  0000 C CNN
-F 2 "" V 9730 2625 30  0001 C CNN
+F 2 "Resistors_SMD:R_0603" V 9730 2625 30  0001 C CNN
 F 3 "" H 9800 2625 30  0000 C CNN
 	1    9800 2625
@@
 F 0 "R44" V 9880 2850 40  0000 C CNN
 F 1 "5k" V 9807 2851 40  0000 C CNN
-F 2 "" V 9730 2850 30  0001 C CNN
+F 2 "Resistors_SMD:R_0603" V 9730 2850 30  0001 C CNN
 F 3 "" H 9800 2850 30  0000 C CNN
 	1    9800 2850
@@
 F 0 "R39" V 7005 2725 40  0000 C CNN
 F 1 "50k" V 6932 2726 40  0000 C CNN
-F 2 "" V 6855 2725 30  0001 C CNN
+F 2 "Resistors_SMD:R_0603" V 6855 2725 30  0001 C CNN
 F 3 "" H 6925 2725 30  0000 C CNN
 	1    6925 2725
@@
 F 0 "C11" H 6725 2850 40  0000 L CNN
 F 1 "10pF" H 6731 2665 40  0000 L CNN
-F 2 "" H 6763 2600 30  0001 C CNN
+F 2 "Capacitors_SMD:c_0603" H 6763 2600 30  0001 C CNN
 F 3 "" H 6725 2750 60  0000 C CNN
 	1    6725 2750
@@
 	6725 3100 6725 2950
 $Comp
-L GND #PWR0106
+L GND #PWR0107
 U 1 1 55A489A5
 P 6825 3175
-F 0 "#PWR0106" H 6825 3175 30  0001 C CNN
+F 0 "#PWR0107" H 6825 3175 30  0001 C CNN
 F 1 "GND" H 6825 3105 30  0001 C CNN
 F 2 "" H 6825 3175 60  0000 C CNN
@@
 F 0 "R40" V 8330 2950 40  0000 C CNN
 F 1 "50k" V 8257 2951 40  0000 C CNN
-F 2 "" V 8180 2950 30  0001 C CNN
+F 2 "Resistors_SMD:R_0603" V 8180 2950 30  0001 C CNN
 F 3 "" H 8250 2950 30  0000 C CNN
 	1    8250 2950
@@
 F 0 "C12" H 8050 3075 40  0000 L CNN
 F 1 "10pF" H 8056 2890 40  0000 L CNN
-F 2 "" H 8088 2825 30  0001 C CNN
+F 2 "Capacitors_SMD:c_0603" H 8088 2825 30  0001 C CNN
 F 3 "" H 8050 2975 60  0000 C CNN
 	1    8050 2975
@@
 	8050 3325 8050 3175
 $Comp
-L GND #PWR0107
+L GND #PWR0108
 U 1 1 55A48CCB
 P 8150 3425
-F 0 "#PWR0107" H 8150 3425 30  0001 C CNN
+F 0 "#PWR0108" H 8150 3425 30  0001 C CNN
 F 1 "GND" H 8150 3355 30  0001 C CNN
 F 2 "" H 8150 3425 60  0000 C CNN
@@
 F 0 "R41" V 9555 3200 40  0000 C CNN
 F 1 "50k" V 9482 3201 40  0000 C CNN
-F 2 "" V 9405 3200 30  0001 C CNN
+F 2 "Resistors_SMD:R_0603" V 9405 3200 30  0001 C CNN
 F 3 "" H 9475 3200 30  0000 C CNN
 	1    9475 3200
@@
 F 0 "C13" H 9275 3325 40  0000 L CNN
 F 1 "10pF" H 9281 3140 40  0000 L CNN
-F 2 "" H 9313 3075 30  0001 C CNN
+F 2 "Capacitors_SMD:c_0603" H 9313 3075 30  0001 C CNN
 F 3 "" H 9275 3225 60  0000 C CNN
 	1    9275 3225
@@
 	9275 3475 9275 3425
 $Comp
-L GND #PWR0108
+L GND #PWR0109
 U 1 1 55A48F7B
 P 9375 3550
-F 0 "#PWR0108" H 9375 3550 30  0001 C CNN
+F 0 "#PWR0109" H 9375 3550 30  0001 C CNN
 F 1 "GND" H 9375 3480 30  0001 C CNN
 F 2 "" H 9375 3550 60  0000 C CNN
