File: board/mainboard/MotorDrivers.sch (KiCad schematic (older format))
At the start: 13 parts, among them P17 Motor2, P2 SWD_KE04, P3 Motor1, U7 MKE04Z8VTG, U8 ZXBM5210-SP, U9 ZXBM5210-SP

Commit message: Added most of the footprints needed to make this work
Parts:
- C14, C28, C30: footprint (none) -> Capacitors_SMD:c_0603
- C15, C27: footprint (none) -> Capacitors_SMD:c_0805
- P2: footprint (none) -> footprints:2x5_Debug_Header; symbol CONN_02X05 -> CONN_CORTEXDBG
- U7: footprint (none) -> footprints:MKE04_
- U8, U9: footprint (none) -> footprints:ZXBM5210_
Connections:
- no-connect marks 6 -> 5
Changed lines of the file:
@@
 F 0 "U8" H 7625 2750 60  0000 C CNN
 F 1 "ZXBM5210-SP" H 7275 3150 60  0000 C CNN
-F 2 "" H 7375 2775 60  0001 C CNN
+F 2 "footprints:ZXBM5210_" H 7375 2775 60  0001 C CNN
 F 3 "" H 7375 2775 60  0000 C CNN
 	1    7500 2775
@@
 F 0 "C28" H 7650 1425 40  0000 L CNN
 F 1 "0.1uF" H 7656 1240 40  0000 L CNN
-F 2 "" H 7688 1175 30  0001 C CNN
+F 2 "Capacitors_SMD:c_0603" H 7688 1175 30  0001 C CNN
 F 3 "" H 7650 1325 60  0000 C CNN
 	1    7650 1325
@@
 F 0 "C15" H 6325 1650 40  0000 L CNN
 F 1 "10uF" H 6331 1465 40  0000 L CNN
-F 2 "" H 6363 1400 30  0001 C CNN
+F 2 "Capacitors_SMD:c_0805" H 6363 1400 30  0001 C CNN
 F 3 "" H 6325 1550 60  0000 C CNN
 	1    6325 1550
@@
 F 0 "C27" H 6325 4550 40  0000 L CNN
 F 1 "10uF" H 6331 4365 40  0000 L CNN
-F 2 "" H 6363 4300 30  0001 C CNN
+F 2 "Capacitors_SMD:c_0805" H 6363 4300 30  0001 C CNN
 F 3 "" H 6325 4450 60  0000 C CNN
 	1    6325 4450
@@
 F 0 "C30" H 7650 4325 40  0000 L CNN
 F 1 "0.1uF" H 7656 4140 40  0000 L CNN
-F 2 "" H 7688 4075 30  0001 C CNN
+F 2 "Capacitors_SMD:c_0603" H 7688 4075 30  0001 C CNN
 F 3 "" H 7650 4225 60  0000 C CNN
 	1    7650 4225
@@
 F 0 "U9" H 7625 5650 60  0000 C CNN
 F 1 "ZXBM5210-SP" H 7275 6050 60  0000 C CNN
-F 2 "" H 7375 5675 60  0001 C CNN
+F 2 "footprints:ZXBM5210_" H 7375 5675 60  0001 C CNN
 F 3 "" H 7375 5675 60  0000 C CNN
 	1    7500 5675
@@
 F 0 "U7" H 3700 4400 60  0000 C CNN
 F 1 "MKE04Z8VTG" H 3675 4750 60  0000 C CNN
-F 2 "" H 3700 4400 60  0001 C CNN
+F 2 "footprints:MKE04_" H 3700 4400 60  0001 C CNN
 F 3 "" H 3700 4400 60  0000 C CNN
 	1    3700 4400
@@
 F 0 "C14" H 2500 4325 40  0000 L CNN
 F 1 "0.1uF" H 2506 4140 40  0000 L CNN
-F 2 "" H 2538 4075 30  0001 C CNN
+F 2 "Capacitors_SMD:c_0603" H 2538 4075 30  0001 C CNN
 F 3 "" H 2500 4225 60  0000 C CNN
 	1    2500 4225
 	1    0    0    -1
 $EndComp
-$Comp
-L CONN_02X05 P2
-U 1 1 55A74FFD
-P 2150 1500
-F 0 "P2" H 2150 1800 50  0000 C CNN
-F 1 "SWD_KE04" H 2150 1200 50  0000 C CNN
-F 2 "" H 2150 300 60  0001 C CNN
-F 3 "" H 2150 300 60  0000 C CNN
-	1    2150 1500
-	1    0    0    -1
-$EndComp
-Text Label 3025 1300 2    60   ~ 0
+Text Label 3325 1300 2    60   ~ 0
 SWDIO_KE04
-Text Label 3025 1400 2    60   ~ 0
+Text Label 3325 1400 2    60   ~ 0
 SWDCLK_KE04
-NoConn ~ 2400 1500
-NoConn ~ 2400 1600
 Text Label 2200 2825 0    60   ~ 0
 SWDIO_KE04
 Text Label 2200 2925 0    60   ~ 0
 SWDCLK_KE04
-Text Label 3025 1700 2    60   ~ 0
+Text Label 3325 1700 2    60   ~ 0
 nRESET_KE04
 Text Label 2200 2725 0    60   ~ 0
@@
 L 3V3 #PWR023
 U 1 1 55A75D91
-P 1750 1175
-F 0 "#PWR023" H 1750 1275 40  0001 C CNN
-F 1 "3V3" H 1750 1300 40  0000 C CNN
-F 2 "" H 1750 1175 60  0000 C CNN
-F 3 "" H 1750 1175 60  0000 C CNN
-	1    1750 1175
+P 1600 1200
+F 0 "#PWR023" H 1600 1300 40  0001 C CNN
+F 1 "3V3" H 1600 1325 40  0000 C CNN
+F 2 "" H 1600 1200 60  0000 C CNN
+F 3 "" H 1600 1200 60  0000 C CNN
+	1    1600 1200
 	1    0    0    -1
 $EndComp
@@
 L GND #PWR024
 U 1 1 55A75F3F
-P 1750 1850
-F 0 "#PWR024" H 1750 1850 30  0001 C CNN
-F 1 "GND" H 1750 1780 30  0001 C CNN
-F 2 "" H 1750 1850 60  0000 C CNN
-F 3 "" H 1750 1850 60  0000 C CNN
-	1    1750 1850
-	1    0    0    -1
-$EndComp
-NoConn ~ 1900 1600
+P 1600 1875
+F 0 "#PWR024" H 1600 1875 30  0001 C CNN
+F 1 "GND" H 1600 1805 30  0001 C CNN
+F 2 "" H 1600 1875 60  0000 C CNN
+F 3 "" H 1600 1875 60  0000 C CNN
+	1    1600 1875
+	1    0    0    -1
+$EndComp
 $Comp
 L R R6
@@
 Connection ~ 2500 4475
 Wire Wire Line
-	1750 1300 1900 1300
-Wire Wire Line
-	1750 1175 1750 1300
-Wire Wire Line
-	2400 1300 3025 1300
-Wire Wire Line
-	2400 1400 3025 1400
-Wire Wire Line
-	2400 1700 3025 1700
+	2700 1300 3325 1300
+Wire Wire Line
+	2700 1400 3325 1400
+Wire Wire Line
+	2700 1700 3325 1700
 Wire Wire Line
 	2150 2725 2775 2725
@@
 Wire Wire Line
 	2200 2925 2775 2925
-Wire Wire Line
-	1900 1700 1750 1700
-Wire Wire Line
-	1750 1700 1750 1850
-Wire Wire Line
-	1900 1400 1750 1400
-Wire Wire Line
-	1750 1400 1750 1725
-Connection ~ 1750 1725
-Wire Wire Line
-	1900 1500 1750 1500
-Connection ~ 1750 1500
 Wire Wire Line
 	2525 3475 2525 3525
@@
 Wire Wire Line
 	6125 1250 6550 1250
+$Comp
+L CONN_CORTEXDBG P2
+U 1 1 55A74FFD
+P 2150 1500
+F 0 "P2" H 1850 1850 50  0000 C CNN
+F 1 "SWD_KE04" H 2150 1200 50  0000 C CNN
+F 2 "footprints:2x5_Debug_Header" H 2150 300 60  0001 C CNN
+F 3 "" H 2150 300 60  0000 C CNN
+	1    2150 1500
+	1    0    0    -1
+$EndComp
+Wire Wire Line
+	1650 1700 1600 1700
+Wire Wire Line
+	1600 1700 1600 1875
+Wire Wire Line
+	1650 1400 1600 1400
+Wire Wire Line
+	1600 1400 1600 1725
+Connection ~ 1600 1725
+Wire Wire Line
+	1650 1500 1600 1500
+Connection ~ 1600 1500
+Wire Wire Line
+	1650 1300 1600 1300
+Wire Wire Line
+	1600 1300 1600 1200
+NoConn ~ 2700 1500
+NoConn ~ 2700 1600
 $EndSCHEMATC

Commit message: Saved last few changes before leaving
Parts:
- P17, P3: footprint (none) -> Pin_Headers:Pin_Header_Straight_1x02
Changed lines of the file:
@@
 F 0 "P3" H 10550 3500 50  0000 C CNN
 F 1 "Motor1" V 10650 3350 50  0000 C CNN
-F 2 "" H 10550 3350 60  0001 C CNN
+F 2 "Pin_Headers:Pin_Header_Straight_1x02" H 10550 3350 60  0001 C CNN
 F 3 "" H 10550 3350 60  0000 C CNN
 	1    10550 3350
@@
 F 0 "P17" V 10550 3850 40  0000 C CNN
 F 1 "Motor2" V 10650 3850 40  0000 C CNN
-F 2 "" H 10600 3850 60  0001 C CNN
+F 2 "Pin_Headers:Pin_Header_Straight_1x02" H 10600 3850 60  0001 C CNN
 F 3 "" H 10600 3850 60  0000 C CNN
 	1    10600 3850
