File: board/cc3200board/cc3200board-io.sch (KiCad schematic (older format))
At the start: 7 parts, among them P1 PROG, P2 CONN_GPIO, P3 CONN_JTAG, U1 CC3200R1M2RGCR

Commit message: Fixed CC3200 symbol, missing GPIO28 pin. Complete pin check on symbol
Connections:
- net labels added: GPIO31
Changed lines of the file:
@@
 Text Label 9175 4675 0    60   ~ 0
 SOP2
+Text HLabel 1250 4575 0    60   Input ~ 0
+GPIO31
 $EndSCHEMATC

Commit message: Finished schematic layout
Connections:
- net labels added: GPIO22, GPIO30, nRESET
- wire segments 57 -> 62
Changed lines of the file:
@@
 Text Label 4300 6750 0    60   ~ 0
 TMS
+Text Label 8175 4575 0    60   ~ 0
+TDI
+Text Label 8175 4675 0    60   ~ 0
+TDO
+Text Label 8175 4775 0    60   ~ 0
+TCK
+Text Label 8175 4875 0    60   ~ 0
+TMS
+Text Label 9350 4575 2    60   ~ 0
+SOP0
+Text Label 9350 4675 2    60   ~ 0
+SOP2
+Text HLabel 1250 4575 0    60   Input ~ 0
+GPIO31
+Text Label 1400 4575 0    60   ~ 0
+GPIO31
+Text HLabel 1250 4725 0    60   Input ~ 0
+nRESET
+Text Label 1425 4725 0    60   ~ 0
+nRESET
+Text Label 9350 4775 2    60   ~ 0
+nRESET
 Wire Wire Line
 	2800 6450 2800 6650
@@
 	2600 6450 2600 6650
 Wire Wire Line
-	3000 6650 3000 6450
+	3000 6450 3000 6650
 Wire Wire Line
 	3000 7300 3000 7150
@@
 Wire Wire Line
 	9150 4675 9350 4675
-Text Label 8225 4575 0    60   ~ 0
-TDI
-Text Label 8225 4675 0    60   ~ 0
-TDO
-Text Label 8225 4775 0    60   ~ 0
-TCK
-Text Label 8225 4875 0    60   ~ 0
-TMS
-Text Label 9175 4575 0    60   ~ 0
-SOP0
-Text Label 9175 4675 0    60   ~ 0
-SOP2
-Text HLabel 1250 4575 0    60   Input ~ 0
-GPIO31
+Wire Wire Line
+	1250 4575 1400 4575
+Wire Wire Line
+	1250 4725 1425 4725
+Wire Wire Line
+	9150 4775 9350 4775
+Wire Wire Line
+	5350 5100 5700 5100
+Wire Wire Line
+	5350 5750 5700 5750
+Text Label 5700 5750 2    60   ~ 0
+GPIO30
+Entry Wire Line
+	5700 5750 5800 5850
+Entry Wire Line
+	5700 5100 5800 5200
+Text Label 5700 5100 2    60   ~ 0
+GPIO22
 $EndSCHEMATC

Commit message: Fixed mirrored footprint, outlines
Parts:
- added WB1: WIFI_BOARD, symbol WIFI_BOARD
Connections:
- net 3V3: now also WB1.17 (Vcc), WB1.9 (Vcc)
- net GND: now also P3.8, WB1.16 (GND), WB1.24 (GND)
- net GPIO0: now also WB1.4 (SPI_SEL0)
- net GPIO10: now also WB1.14 (UART_TX)
- net GPIO11: now also WB1.13 (UART_RX)
- net GPIO12: now also WB1.12 (I2C_CL)
- net GPIO13: now also WB1.11 (I2C_DA)
- net GPIO14: now also WB1.1 (SPI_SCK)
- net GPIO15: now also WB1.3 (SPI_MISO)
- net GPIO16: now also WB1.2 (SPI_MOSI)
- net GPIO17: now also WB1.7 (SPI_CS)
- net GPIO22: now also WB1.5 (SPI_SEL1)
- net GPIO3: now also WB1.10 (CONTROL)
- net GPIO30: now also WB1.6 (SPI_SEL2)
- net GPIO31: now also WB1.8 (GLCD_A0)
- net GPIO4: now also WB1.18 (MPUINT)
- net GPIO5: now also WB1.19 (RTCINT1)
- net GPIO6: now also WB1.20 (RTCINT2)
- net GPIO7: now also WB1.21 (SD_SWITCH)
- net GPIO8: now also WB1.22 (MOTOR1F)
- net GPIO9: now also WB1.23 (MOTOR2F)
- new net GPIO28: WB1.15 (INT)
Other:
- moved on the sheet: P1, P2, P3

Commit message: Rev 1.0 of CC3200board
Parts:
- removed P2: CONN_GPIO, symbol CONN_8X2
Connections:
- wire segments 91 -> 92
Changed lines of the file:
@@
 $EndComp
 $Comp
-L GND #PWR028
+L GND #PWR030
 U 1 1 5453196F
 P 2800 7400
-F 0 "#PWR028" H 2800 7400 30  0001 C CNN
+F 0 "#PWR030" H 2800 7400 30  0001 C CNN
 F 1 "GND" H 2800 7330 30  0001 C CNN
 F 2 "" H 2800 7400 60  0000 C CNN
@@
 GPIO[7:0]
 $Comp
-L GND #PWR029
+L GND #PWR031
 U 1 1 54533722
 P 8200 800
-F 0 "#PWR029" H 8200 800 30  0001 C CNN
+F 0 "#PWR031" H 8200 800 30  0001 C CNN
 F 1 "GND" H 8200 730 30  0001 C CNN
 F 2 "" H 8200 800 60  0000 C CNN
@@
 Text Label 8150 1300 0    60   ~ 0
 GPIO[7:0]
-$Comp
-L CONN_8X2 P2
-U 1 1 54533F4C
-P 8900 1850
-F 0 "P2" H 8900 2300 60  0000 C CNN
-F 1 "CONN_GPIO" V 8900 1850 50  0000 C CNN
-F 2 "" H 8900 1850 60  0001 C CNN
-F 3 "" H 8900 1850 60  0000 C CNN
-	1    8900 1850
-	1    0    0    -1
-$EndComp
 Text Label 8200 1500 0    60   ~ 0
 GPIO0
@@
 Text Label 4300 6750 0    60   ~ 0
 TMS
+Text Label 8325 3050 0    60   ~ 0
+TDI
+Text Label 8325 2950 0    60   ~ 0
+TDO
+Text Label 8325 2850 0    60   ~ 0
+TCK
 Text Label 8325 2750 0    60   ~ 0
-TDI
-Text Label 8325 2850 0    60   ~ 0
-TDO
-Text Label 8325 2950 0    60   ~ 0
-TCK
-Text Label 8325 3050 0    60   ~ 0
 TMS
 Text Label 9500 2750 2    60   ~ 0
@@
 	8200 800  8550 800
 Wire Wire Line
-	8550 900  7675 900
+	7675 900  8550 900
 Wire Wire Line
 	8250 1000 8550 1000
@@
 GPIO28
 $Comp
-L GND #PWR030
+L GND #PWR032
 U 1 1 5473ED2E
 P 9725 4850
-F 0 "#PWR030" H 9725 4850 30  0001 C CNN
+F 0 "#PWR032" H 9725 4850 30  0001 C CNN
 F 1 "GND" H 9725 4780 30  0001 C CNN
 F 2 "" H 9725 4850 60  0000 C CNN
@@
 	9725 4750 9725 4850
 $Comp
-L GND #PWR031
+L GND #PWR033
 U 1 1 5473EDFA
 P 9750 6225
-F 0 "#PWR031" H 9750 6225 30  0001 C CNN
+F 0 "#PWR033" H 9750 6225 30  0001 C CNN
 F 1 "GND" H 9750 6155 30  0001 C CNN
 F 2 "" H 9750 6225 60  0000 C CNN
@@
 3V3
 $Comp
-L GND #PWR?
+L GND #PWR034
 U 1 1 54740A51
 P 9475 3150
-F 0 "#PWR?" H 9475 3150 30  0001 C CNN
+F 0 "#PWR034" H 9475 3150 30  0001 C CNN
 F 1 "GND" H 9475 3080 30  0001 C CNN
 F 2 "" H 9475 3150 60  0000 C CNN
@@
 Wire Wire Line
 	9475 3050 9475 3150
+Wire Wire Line
+	5350 6000 5675 6000
+Text Label 5675 6000 0    60   ~ 0
+GPIO28
 $EndSCHEMATC

Commit message: Fixed error in GND plane on L4
Parts:
- U1: value CC3200R1M2RGCR -> CC3200
Changed lines of the file:
@@
 P 3650 3600
 F 0 "U1" H 2300 6400 45  0000 C CNN
-F 1 "CC3200R1M2RGCR" H 4700 1100 45  0000 C CNN
+F 1 "CC3200" H 4700 1100 45  0000 C CNN
 F 2 "VQFN64" H 3650 4100 35  0000 C CIN
 F 3 "" H 4350 4000 60  0000 C CNN
@@
 $EndComp
 $Comp
-L GND #PWR030
+L GND #PWR029
 U 1 1 5453196F
 P 2800 7400
-F 0 "#PWR030" H 2800 7400 30  0001 C CNN
+F 0 "#PWR029" H 2800 7400 30  0001 C CNN
 F 1 "GND" H 2800 7330 30  0001 C CNN
 F 2 "" H 2800 7400 60  0000 C CNN
@@
 GPIO[7:0]
 $Comp
-L GND #PWR031
+L GND #PWR030
 U 1 1 54533722
 P 8200 800
-F 0 "#PWR031" H 8200 800 30  0001 C CNN
+F 0 "#PWR030" H 8200 800 30  0001 C CNN
 F 1 "GND" H 8200 730 30  0001 C CNN
 F 2 "" H 8200 800 60  0000 C CNN
@@
 GPIO28
 $Comp
-L GND #PWR032
+L GND #PWR031
 U 1 1 5473ED2E
 P 9725 4850
-F 0 "#PWR032" H 9725 4850 30  0001 C CNN
+F 0 "#PWR031" H 9725 4850 30  0001 C CNN
 F 1 "GND" H 9725 4780 30  0001 C CNN
 F 2 "" H 9725 4850 60  0000 C CNN
@@
 	9725 4750 9725 4850
 $Comp
-L GND #PWR033
+L GND #PWR032
 U 1 1 5473EDFA
 P 9750 6225
-F 0 "#PWR033" H 9750 6225 30  0001 C CNN
+F 0 "#PWR032" H 9750 6225 30  0001 C CNN
 F 1 "GND" H 9750 6155 30  0001 C CNN
 F 2 "" H 9750 6225 60  0000 C CNN
@@
 3V3
 $Comp
-L GND #PWR034
+L GND #PWR033
 U 1 1 54740A51
 P 9475 3150
-F 0 "#PWR034" H 9475 3150 30  0001 C CNN
+F 0 "#PWR033" H 9475 3150 30  0001 C CNN
 F 1 "GND" H 9475 3080 30  0001 C CNN
 F 2 "" H 9475 3150 60  0000 C CNN
