File: board/cc3200modboard/cc3200modboard.kicad_pcb (KiCad board)
At the start: 2 copper layers, 40.7 x 33.3 mm, 20 parts, among them P1 PROG, P2 JTAG, P3 BOOTLDR, SW1 RESET, U1 CC3200MOD

Commit message: Committed version of CC3200 PCB for r2
Routing:
- net GND: track 67.9 -> 71.0 mm
- net /RF_FEED: track 9.11 -> 8.54 mm
Other:
- net class IMP_50OHM: clearance 0.2 -> 0.1524; trace_width 0.7646 -> 0.894771
- board text added: "Darren S Hasith Vi Robert N"

Commit message: Finished revision 2 of WiFi Board
Parts:
- added G***: LOGO, crab:crab, F.Cu at (153.6, 120.1)
- added R5: 10K, Resistors_SMD:R_0805, F.Cu at (157.8, 116.2)
- moved L1 11.4 mm to (144.1, 115.0)
- moved C6 11.4 mm to (145.1, 117.2)
- moved E1 5.04 mm to (147.3, 122.5), turned to 90 degrees
- moved D2 2.07 mm to (134.4, 117.6), turned to 270 degrees
- moved D1 1.66 mm to (136.3, 117.6), turned to 270 degrees
Routing:
- net GND: track 71.0 -> 39.6 mm, vias 41 -> 31
- net /GPIO1: track 52.4 -> 26.9 mm
- net /nRESET: track 76.3 -> 51.6 mm, vias 8 -> 0
- net /GPIO9: track 27.7 -> 4.53 mm, vias 1 -> 0
- net /TDO: track 35.6 -> 13.6 mm
- net /GPIO8: track 26.4 -> 5.06 mm, vias 1 -> 0
- net /GPIO0: track 12.5 -> 32.4 mm, vias 0 -> 2
- net /TCK: track 43.7 -> 24.0 mm, vias 1 -> 0
- net /GPIO7: track 25.2 -> 5.58 mm, vias 1 -> 0
- net /GPIO6: track 25.6 -> 6.11 mm, vias 1 -> 0
- net /TMS: track 35.7 -> 17.3 mm, vias 1 -> 0
- net /GPIO5: track 25.8 -> 7.66 mm, vias 1 -> 0
- net /GPIO3: track 28.4 -> 10.4 mm, vias 2 -> 1
- net /GPIO4: track 26.3 -> 8.93 mm, vias 1 -> 0
- net /GPIO2: track 43.4 -> 27.5 mm, vias 3 -> 1
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Other:
- board size 40.7 x 33.3 mm -> 40.7 x 33.6 mm
- board text added: "Darren S Hasith V Robert N"
- board text added: "Proxima r2.5"
- board text added: "Wi-Fi Crab"
- board text removed: "Darren S Hasith Vi Robert N"
- board text removed: "Proxima r2.0"
